File: kicad01_power_board_for_nuclear_team/002_input28to22v.kicad_sch (KiCad schematic)
At the start: 9 parts, among them Q251 nmos75v80a_IRFS3607TRLPBF

Commit message: x
Parts:
- C201, C211: symbol 1001_un:c0805_35v10u -> 1003_cap:c0805_35v10u
- PTC201: symbol 1001_un:PTC_fuse_7A -> 1002_res:PTC_fuse_7A
- Q251: symbol 1001_un:nmos75v80a_IRFS3607TRLPBF -> 1004_led_mos:nmosTO263_75v80A; PartDesc (none) -> N-Channel 75 V 80A (Tc) 140W (Tc) Surface Mount D2PAK; PartNum (none) -> IRFS3607TRLPBF
- R211: symbol 1001_un:R1206_0.0 -> 1002_res:R1206_0.0
- R221, R222: symbol 1001_un:R0603_1M -> 1002_res:R0603_1M
Changed lines of the file:
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@@
     (pin "1")
   )
-  (symbol (lib_id "1001_un:R1206_0.0") (at 116.84 62.23 0) (unit 1)
+  (symbol (lib_id "1002_res:R1206_0.0") (at 116.84 62.23 0) (unit 1)
     (in_bom yes) (on_board yes)
     (property "Reference" "R211" (id 0) (at 116.84 59.69 0)
@@
     (pin "2")
   )
-  (symbol (lib_id "1001_un:R0603_1M") (at 105.41 69.85 90) (unit 1)
+  (symbol (lib_id "1002_res:R0603_1M") (at 105.41 69.85 90) (unit 1)
     (in_bom yes) (on_board yes) (fields_autoplaced)
     (property "Reference" "R221" (id 0) (at 107.95 69.215 90)
@@
     (pin "2")
   )
-  (symbol (lib_id "1001_un:R0603_1M") (at 105.41 80.01 90) (unit 1)
+  (symbol (lib_id "1002_res:R0603_1M") (at 105.41 80.01 90) (unit 1)
     (in_bom yes) (on_board yes) (fields_autoplaced)
     (property "Reference" "R222" (id 0) (at 107.95 79.375 90)
@@
     (pin "2")
   )
-  (symbol (lib_id "1001_un:c0805_35v10u") (at 72.39 72.39 0) (unit 1)
+  (symbol (lib_id "1003_cap:c0805_35v10u") (at 72.39 72.39 0) (unit 1)
     (in_bom yes) (on_board yes)
     (property "Reference" "C211" (id 0) (at 73.66 76.2 0)
@@
     (pin "2")
   )
-  (symbol (lib_id "1001_un:nmos75v80a_IRFS3607TRLPBF") (at 93.98 83.82 90) (mirror x) (unit 1)
+  (symbol (lib_id "1004_led_mos:nmosTO263_75v80A") (at 93.98 83.82 90) (mirror x) (unit 1)
     (in_bom yes) (on_board yes)
     (property "Reference" "Q251" (id 0) (at 87.63 87.63 0)
@@
       (effects (font (size 1.27 1.27) italic) (justify left) hide)
     )
-    (property "Datasheet" "https://www.digikey.com/en/products/detail/infineon-technologies/IRFS3607TRLPBF/1925542" (id 3) (at 72.39 66.04 0)
+    (property "Datasheet" "https://www.digikey.com/en/products/detail/infineon-technologies/IRFS3607TRLPBF/1925392" (id 3) (at 72.39 66.04 0)
       (effects (font (size 1.27 1.27)) (justify left) hide)
+    )
+    (property "PartNum" "IRFS3607TRLPBF" (id 4) (at 69.85 83.82 0)
+      (effects (font (size 1.27 1.27)) hide)
+    )
+    (property "PartDesc" "N-Channel 75 V 80A (Tc) 140W (Tc) Surface Mount D2PAK" (id 5) (at 78.74 90.17 0)
+      (effects (font (size 1.27 1.27)) hide)
     )
     (pin "1")
@@
     (pin "3")
   )
-  (symbol (lib_id "1001_un:PTC_fuse_7A") (at 81.28 86.36 0) (unit 1)
+  (symbol (lib_id "1002_res:PTC_fuse_7A") (at 81.28 86.36 0) (unit 1)
     (in_bom yes) (on_board yes) (fields_autoplaced)
     (property "Reference" "PTC201" (id 0) (at 81.28 81.28 0)
@@
     (pin "2")
   )
-  (symbol (lib_id "1001_un:c0805_35v10u") (at 41.91 73.66 0) (unit 1)
+  (symbol (lib_id "1003_cap:c0805_35v10u") (at 41.91 73.66 0) (unit 1)
     (in_bom yes) (on_board yes)
     (property "Reference" "C201" (id 0) (at 43.18 77.47 0)

Commit message: x
Parts:
- H201, H211: symbol 1001_un:hdr_2x1_1-1123723-2 -> 1008_hdr:hdr_2x1_1-1123723-2
Changed lines of the file:
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@@
     (pin "2")
   )
-  (symbol (lib_id "1001_un:hdr_2x1_1-1123723-2") (at 62.23 72.39 90) (unit 1)
+  (symbol (lib_id "1008_hdr:hdr_2x1_1-1123723-2") (at 62.23 72.39 90) (unit 1)
     (in_bom yes) (on_board yes)
     (property "Reference" "H211" (id 0) (at 62.23 67.31 90)
@@
     (pin "2")
   )
-  (symbol (lib_id "1001_un:hdr_2x1_1-1123723-2") (at 31.75 72.39 90) (unit 1)
+  (symbol (lib_id "1008_hdr:hdr_2x1_1-1123723-2") (at 31.75 72.39 90) (unit 1)
     (in_bom yes) (on_board yes)
     (property "Reference" "H201" (id 0) (at 31.75 67.31 90)

Commit message: x
Parts:
- C201, C211: footprint 02_dyn_pcblib:C0805mix0603 -> 2004_cap:C0805mix0603
- H201, H211: footprint 02_dyn_pcblib:hdr_2x1_1-1123723-2 -> 2002_hdr:hdr_2x1_1-1123723-2
- PTC201: footprint 02_dyn_pcblib:ptc_fuse_2920 -> 2003_res:ptc_fuse_2920
- Q251: value nmos75v80a_IRFS3607TRLPBF -> nmosTO263_75v80A; footprint 02_dyn_pcblib:d2pak_TO263 -> 2001_dyn_pcblib:d2pak_TO263
- R211: footprint 02_dyn_pcblib:R1206mix0603 -> 2003_res:R1206mix0603
- R221, R222: footprint 02_dyn_pcblib:C0603 -> 2004_cap:C0603
Changed lines of the file:
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@@
       (effects (font (size 0.5 0.5)))
     )
-    (property "Footprint" "02_dyn_pcblib:R1206mix0603" (id 2) (at 116.84 50.8 0)
+    (property "Footprint" "2003_res:R1206mix0603" (id 2) (at 116.84 50.8 0)
       (effects (font (size 1.27 1.27)) hide)
     )
@@
       (effects (font (size 0.5 0.5)))
     )
-    (property "Footprint" "02_dyn_pcblib:C0603" (id 2) (at 95.25 68.58 0)
+    (property "Footprint" "2004_cap:C0603" (id 2) (at 95.25 68.58 0)
       (effects (font (size 1.27 1.27)) hide)
     )
@@
       (effects (font (size 0.5 0.5)))
     )
-    (property "Footprint" "02_dyn_pcblib:C0603" (id 2) (at 95.25 78.74 0)
+    (property "Footprint" "2004_cap:C0603" (id 2) (at 95.25 78.74 0)
       (effects (font (size 1.27 1.27)) hide)
     )
@@
       (effects (font (size 0.5 0.5)))
     )
-    (property "Footprint" "02_dyn_pcblib:C0805mix0603" (id 2) (at 73.279 59.563 0)
+    (property "Footprint" "2004_cap:C0805mix0603" (id 2) (at 73.279 59.563 0)
       (effects (font (size 1.27 1.27)) hide)
     )
@@
       (effects (font (size 0.4 0.4)))
     )
-    (property "Footprint" "02_dyn_pcblib:hdr_2x1_1-1123723-2" (id 2) (at 50.8 72.39 0)
+    (property "Footprint" "2002_hdr:hdr_2x1_1-1123723-2" (id 2) (at 50.8 72.39 0)
       (effects (font (size 1.27 1.27)) hide)
     )
@@
       (effects (font (size 0.4 0.4)))
     )
-    (property "Footprint" "02_dyn_pcblib:hdr_2x1_1-1123723-2" (id 2) (at 20.32 72.39 0)
+    (property "Footprint" "2002_hdr:hdr_2x1_1-1123723-2" (id 2) (at 20.32 72.39 0)
       (effects (font (size 1.27 1.27)) hide)
     )
@@
       (effects (font (size 1.27 1.27)) (justify left))
     )
-    (property "Value" "nmos75v80a_IRFS3607TRLPBF" (id 1) (at 99.06 90.17 90)
+    (property "Value" "nmosTO263_75v80A" (id 1) (at 99.06 90.17 90)
       (effects (font (size 0.4 0.4)) (justify left))
     )
-    (property "Footprint" "02_dyn_pcblib:d2pak_TO263" (id 2) (at 74.93 71.12 0)
+    (property "Footprint" "2001_dyn_pcblib:d2pak_TO263" (id 2) (at 74.93 71.12 0)
       (effects (font (size 1.27 1.27) italic) (justify left) hide)
     )
@@
       (effects (font (size 0.5 0.5)))
     )
-    (property "Footprint" "02_dyn_pcblib:ptc_fuse_2920" (id 2) (at 81.28 74.93 0)
+    (property "Footprint" "2003_res:ptc_fuse_2920" (id 2) (at 81.28 74.93 0)
       (effects (font (size 1.27 1.27)) hide)
     )
@@
       (effects (font (size 0.5 0.5)))
     )
-    (property "Footprint" "02_dyn_pcblib:C0805mix0603" (id 2) (at 42.799 60.833 0)
+    (property "Footprint" "2004_cap:C0805mix0603" (id 2) (at 42.799 60.833 0)
       (effects (font (size 1.27 1.27)) hide)
     )
