File: kicad01_power_board_for_nuclear_team/untitled.kicad_sch (KiCad schematic)
At the start: 21 parts

Commit message: ix
Parts:
- C?: symbol 01dyn_lib:c0805_35v10u -> 1001_un:c0805_35v10u
- C?: symbol 01dyn_lib:c0603_10v3.3u -> 1001_un:c0603_10v3.3u
- C?: symbol 01dyn_lib:c0603_50v0.1u -> 1001_un:c0603_50v0.1u
- C? (x2): symbol 01dyn_lib:c0603_100v10n -> 1001_un:c0603_100v10n
- C?: symbol 01dyn_lib:c0603_50v1u -> 1001_un:c0603_50v1u
- D?: symbol 01dyn_lib:LED0603_red -> 1001_un:LED0603_red
- L?: symbol 01dyn_lib:L3.3uH_7.4x6.6mm_30mhO_9.5A -> 1001_un:L3.3uH_7.4x6.6mm_30mhO_9.5A
- R? (x4): symbol 01dyn_lib:R0603_100k -> 1001_un:R0603_100k
- R? (x5): symbol 01dyn_lib:R0603_10k -> 1001_un:R0603_10k
- R?: symbol 01dyn_lib:R1206_0.0 -> 1001_un:R1206_0.0
- R?: symbol 01dyn_lib:R0603_49.9k -> 1001_un:R0603_49.9k
- R?: symbol 01dyn_lib:R0603_DNP -> 1001_un:R0603_DNP
- U?: symbol 01dyn_lib:dcdc_lt8612x -> 1001_un:dcdc_lt8612x
Changed lines of the file:
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@@
     )
   )
-  (symbol (lib_id "01dyn_lib:LED0603_red") (at 86.36 55.88 180) (unit 1)
+  (symbol (lib_id "1001_un:LED0603_red") (at 86.36 55.88 180) (unit 1)
     (in_bom yes) (on_board yes)
     (property "Reference" "D?" (id 0) (at 90.17 54.61 0))
@@
     (pin "2")
   )
-  (symbol (lib_id "01dyn_lib:R0603_100k") (at 190.5 66.04 180) (unit 1)
+  (symbol (lib_id "1001_un:R0603_100k") (at 190.5 66.04 180) (unit 1)
     (in_bom yes) (on_board yes)
     (property "Reference" "R?" (id 0) (at 193.04 63.5 0)
@@
     (pin "2")
   )
-  (symbol (lib_id "01dyn_lib:R0603_10k") (at 74.93 82.55 90) (unit 1)
+  (symbol (lib_id "1001_un:R0603_10k") (at 74.93 82.55 90) (unit 1)
     (in_bom yes) (on_board yes)
     (property "Reference" "R?" (id 0) (at 77.47 82.55 0)
@@
     (pin "1")
   )
-  (symbol (lib_id "01dyn_lib:R0603_10k") (at 68.58 82.55 90) (unit 1)
+  (symbol (lib_id "1001_un:R0603_10k") (at 68.58 82.55 90) (unit 1)
     (in_bom yes) (on_board yes)
     (property "Reference" "R?" (id 0) (at 69.85 77.47 0)
@@
     (pin "2")
   )
-  (symbol (lib_id "01dyn_lib:R0603_10k") (at 172.72 66.04 180) (unit 1)
+  (symbol (lib_id "1001_un:R0603_10k") (at 172.72 66.04 180) (unit 1)
     (in_bom yes) (on_board yes)
     (property "Reference" "R?" (id 0) (at 172.72 63.5 0)
@@
     (pin "2")
   )
-  (symbol (lib_id "01dyn_lib:R1206_0.0") (at 170.18 35.56 180) (unit 1)
+  (symbol (lib_id "1001_un:R1206_0.0") (at 170.18 35.56 180) (unit 1)
     (in_bom yes) (on_board yes) (fields_autoplaced)
     (property "Reference" "R?" (id 0) (at 170.18 30.48 0)
@@
     (pin "2")
   )
-  (symbol (lib_id "01dyn_lib:R0603_100k") (at 88.9 72.39 90) (unit 1)
+  (symbol (lib_id "1001_un:R0603_100k") (at 88.9 72.39 90) (unit 1)
     (in_bom yes) (on_board yes)
     (property "Reference" "R?" (id 0) (at 87.63 69.85 0)
@@
     (pin "2")
   )
-  (symbol (lib_id "01dyn_lib:c0805_35v10u") (at 58.42 109.22 180) (unit 1)
+  (symbol (lib_id "1001_un:c0805_35v10u") (at 58.42 109.22 180) (unit 1)
     (in_bom yes) (on_board yes)
     (property "Reference" "C?" (id 0) (at 60.96 111.76 0))
@@
     (pin "1")
   )
-  (symbol (lib_id "01dyn_lib:R0603_100k") (at 64.77 81.28 90) (unit 1)
+  (symbol (lib_id "1001_un:R0603_100k") (at 64.77 81.28 90) (unit 1)
     (in_bom yes) (on_board yes)
     (property "Reference" "R?" (id 0) (at 63.5 83.82 0)
@@
     (pin "2")
   )
-  (symbol (lib_id "01dyn_lib:c0603_10v3.3u") (at 200.66 111.76 180) (unit 1)
+  (symbol (lib_id "1001_un:c0603_10v3.3u") (at 200.66 111.76 180) (unit 1)
     (in_bom yes) (on_board yes)
     (property "Reference" "C?" (id 0) (at 201.93 109.22 0)
@@
     (pin "2")
   )
-  (symbol (lib_id "01dyn_lib:c0603_50v0.1u") (at 139.7 93.98 90) (unit 1)
+  (symbol (lib_id "1001_un:c0603_50v0.1u") (at 139.7 93.98 90) (unit 1)
     (in_bom yes) (on_board yes)
     (property "Reference" "C?" (id 0) (at 144.78 92.71 90))
@@
     (pin "2")
   )
-  (symbol (lib_id "01dyn_lib:dcdc_lt8612x") (at 102.87 83.82 0) (unit 1)
+  (symbol (lib_id "1001_un:dcdc_lt8612x") (at 102.87 83.82 0) (unit 1)
     (in_bom yes) (on_board yes)
     (property "Reference" "U?" (id 0) (at 93.98 80.01 0)
@@
     (pin "9")
   )
-  (symbol (lib_id "01dyn_lib:R0603_10k") (at 106.68 55.88 180) (unit 1)
+  (symbol (lib_id "1001_un:R0603_10k") (at 106.68 55.88 180) (unit 1)
     (in_bom yes) (on_board yes)
     (property "Reference" "R?" (id 0) (at 111.76 54.61 0)
@@
     (pin "2")
   )
-  (symbol (lib_id "01dyn_lib:R0603_49.9k") (at 74.93 72.39 90) (unit 1)
+  (symbol (lib_id "1001_un:R0603_49.9k") (at 74.93 72.39 90) (unit 1)
     (in_bom yes) (on_board yes)
     (property "Reference" "R?" (id 0) (at 73.66 69.85 0)
@@
     (pin "2")
   )
-  (symbol (lib_id "01dyn_lib:L3.3uH_7.4x6.6mm_30mhO_9.5A") (at 181.61 99.06 0) (unit 1)
+  (symbol (lib_id "1001_un:L3.3uH_7.4x6.6mm_30mhO_9.5A") (at 181.61 99.06 0) (unit 1)
     (in_bom yes) (on_board yes)
     (property "Reference" "L?" (id 0) (at 181.61 95.25 0)
@@
     (pin "1")
   )
-  (symbol (lib_id "01dyn_lib:R0603_100k") (at 64.77 69.85 90) (unit 1)
+  (symbol (lib_id "1001_un:R0603_100k") (at 64.77 69.85 90) (unit 1)
     (in_bom yes) (on_board yes)
     (property "Reference" "R?" (id 0) (at 63.5 63.5 0)
@@
     (pin "2")
   )
-  (symbol (lib_id "01dyn_lib:R0603_10k") (at 160.02 66.04 180) (unit 1)
+  (symbol (lib_id "1001_un:R0603_10k") (at 160.02 66.04 180) (unit 1)
     (in_bom yes) (on_board yes)
     (property "Reference" "R?" (id 0) (at 162.56 63.5 0)
@@
     (pin "2")
   )
-  (symbol (lib_id "01dyn_lib:c0603_100v10n") (at 85.09 81.28 0) (unit 1)
+  (symbol (lib_id "1001_un:c0603_100v10n") (at 85.09 81.28 0) (unit 1)
     (in_bom yes) (on_board yes)
     (property "Reference" "C?" (id 0) (at 85.09 85.09 0)
@@
     (pin "2")
   )
-  (symbol (lib_id "01dyn_lib:R0603_DNP") (at 146.05 55.88 0) (unit 1)
+  (symbol (lib_id "1001_un:R0603_DNP") (at 146.05 55.88 0) (unit 1)
     (in_bom yes) (on_board yes)
     (property "Reference" "R?" (id 0) (at 151.13 54.61 0)
@@
     (pin "2")
   )
-  (symbol (lib_id "01dyn_lib:c0603_100v10n") (at 190.5 71.12 270) (unit 1)
+  (symbol (lib_id "1001_un:c0603_100v10n") (at 190.5 71.12 270) (unit 1)
     (in_bom yes) (on_board yes)
     (property "Reference" "C?" (id 0) (at 191.77 73.66 90)
@@
     (pin "2")
   )
-  (symbol (lib_id "01dyn_lib:c0603_50v1u") (at 128.27 67.31 180) (unit 1)
+  (symbol (lib_id "1001_un:c0603_50v1u") (at 128.27 67.31 180) (unit 1)
     (in_bom yes) (on_board yes)
     (property "Reference" "C?" (id 0) (at 130.81 69.85 0))

Commit message: x
Parts:
- C?: symbol 1001_un:c0805_35v10u -> 1003_cap:c0805_35v10u
- C?: symbol 1001_un:c0603_10v3.3u -> 1003_cap:c0603_10v3.3u
- C?: symbol 1001_un:c0603_50v0.1u -> 1003_cap:c0603_50v0.1u
- C? (x2): symbol 1001_un:c0603_100v10n -> 1003_cap:c0603_100v10n
- C?: symbol 1001_un:c0603_50v1u -> 1003_cap:c0603_50v1u
- D?: symbol 1001_un:LED0603_red -> 1004_led_mos:LED0603_red
- R? (x4): symbol 1001_un:R0603_100k -> 1002_res:R0603_100k
- R? (x5): symbol 1001_un:R0603_10k -> 1002_res:R0603_10k
- R?: symbol 1001_un:R1206_0.0 -> 1002_res:R1206_0.0
- R?: symbol 1001_un:R0603_49.9k -> 1002_res:R0603_49.9k
- R?: symbol 1001_un:R0603_DNP -> 1002_res:R0603_DNP
Changed lines of the file:
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@@
     )
   )
-  (symbol (lib_id "1001_un:LED0603_red") (at 86.36 55.88 180) (unit 1)
+  (symbol (lib_id "1004_led_mos:LED0603_red") (at 86.36 55.88 180) (unit 1)
     (in_bom yes) (on_board yes)
     (property "Reference" "D?" (id 0) (at 90.17 54.61 0))
@@
     (pin "2")
   )
-  (symbol (lib_id "1001_un:R0603_100k") (at 190.5 66.04 180) (unit 1)
+  (symbol (lib_id "1002_res:R0603_100k") (at 190.5 66.04 180) (unit 1)
     (in_bom yes) (on_board yes)
     (property "Reference" "R?" (id 0) (at 193.04 63.5 0)
@@
     (pin "2")
   )
-  (symbol (lib_id "1001_un:R0603_10k") (at 74.93 82.55 90) (unit 1)
+  (symbol (lib_id "1002_res:R0603_10k") (at 74.93 82.55 90) (unit 1)
     (in_bom yes) (on_board yes)
     (property "Reference" "R?" (id 0) (at 77.47 82.55 0)
@@
     (pin "1")
   )
-  (symbol (lib_id "1001_un:R0603_10k") (at 68.58 82.55 90) (unit 1)
+  (symbol (lib_id "1002_res:R0603_10k") (at 68.58 82.55 90) (unit 1)
     (in_bom yes) (on_board yes)
     (property "Reference" "R?" (id 0) (at 69.85 77.47 0)
@@
     (pin "2")
   )
-  (symbol (lib_id "1001_un:R0603_10k") (at 172.72 66.04 180) (unit 1)
+  (symbol (lib_id "1002_res:R0603_10k") (at 172.72 66.04 180) (unit 1)
     (in_bom yes) (on_board yes)
     (property "Reference" "R?" (id 0) (at 172.72 63.5 0)
@@
     (pin "2")
   )
-  (symbol (lib_id "1001_un:R1206_0.0") (at 170.18 35.56 180) (unit 1)
+  (symbol (lib_id "1002_res:R1206_0.0") (at 170.18 35.56 180) (unit 1)
     (in_bom yes) (on_board yes) (fields_autoplaced)
     (property "Reference" "R?" (id 0) (at 170.18 30.48 0)
@@
     (pin "2")
   )
-  (symbol (lib_id "1001_un:R0603_100k") (at 88.9 72.39 90) (unit 1)
+  (symbol (lib_id "1002_res:R0603_100k") (at 88.9 72.39 90) (unit 1)
     (in_bom yes) (on_board yes)
     (property "Reference" "R?" (id 0) (at 87.63 69.85 0)
@@
     (pin "2")
   )
-  (symbol (lib_id "1001_un:c0805_35v10u") (at 58.42 109.22 180) (unit 1)
+  (symbol (lib_id "1003_cap:c0805_35v10u") (at 58.42 109.22 180) (unit 1)
     (in_bom yes) (on_board yes)
     (property "Reference" "C?" (id 0) (at 60.96 111.76 0))
@@
     (pin "1")
   )
-  (symbol (lib_id "1001_un:R0603_100k") (at 64.77 81.28 90) (unit 1)
+  (symbol (lib_id "1002_res:R0603_100k") (at 64.77 81.28 90) (unit 1)
     (in_bom yes) (on_board yes)
     (property "Reference" "R?" (id 0) (at 63.5 83.82 0)
@@
     (pin "2")
   )
-  (symbol (lib_id "1001_un:c0603_10v3.3u") (at 200.66 111.76 180) (unit 1)
+  (symbol (lib_id "1003_cap:c0603_10v3.3u") (at 200.66 111.76 180) (unit 1)
     (in_bom yes) (on_board yes)
     (property "Reference" "C?" (id 0) (at 201.93 109.22 0)
@@
     (pin "2")
   )
-  (symbol (lib_id "1001_un:c0603_50v0.1u") (at 139.7 93.98 90) (unit 1)
+  (symbol (lib_id "1003_cap:c0603_50v0.1u") (at 139.7 93.98 90) (unit 1)
     (in_bom yes) (on_board yes)
     (property "Reference" "C?" (id 0) (at 144.78 92.71 90))
@@
     (pin "9")
   )
-  (symbol (lib_id "1001_un:R0603_10k") (at 106.68 55.88 180) (unit 1)
+  (symbol (lib_id "1002_res:R0603_10k") (at 106.68 55.88 180) (unit 1)
     (in_bom yes) (on_board yes)
     (property "Reference" "R?" (id 0) (at 111.76 54.61 0)
@@
     (pin "2")
   )
-  (symbol (lib_id "1001_un:R0603_49.9k") (at 74.93 72.39 90) (unit 1)
+  (symbol (lib_id "1002_res:R0603_49.9k") (at 74.93 72.39 90) (unit 1)
     (in_bom yes) (on_board yes)
     (property "Reference" "R?" (id 0) (at 73.66 69.85 0)
@@
     (pin "1")
   )
-  (symbol (lib_id "1001_un:R0603_100k") (at 64.77 69.85 90) (unit 1)
+  (symbol (lib_id "1002_res:R0603_100k") (at 64.77 69.85 90) (unit 1)
     (in_bom yes) (on_board yes)
     (property "Reference" "R?" (id 0) (at 63.5 63.5 0)
@@
     (pin "2")
   )
-  (symbol (lib_id "1001_un:R0603_10k") (at 160.02 66.04 180) (unit 1)
+  (symbol (lib_id "1002_res:R0603_10k") (at 160.02 66.04 180) (unit 1)
     (in_bom yes) (on_board yes)
     (property "Reference" "R?" (id 0) (at 162.56 63.5 0)
@@
     (pin "2")
   )
-  (symbol (lib_id "1001_un:c0603_100v10n") (at 85.09 81.28 0) (unit 1)
+  (symbol (lib_id "1003_cap:c0603_100v10n") (at 85.09 81.28 0) (unit 1)
     (in_bom yes) (on_board yes)
     (property "Reference" "C?" (id 0) (at 85.09 85.09 0)
@@
     (pin "2")
   )
-  (symbol (lib_id "1001_un:R0603_DNP") (at 146.05 55.88 0) (unit 1)
+  (symbol (lib_id "1002_res:R0603_DNP") (at 146.05 55.88 0) (unit 1)
     (in_bom yes) (on_board yes)
     (property "Reference" "R?" (id 0) (at 151.13 54.61 0)
@@
     (pin "2")
   )
-  (symbol (lib_id "1001_un:c0603_100v10n") (at 190.5 71.12 270) (unit 1)
+  (symbol (lib_id "1003_cap:c0603_100v10n") (at 190.5 71.12 270) (unit 1)
     (in_bom yes) (on_board yes)
     (property "Reference" "C?" (id 0) (at 191.77 73.66 90)
@@
     (pin "2")
   )
-  (symbol (lib_id "1001_un:c0603_50v1u") (at 128.27 67.31 180) (unit 1)
+  (symbol (lib_id "1003_cap:c0603_50v1u") (at 128.27 67.31 180) (unit 1)
     (in_bom yes) (on_board yes)
     (property "Reference" "C?" (id 0) (at 130.81 69.85 0))
