File: kicad01_power_board_for_nuclear_team/003_dcdc_18v.kicad_sch (KiCad schematic)
At the start: 21 parts, among them U301 dcdc_lt8612x

Commit message: ix
Parts:
- C321: symbol 01dyn_lib:c0805_35v10u -> 1001_un:c0805_35v10u
- C322, C365: symbol 01dyn_lib:c0603_100v10n -> 1001_un:c0603_100v10n
- C324: symbol 01dyn_lib:c0603_50v1u -> 1001_un:c0603_50v1u
- C325: symbol 01dyn_lib:c0603_50v0.1u -> 1001_un:c0603_50v0.1u
- C371: symbol 01dyn_lib:c0603_10v3.3u -> 1001_un:c0603_10v3.3u
- D351: symbol 01dyn_lib:LED0603_red -> 1001_un:LED0603_red
- L371: symbol 01dyn_lib:L3.3uH_7.4x6.6mm_30mhO_9.5A -> 1001_un:L3.3uH_7.4x6.6mm_30mhO_9.5A
- R311, R312, R323, R365: symbol 01dyn_lib:R0603_100k -> 1001_un:R0603_100k
- R313, R332, R351, R361, R362: symbol 01dyn_lib:R0603_10k -> 1001_un:R0603_10k
- R331: symbol 01dyn_lib:R0603_49.9k -> 1001_un:R0603_49.9k
- R352: symbol 01dyn_lib:R0603_DNP -> 1001_un:R0603_DNP
- R391: symbol 01dyn_lib:R1206_0.0 -> 1001_un:R1206_0.0
- U301: symbol 01dyn_lib:dcdc_lt8612x -> 1001_un:dcdc_lt8612x
Changed lines of the file:
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@@
     )
   )
-  (symbol (lib_id "01dyn_lib:LED0603_red") (at 86.36 55.88 180) (unit 1)
+  (symbol (lib_id "1001_un:LED0603_red") (at 86.36 55.88 180) (unit 1)
     (in_bom yes) (on_board yes)
     (property "Reference" "D351" (id 0) (at 90.17 54.61 0))
@@
     (pin "2")
   )
-  (symbol (lib_id "01dyn_lib:R0603_100k") (at 190.5 66.04 180) (unit 1)
+  (symbol (lib_id "1001_un:R0603_100k") (at 190.5 66.04 180) (unit 1)
     (in_bom yes) (on_board yes)
     (property "Reference" "R365" (id 0) (at 193.04 63.5 0)
@@
     (pin "2")
   )
-  (symbol (lib_id "01dyn_lib:R0603_10k") (at 74.93 82.55 90) (unit 1)
+  (symbol (lib_id "1001_un:R0603_10k") (at 74.93 82.55 90) (unit 1)
     (in_bom yes) (on_board yes)
     (property "Reference" "R332" (id 0) (at 77.47 82.55 0)
@@
     (pin "1")
   )
-  (symbol (lib_id "01dyn_lib:R0603_10k") (at 68.58 82.55 90) (unit 1)
+  (symbol (lib_id "1001_un:R0603_10k") (at 68.58 82.55 90) (unit 1)
     (in_bom yes) (on_board yes)
     (property "Reference" "R313" (id 0) (at 69.85 77.47 0)
@@
     (pin "2")
   )
-  (symbol (lib_id "01dyn_lib:R0603_10k") (at 172.72 66.04 180) (unit 1)
+  (symbol (lib_id "1001_un:R0603_10k") (at 172.72 66.04 180) (unit 1)
     (in_bom yes) (on_board yes)
     (property "Reference" "R362" (id 0) (at 172.72 63.5 0)
@@
     (pin "2")
   )
-  (symbol (lib_id "01dyn_lib:R1206_0.0") (at 170.18 35.56 180) (unit 1)
+  (symbol (lib_id "1001_un:R1206_0.0") (at 170.18 35.56 180) (unit 1)
     (in_bom yes) (on_board yes) (fields_autoplaced)
     (property "Reference" "R391" (id 0) (at 170.18 30.48 0)
@@
     (pin "2")
   )
-  (symbol (lib_id "01dyn_lib:R0603_100k") (at 88.9 72.39 90) (unit 1)
+  (symbol (lib_id "1001_un:R0603_100k") (at 88.9 72.39 90) (unit 1)
     (in_bom yes) (on_board yes)
     (property "Reference" "R323" (id 0) (at 87.63 69.85 0)
@@
     (pin "2")
   )
-  (symbol (lib_id "01dyn_lib:c0805_35v10u") (at 58.42 109.22 180) (unit 1)
+  (symbol (lib_id "1001_un:c0805_35v10u") (at 58.42 109.22 180) (unit 1)
     (in_bom yes) (on_board yes)
     (property "Reference" "C321" (id 0) (at 60.96 111.76 0))
@@
     (pin "1")
   )
-  (symbol (lib_id "01dyn_lib:R0603_100k") (at 64.77 81.28 90) (unit 1)
+  (symbol (lib_id "1001_un:R0603_100k") (at 64.77 81.28 90) (unit 1)
     (in_bom yes) (on_board yes)
     (property "Reference" "R312" (id 0) (at 63.5 83.82 0)
@@
     (pin "2")
   )
-  (symbol (lib_id "01dyn_lib:c0603_10v3.3u") (at 200.66 111.76 180) (unit 1)
+  (symbol (lib_id "1001_un:c0603_10v3.3u") (at 200.66 111.76 180) (unit 1)
     (in_bom yes) (on_board yes)
     (property "Reference" "C371" (id 0) (at 201.93 109.22 0)
@@
     (pin "2")
   )
-  (symbol (lib_id "01dyn_lib:c0603_50v0.1u") (at 139.7 93.98 90) (unit 1)
+  (symbol (lib_id "1001_un:c0603_50v0.1u") (at 139.7 93.98 90) (unit 1)
     (in_bom yes) (on_board yes)
     (property "Reference" "C325" (id 0) (at 144.78 92.71 90))
@@
     (pin "2")
   )
-  (symbol (lib_id "01dyn_lib:dcdc_lt8612x") (at 102.87 83.82 0) (unit 1)
+  (symbol (lib_id "1001_un:dcdc_lt8612x") (at 102.87 83.82 0) (unit 1)
     (in_bom yes) (on_board yes)
     (property "Reference" "U301" (id 0) (at 93.98 80.01 0)
@@
     (pin "9")
   )
-  (symbol (lib_id "01dyn_lib:R0603_10k") (at 106.68 55.88 180) (unit 1)
+  (symbol (lib_id "1001_un:R0603_10k") (at 106.68 55.88 180) (unit 1)
     (in_bom yes) (on_board yes)
     (property "Reference" "R351" (id 0) (at 111.76 54.61 0)
@@
     (pin "2")
   )
-  (symbol (lib_id "01dyn_lib:R0603_49.9k") (at 74.93 72.39 90) (unit 1)
+  (symbol (lib_id "1001_un:R0603_49.9k") (at 74.93 72.39 90) (unit 1)
     (in_bom yes) (on_board yes)
     (property "Reference" "R331" (id 0) (at 73.66 69.85 0)
@@
     (pin "2")
   )
-  (symbol (lib_id "01dyn_lib:L3.3uH_7.4x6.6mm_30mhO_9.5A") (at 181.61 99.06 0) (unit 1)
+  (symbol (lib_id "1001_un:L3.3uH_7.4x6.6mm_30mhO_9.5A") (at 181.61 99.06 0) (unit 1)
     (in_bom yes) (on_board yes)
     (property "Reference" "L371" (id 0) (at 181.61 95.25 0)
@@
     (pin "1")
   )
-  (symbol (lib_id "01dyn_lib:R0603_100k") (at 64.77 69.85 90) (unit 1)
+  (symbol (lib_id "1001_un:R0603_100k") (at 64.77 69.85 90) (unit 1)
     (in_bom yes) (on_board yes)
     (property "Reference" "R311" (id 0) (at 63.5 63.5 0)
@@
     (pin "2")
   )
-  (symbol (lib_id "01dyn_lib:R0603_10k") (at 160.02 66.04 180) (unit 1)
+  (symbol (lib_id "1001_un:R0603_10k") (at 160.02 66.04 180) (unit 1)
     (in_bom yes) (on_board yes)
     (property "Reference" "R361" (id 0) (at 162.56 63.5 0)
@@
     (pin "2")
   )
-  (symbol (lib_id "01dyn_lib:c0603_100v10n") (at 85.09 81.28 0) (unit 1)
+  (symbol (lib_id "1001_un:c0603_100v10n") (at 85.09 81.28 0) (unit 1)
     (in_bom yes) (on_board yes)
     (property "Reference" "C322" (id 0) (at 85.09 85.09 0)
@@
     (pin "2")
   )
-  (symbol (lib_id "01dyn_lib:R0603_DNP") (at 146.05 55.88 0) (unit 1)
+  (symbol (lib_id "1001_un:R0603_DNP") (at 146.05 55.88 0) (unit 1)
     (in_bom yes) (on_board yes)
     (property "Reference" "R352" (id 0) (at 151.13 54.61 0)
@@
     (pin "2")
   )
-  (symbol (lib_id "01dyn_lib:c0603_100v10n") (at 190.5 71.12 270) (unit 1)
+  (symbol (lib_id "1001_un:c0603_100v10n") (at 190.5 71.12 270) (unit 1)
     (in_bom yes) (on_board yes)
     (property "Reference" "C365" (id 0) (at 191.77 73.66 90)
@@
     (pin "2")
   )
-  (symbol (lib_id "01dyn_lib:c0603_50v1u") (at 128.27 67.31 180) (unit 1)
+  (symbol (lib_id "1001_un:c0603_50v1u") (at 128.27 67.31 180) (unit 1)
     (in_bom yes) (on_board yes)
     (property "Reference" "C324" (id 0) (at 130.81 69.85 0))

Commit message: x
Parts:
- C321: symbol 1001_un:c0805_35v10u -> 1003_cap:c0805_35v10u
- C322, C365: symbol 1001_un:c0603_100v10n -> 1003_cap:c0603_100v10n
- C324: symbol 1001_un:c0603_50v1u -> 1003_cap:c0603_50v1u
- C325: symbol 1001_un:c0603_50v0.1u -> 1003_cap:c0603_50v0.1u
- C371: symbol 1001_un:c0603_10v3.3u -> 1003_cap:c0603_10v3.3u
- D351: symbol 1001_un:LED0603_red -> 1004_led_mos:LED0603_red
- R311, R312, R323, R365: symbol 1001_un:R0603_100k -> 1002_res:R0603_100k
- R313, R332, R351, R361, R362: symbol 1001_un:R0603_10k -> 1002_res:R0603_10k
- R331: symbol 1001_un:R0603_49.9k -> 1002_res:R0603_49.9k
- R352: symbol 1001_un:R0603_DNP -> 1002_res:R0603_DNP
- R391: symbol 1001_un:R1206_0.0 -> 1002_res:R1206_0.0
Changed lines of the file:
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@@
     )
   )
-  (symbol (lib_id "1001_un:LED0603_red") (at 86.36 55.88 180) (unit 1)
+  (symbol (lib_id "1004_led_mos:LED0603_red") (at 86.36 55.88 180) (unit 1)
     (in_bom yes) (on_board yes)
     (property "Reference" "D351" (id 0) (at 90.17 54.61 0))
@@
     (pin "2")
   )
-  (symbol (lib_id "1001_un:R0603_100k") (at 190.5 66.04 180) (unit 1)
+  (symbol (lib_id "1002_res:R0603_100k") (at 190.5 66.04 180) (unit 1)
     (in_bom yes) (on_board yes)
     (property "Reference" "R365" (id 0) (at 193.04 63.5 0)
@@
     (pin "2")
   )
-  (symbol (lib_id "1001_un:R0603_10k") (at 74.93 82.55 90) (unit 1)
+  (symbol (lib_id "1002_res:R0603_10k") (at 74.93 82.55 90) (unit 1)
     (in_bom yes) (on_board yes)
     (property "Reference" "R332" (id 0) (at 77.47 82.55 0)
@@
     (pin "1")
   )
-  (symbol (lib_id "1001_un:R0603_10k") (at 68.58 82.55 90) (unit 1)
+  (symbol (lib_id "1002_res:R0603_10k") (at 68.58 82.55 90) (unit 1)
     (in_bom yes) (on_board yes)
     (property "Reference" "R313" (id 0) (at 69.85 77.47 0)
@@
     (pin "2")
   )
-  (symbol (lib_id "1001_un:R0603_10k") (at 172.72 66.04 180) (unit 1)
+  (symbol (lib_id "1002_res:R0603_10k") (at 172.72 66.04 180) (unit 1)
     (in_bom yes) (on_board yes)
     (property "Reference" "R362" (id 0) (at 172.72 63.5 0)
@@
     (pin "2")
   )
-  (symbol (lib_id "1001_un:R1206_0.0") (at 170.18 35.56 180) (unit 1)
+  (symbol (lib_id "1002_res:R1206_0.0") (at 170.18 35.56 180) (unit 1)
     (in_bom yes) (on_board yes) (fields_autoplaced)
     (property "Reference" "R391" (id 0) (at 170.18 30.48 0)
@@
     (pin "2")
   )
-  (symbol (lib_id "1001_un:R0603_100k") (at 88.9 72.39 90) (unit 1)
+  (symbol (lib_id "1002_res:R0603_100k") (at 88.9 72.39 90) (unit 1)
     (in_bom yes) (on_board yes)
     (property "Reference" "R323" (id 0) (at 87.63 69.85 0)
@@
     (pin "2")
   )
-  (symbol (lib_id "1001_un:c0805_35v10u") (at 58.42 109.22 180) (unit 1)
+  (symbol (lib_id "1003_cap:c0805_35v10u") (at 58.42 109.22 180) (unit 1)
     (in_bom yes) (on_board yes)
     (property "Reference" "C321" (id 0) (at 60.96 111.76 0))
@@
     (pin "1")
   )
-  (symbol (lib_id "1001_un:R0603_100k") (at 64.77 81.28 90) (unit 1)
+  (symbol (lib_id "1002_res:R0603_100k") (at 64.77 81.28 90) (unit 1)
     (in_bom yes) (on_board yes)
     (property "Reference" "R312" (id 0) (at 63.5 83.82 0)
@@
     (pin "2")
   )
-  (symbol (lib_id "1001_un:c0603_10v3.3u") (at 200.66 111.76 180) (unit 1)
+  (symbol (lib_id "1003_cap:c0603_10v3.3u") (at 200.66 111.76 180) (unit 1)
     (in_bom yes) (on_board yes)
     (property "Reference" "C371" (id 0) (at 201.93 109.22 0)
@@
     (pin "2")
   )
-  (symbol (lib_id "1001_un:c0603_50v0.1u") (at 139.7 93.98 90) (unit 1)
+  (symbol (lib_id "1003_cap:c0603_50v0.1u") (at 139.7 93.98 90) (unit 1)
     (in_bom yes) (on_board yes)
     (property "Reference" "C325" (id 0) (at 144.78 92.71 90))
@@
     (pin "9")
   )
-  (symbol (lib_id "1001_un:R0603_10k") (at 106.68 55.88 180) (unit 1)
+  (symbol (lib_id "1002_res:R0603_10k") (at 106.68 55.88 180) (unit 1)
     (in_bom yes) (on_board yes)
     (property "Reference" "R351" (id 0) (at 111.76 54.61 0)
@@
     (pin "2")
   )
-  (symbol (lib_id "1001_un:R0603_49.9k") (at 74.93 72.39 90) (unit 1)
+  (symbol (lib_id "1002_res:R0603_49.9k") (at 74.93 72.39 90) (unit 1)
     (in_bom yes) (on_board yes)
     (property "Reference" "R331" (id 0) (at 73.66 69.85 0)
@@
     (pin "1")
   )
-  (symbol (lib_id "1001_un:R0603_100k") (at 64.77 69.85 90) (unit 1)
+  (symbol (lib_id "1002_res:R0603_100k") (at 64.77 69.85 90) (unit 1)
     (in_bom yes) (on_board yes)
     (property "Reference" "R311" (id 0) (at 63.5 63.5 0)
@@
     (pin "2")
   )
-  (symbol (lib_id "1001_un:R0603_10k") (at 160.02 66.04 180) (unit 1)
+  (symbol (lib_id "1002_res:R0603_10k") (at 160.02 66.04 180) (unit 1)
     (in_bom yes) (on_board yes)
     (property "Reference" "R361" (id 0) (at 162.56 63.5 0)
@@
     (pin "2")
   )
-  (symbol (lib_id "1001_un:c0603_100v10n") (at 85.09 81.28 0) (unit 1)
+  (symbol (lib_id "1003_cap:c0603_100v10n") (at 85.09 81.28 0) (unit 1)
     (in_bom yes) (on_board yes)
     (property "Reference" "C322" (id 0) (at 85.09 85.09 0)
@@
     (pin "2")
   )
-  (symbol (lib_id "1001_un:R0603_DNP") (at 146.05 55.88 0) (unit 1)
+  (symbol (lib_id "1002_res:R0603_DNP") (at 146.05 55.88 0) (unit 1)
     (in_bom yes) (on_board yes)
     (property "Reference" "R352" (id 0) (at 151.13 54.61 0)
@@
     (pin "2")
   )
-  (symbol (lib_id "1001_un:c0603_100v10n") (at 190.5 71.12 270) (unit 1)
+  (symbol (lib_id "1003_cap:c0603_100v10n") (at 190.5 71.12 270) (unit 1)
     (in_bom yes) (on_board yes)
     (property "Reference" "C365" (id 0) (at 191.77 73.66 90)
@@
     (pin "2")
   )
-  (symbol (lib_id "1001_un:c0603_50v1u") (at 128.27 67.31 180) (unit 1)
+  (symbol (lib_id "1003_cap:c0603_50v1u") (at 128.27 67.31 180) (unit 1)
     (in_bom yes) (on_board yes)
     (property "Reference" "C324" (id 0) (at 130.81 69.85 0))

Commit message: x
Parts:
- L371: symbol 1001_un:L3.3uH_7.4x6.6mm_30mhO_9.5A -> 1006_Inductance:L3.3uH_7.4x6.6mm_30mhO_9.5A
- U301: symbol 1001_un:dcdc_lt8612x -> 1009_ic:dcdc_lt8612x
Changed lines of the file:
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@@
     (pin "2")
   )
-  (symbol (lib_id "1001_un:dcdc_lt8612x") (at 102.87 83.82 0) (unit 1)
+  (symbol (lib_id "1009_ic:dcdc_lt8612x") (at 102.87 83.82 0) (unit 1)
     (in_bom yes) (on_board yes)
     (property "Reference" "U301" (id 0) (at 93.98 80.01 0)
@@
     (pin "2")
   )
-  (symbol (lib_id "1001_un:L3.3uH_7.4x6.6mm_30mhO_9.5A") (at 181.61 99.06 0) (unit 1)
+  (symbol (lib_id "1006_Inductance:L3.3uH_7.4x6.6mm_30mhO_9.5A") (at 181.61 99.06 0) (unit 1)
     (in_bom yes) (on_board yes)
     (property "Reference" "L371" (id 0) (at 181.61 95.25 0)

Commit message: x
Parts:
- C321: footprint 02_dyn_pcblib:C0805mix0603 -> 2004_cap:C0805mix0603
- D351: footprint 02_dyn_pcblib:LED0603 -> 2007_LED:LED0603
- L371: footprint 02_dyn_pcblib:L7.1x6.6mm -> 2005_inductance:L7.1x6.6mm
- R391: footprint 02_dyn_pcblib:R1206mix0603 -> 2003_res:R1206mix0603
- U301: footprint 02_dyn_pcblib:QFN-28-1EP_3x6mm_P0.5mm_EP1.7x4.75mmX -> 2006_qfn:QFN-28-1EP_3x6mm_P0.5mm_EP1.7x4.75mmX
Changed lines of the file:
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@@
       (effects (font (size 0.5 0.5)) (justify left))
     )
-    (property "Footprint" "02_dyn_pcblib:LED0603" (id 2) (at 86.36 64.77 0)
+    (property "Footprint" "2007_LED:LED0603" (id 2) (at 86.36 64.77 0)
       (effects (font (size 1.27 1.27)) hide)
     )
@@
       (effects (font (size 0.5 0.5)))
     )
-    (property "Footprint" "02_dyn_pcblib:R1206mix0603" (id 2) (at 170.18 46.99 0)
+    (property "Footprint" "2003_res:R1206mix0603" (id 2) (at 170.18 46.99 0)
       (effects (font (size 1.27 1.27)) hide)
     )
@@
       (effects (font (size 0.5 0.5)))
     )
-    (property "Footprint" "02_dyn_pcblib:C0805mix0603" (id 2) (at 57.531 122.047 0)
+    (property "Footprint" "2004_cap:C0805mix0603" (id 2) (at 57.531 122.047 0)
       (effects (font (size 1.27 1.27)) hide)
     )
@@
     )
     (property "Value" "dcdc_lt8612x" (id 1) (at 106.68 97.79 0))
-    (property "Footprint" "02_dyn_pcblib:QFN-28-1EP_3x6mm_P0.5mm_EP1.7x4.75mmX" (id 2) (at 109.22 55.88 0)
+    (property "Footprint" "2006_qfn:QFN-28-1EP_3x6mm_P0.5mm_EP1.7x4.75mmX" (id 2) (at 109.22 55.88 0)
       (effects (font (size 1.27 1.27)) hide)
     )
@@
       (effects (font (size 0.5 0.5)) (justify left))
     )
-    (property "Footprint" "02_dyn_pcblib:L7.1x6.6mm" (id 2) (at 180.34 88.9 0)
-      (effects (font (size 1.27 1.27)) hide)
-    )
+    (property "Footprint" "2005_inductance:L7.1x6.6mm" (id 2) (at 180.34 88.9 0)
+      (effects (font (size 1.27 1.27)) hide)
+    )
