File: kicad01_power_board_for_nuclear_team/004_dcdc_18v.kicad_sch (KiCad schematic)
At the start: 21 parts, among them U2 dcdc_lt8612x

Commit message: ix
Parts:
- C10: symbol 01dyn_lib:c0603_50v0.1u -> 1001_un:c0603_50v0.1u
- C11, C8: symbol 01dyn_lib:c0603_100v10n -> 1001_un:c0603_100v10n
- C12: symbol 01dyn_lib:c0603_10v3.3u -> 1001_un:c0603_10v3.3u
- C7: symbol 01dyn_lib:c0805_35v10u -> 1001_un:c0805_35v10u
- C9: symbol 01dyn_lib:c0603_50v1u -> 1001_un:c0603_50v1u
- D2: symbol 01dyn_lib:LED0603_red -> 1001_un:LED0603_red
- L2: symbol 01dyn_lib:L3.3uH_7.4x6.6mm_30mhO_9.5A -> 1001_un:L3.3uH_7.4x6.6mm_30mhO_9.5A
- R13, R14, R18, R24: symbol 01dyn_lib:R0603_100k -> 1001_un:R0603_100k
- R15, R17, R19, R21, R23: symbol 01dyn_lib:R0603_10k -> 1001_un:R0603_10k
- R16: symbol 01dyn_lib:R0603_49.9k -> 1001_un:R0603_49.9k
- R20: symbol 01dyn_lib:R0603_DNP -> 1001_un:R0603_DNP
- R22: symbol 01dyn_lib:R1206_0.0 -> 1001_un:R1206_0.0
- U2: symbol 01dyn_lib:dcdc_lt8612x -> 1001_un:dcdc_lt8612x
Changed lines of the file:
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@@
     )
   )
-  (symbol (lib_id "01dyn_lib:c0603_50v1u") (at 135.89 76.2 180) (unit 1)
+  (symbol (lib_id "1001_un:c0603_50v1u") (at 135.89 76.2 180) (unit 1)
     (in_bom yes) (on_board yes)
     (property "Reference" "C9" (id 0) (at 138.43 78.74 0))
@@
     (pin "1")
   )
-  (symbol (lib_id "01dyn_lib:c0603_10v3.3u") (at 208.28 120.65 180) (unit 1)
+  (symbol (lib_id "1001_un:c0603_10v3.3u") (at 208.28 120.65 180) (unit 1)
     (in_bom yes) (on_board yes)
     (property "Reference" "C12" (id 0) (at 209.55 118.11 0)
@@
     (pin "2")
   )
-  (symbol (lib_id "01dyn_lib:R0603_10k") (at 114.3 64.77 180) (unit 1)
+  (symbol (lib_id "1001_un:R0603_10k") (at 114.3 64.77 180) (unit 1)
     (in_bom yes) (on_board yes)
     (property "Reference" "R19" (id 0) (at 119.38 63.5 0)
@@
     (pin "2")
   )
-  (symbol (lib_id "01dyn_lib:R0603_100k") (at 72.39 90.17 90) (unit 1)
+  (symbol (lib_id "1001_un:R0603_100k") (at 72.39 90.17 90) (unit 1)
     (in_bom yes) (on_board yes)
     (property "Reference" "R14" (id 0) (at 71.12 92.71 0)
@@
     (pin "2")
   )
-  (symbol (lib_id "01dyn_lib:c0805_35v10u") (at 66.04 118.11 180) (unit 1)
+  (symbol (lib_id "1001_un:c0805_35v10u") (at 66.04 118.11 180) (unit 1)
     (in_bom yes) (on_board yes)
     (property "Reference" "C7" (id 0) (at 68.58 120.65 0))
@@
     (pin "1")
   )
-  (symbol (lib_id "01dyn_lib:R1206_0.0") (at 177.8 44.45 180) (unit 1)
+  (symbol (lib_id "1001_un:R1206_0.0") (at 177.8 44.45 180) (unit 1)
     (in_bom yes) (on_board yes) (fields_autoplaced)
     (property "Reference" "R22" (id 0) (at 177.8 39.37 0)
@@
     (pin "2")
   )
-  (symbol (lib_id "01dyn_lib:R0603_100k") (at 96.52 81.28 90) (unit 1)
+  (symbol (lib_id "1001_un:R0603_100k") (at 96.52 81.28 90) (unit 1)
     (in_bom yes) (on_board yes)
     (property "Reference" "R18" (id 0) (at 95.25 78.74 0)
@@
     (pin "2")
   )
-  (symbol (lib_id "01dyn_lib:R0603_10k") (at 82.55 91.44 90) (unit 1)
+  (symbol (lib_id "1001_un:R0603_10k") (at 82.55 91.44 90) (unit 1)
     (in_bom yes) (on_board yes)
     (property "Reference" "R17" (id 0) (at 85.09 91.44 0)
@@
     (pin "2")
   )
-  (symbol (lib_id "01dyn_lib:R0603_49.9k") (at 82.55 81.28 90) (unit 1)
+  (symbol (lib_id "1001_un:R0603_49.9k") (at 82.55 81.28 90) (unit 1)
     (in_bom yes) (on_board yes)
     (property "Reference" "R16" (id 0) (at 81.28 78.74 0)
@@
     (pin "2")
   )
-  (symbol (lib_id "01dyn_lib:R0603_100k") (at 72.39 78.74 90) (unit 1)
+  (symbol (lib_id "1001_un:R0603_100k") (at 72.39 78.74 90) (unit 1)
     (in_bom yes) (on_board yes)
     (property "Reference" "R13" (id 0) (at 71.12 72.39 0)
@@
     (pin "2")
   )
-  (symbol (lib_id "01dyn_lib:dcdc_lt8612x") (at 110.49 92.71 0) (unit 1)
+  (symbol (lib_id "1001_un:dcdc_lt8612x") (at 110.49 92.71 0) (unit 1)
     (in_bom yes) (on_board yes)
     (property "Reference" "U2" (id 0) (at 101.6 88.9 0)
@@
     (pin "9")
   )
-  (symbol (lib_id "01dyn_lib:c0603_100v10n") (at 92.71 90.17 0) (unit 1)
+  (symbol (lib_id "1001_un:c0603_100v10n") (at 92.71 90.17 0) (unit 1)
     (in_bom yes) (on_board yes)
     (property "Reference" "C8" (id 0) (at 92.71 93.98 0)
@@
     (pin "2")
   )
-  (symbol (lib_id "01dyn_lib:R0603_10k") (at 167.64 74.93 180) (unit 1)
+  (symbol (lib_id "1001_un:R0603_10k") (at 167.64 74.93 180) (unit 1)
     (in_bom yes) (on_board yes)
     (property "Reference" "R21" (id 0) (at 170.18 72.39 0)
@@
     (pin "2")
   )
-  (symbol (lib_id "01dyn_lib:R0603_10k") (at 180.34 74.93 180) (unit 1)
+  (symbol (lib_id "1001_un:R0603_10k") (at 180.34 74.93 180) (unit 1)
     (in_bom yes) (on_board yes)
     (property "Reference" "R23" (id 0) (at 180.34 72.39 0)
@@
     (pin "2")
   )
-  (symbol (lib_id "01dyn_lib:LED0603_red") (at 93.98 64.77 180) (unit 1)
+  (symbol (lib_id "1001_un:LED0603_red") (at 93.98 64.77 180) (unit 1)
     (in_bom yes) (on_board yes)
     (property "Reference" "D2" (id 0) (at 97.79 63.5 0))
@@
     (pin "1")
   )
-  (symbol (lib_id "01dyn_lib:R0603_10k") (at 76.2 91.44 90) (unit 1)
+  (symbol (lib_id "1001_un:R0603_10k") (at 76.2 91.44 90) (unit 1)
     (in_bom yes) (on_board yes)
     (property "Reference" "R15" (id 0) (at 77.47 86.36 0)
@@
     (pin "2")
   )
-  (symbol (lib_id "01dyn_lib:c0603_100v10n") (at 198.12 80.01 270) (unit 1)
+  (symbol (lib_id "1001_un:c0603_100v10n") (at 198.12 80.01 270) (unit 1)
     (in_bom yes) (on_board yes)
     (property "Reference" "C11" (id 0) (at 199.39 82.55 90)
@@
     (pin "2")
   )
-  (symbol (lib_id "01dyn_lib:R0603_DNP") (at 153.67 64.77 0) (unit 1)
+  (symbol (lib_id "1001_un:R0603_DNP") (at 153.67 64.77 0) (unit 1)
     (in_bom yes) (on_board yes)
     (property "Reference" "R20" (id 0) (at 158.75 63.5 0)
@@
     (pin "2")
   )
-  (symbol (lib_id "01dyn_lib:L3.3uH_7.4x6.6mm_30mhO_9.5A") (at 189.23 107.95 0) (unit 1)
+  (symbol (lib_id "1001_un:L3.3uH_7.4x6.6mm_30mhO_9.5A") (at 189.23 107.95 0) (unit 1)
     (in_bom yes) (on_board yes)
     (property "Reference" "L2" (id 0) (at 189.23 104.14 0)
@@
     (pin "2")
   )
-  (symbol (lib_id "01dyn_lib:R0603_100k") (at 198.12 74.93 180) (unit 1)
+  (symbol (lib_id "1001_un:R0603_100k") (at 198.12 74.93 180) (unit 1)
     (in_bom yes) (on_board yes)
     (property "Reference" "R24" (id 0) (at 200.66 72.39 0)
@@
     (pin "1")
   )
-  (symbol (lib_id "01dyn_lib:c0603_50v0.1u") (at 147.32 102.87 90) (unit 1)
+  (symbol (lib_id "1001_un:c0603_50v0.1u") (at 147.32 102.87 90) (unit 1)
     (in_bom yes) (on_board yes)
     (property "Reference" "C10" (id 0) (at 152.4 101.6 90))

Commit message: x
Parts:
- C10: symbol 1001_un:c0603_50v0.1u -> 1003_cap:c0603_50v0.1u
- C11, C8: symbol 1001_un:c0603_100v10n -> 1003_cap:c0603_100v10n
- C12: symbol 1001_un:c0603_10v3.3u -> 1003_cap:c0603_10v3.3u
- C7: symbol 1001_un:c0805_35v10u -> 1003_cap:c0805_35v10u
- C9: symbol 1001_un:c0603_50v1u -> 1003_cap:c0603_50v1u
- D2: symbol 1001_un:LED0603_red -> 1004_led_mos:LED0603_red
- R13, R14, R18, R24: symbol 1001_un:R0603_100k -> 1002_res:R0603_100k
- R15, R17, R19, R21, R23: symbol 1001_un:R0603_10k -> 1002_res:R0603_10k
- R16: symbol 1001_un:R0603_49.9k -> 1002_res:R0603_49.9k
- R20: symbol 1001_un:R0603_DNP -> 1002_res:R0603_DNP
- R22: symbol 1001_un:R1206_0.0 -> 1002_res:R1206_0.0
Changed lines of the file:
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@@
     )
   )
-  (symbol (lib_id "1001_un:c0603_50v1u") (at 135.89 76.2 180) (unit 1)
+  (symbol (lib_id "1003_cap:c0603_50v1u") (at 135.89 76.2 180) (unit 1)
     (in_bom yes) (on_board yes)
     (property "Reference" "C9" (id 0) (at 138.43 78.74 0))
@@
     (pin "1")
   )
-  (symbol (lib_id "1001_un:c0603_10v3.3u") (at 208.28 120.65 180) (unit 1)
+  (symbol (lib_id "1003_cap:c0603_10v3.3u") (at 208.28 120.65 180) (unit 1)
     (in_bom yes) (on_board yes)
     (property "Reference" "C12" (id 0) (at 209.55 118.11 0)
@@
     (pin "2")
   )
-  (symbol (lib_id "1001_un:R0603_10k") (at 114.3 64.77 180) (unit 1)
+  (symbol (lib_id "1002_res:R0603_10k") (at 114.3 64.77 180) (unit 1)
     (in_bom yes) (on_board yes)
     (property "Reference" "R19" (id 0) (at 119.38 63.5 0)
@@
     (pin "2")
   )
-  (symbol (lib_id "1001_un:R0603_100k") (at 72.39 90.17 90) (unit 1)
+  (symbol (lib_id "1002_res:R0603_100k") (at 72.39 90.17 90) (unit 1)
     (in_bom yes) (on_board yes)
     (property "Reference" "R14" (id 0) (at 71.12 92.71 0)
@@
     (pin "2")
   )
-  (symbol (lib_id "1001_un:c0805_35v10u") (at 66.04 118.11 180) (unit 1)
+  (symbol (lib_id "1003_cap:c0805_35v10u") (at 66.04 118.11 180) (unit 1)
     (in_bom yes) (on_board yes)
     (property "Reference" "C7" (id 0) (at 68.58 120.65 0))
@@
     (pin "1")
   )
-  (symbol (lib_id "1001_un:R1206_0.0") (at 177.8 44.45 180) (unit 1)
+  (symbol (lib_id "1002_res:R1206_0.0") (at 177.8 44.45 180) (unit 1)
     (in_bom yes) (on_board yes) (fields_autoplaced)
     (property "Reference" "R22" (id 0) (at 177.8 39.37 0)
@@
     (pin "2")
   )
-  (symbol (lib_id "1001_un:R0603_100k") (at 96.52 81.28 90) (unit 1)
+  (symbol (lib_id "1002_res:R0603_100k") (at 96.52 81.28 90) (unit 1)
     (in_bom yes) (on_board yes)
     (property "Reference" "R18" (id 0) (at 95.25 78.74 0)
@@
     (pin "2")
   )
-  (symbol (lib_id "1001_un:R0603_10k") (at 82.55 91.44 90) (unit 1)
+  (symbol (lib_id "1002_res:R0603_10k") (at 82.55 91.44 90) (unit 1)
     (in_bom yes) (on_board yes)
     (property "Reference" "R17" (id 0) (at 85.09 91.44 0)
@@
     (pin "2")
   )
-  (symbol (lib_id "1001_un:R0603_49.9k") (at 82.55 81.28 90) (unit 1)
+  (symbol (lib_id "1002_res:R0603_49.9k") (at 82.55 81.28 90) (unit 1)
     (in_bom yes) (on_board yes)
     (property "Reference" "R16" (id 0) (at 81.28 78.74 0)
@@
     (pin "2")
   )
-  (symbol (lib_id "1001_un:R0603_100k") (at 72.39 78.74 90) (unit 1)
+  (symbol (lib_id "1002_res:R0603_100k") (at 72.39 78.74 90) (unit 1)
     (in_bom yes) (on_board yes)
     (property "Reference" "R13" (id 0) (at 71.12 72.39 0)
@@
     (pin "9")
   )
-  (symbol (lib_id "1001_un:c0603_100v10n") (at 92.71 90.17 0) (unit 1)
+  (symbol (lib_id "1003_cap:c0603_100v10n") (at 92.71 90.17 0) (unit 1)
     (in_bom yes) (on_board yes)
     (property "Reference" "C8" (id 0) (at 92.71 93.98 0)
@@
     (pin "2")
   )
-  (symbol (lib_id "1001_un:R0603_10k") (at 167.64 74.93 180) (unit 1)
+  (symbol (lib_id "1002_res:R0603_10k") (at 167.64 74.93 180) (unit 1)
     (in_bom yes) (on_board yes)
     (property "Reference" "R21" (id 0) (at 170.18 72.39 0)
@@
     (pin "2")
   )
-  (symbol (lib_id "1001_un:R0603_10k") (at 180.34 74.93 180) (unit 1)
+  (symbol (lib_id "1002_res:R0603_10k") (at 180.34 74.93 180) (unit 1)
     (in_bom yes) (on_board yes)
     (property "Reference" "R23" (id 0) (at 180.34 72.39 0)
@@
     (pin "2")
   )
-  (symbol (lib_id "1001_un:LED0603_red") (at 93.98 64.77 180) (unit 1)
+  (symbol (lib_id "1004_led_mos:LED0603_red") (at 93.98 64.77 180) (unit 1)
     (in_bom yes) (on_board yes)
     (property "Reference" "D2" (id 0) (at 97.79 63.5 0))
@@
     (pin "1")
   )
-  (symbol (lib_id "1001_un:R0603_10k") (at 76.2 91.44 90) (unit 1)
+  (symbol (lib_id "1002_res:R0603_10k") (at 76.2 91.44 90) (unit 1)
     (in_bom yes) (on_board yes)
     (property "Reference" "R15" (id 0) (at 77.47 86.36 0)
@@
     (pin "2")
   )
-  (symbol (lib_id "1001_un:c0603_100v10n") (at 198.12 80.01 270) (unit 1)
+  (symbol (lib_id "1003_cap:c0603_100v10n") (at 198.12 80.01 270) (unit 1)
     (in_bom yes) (on_board yes)
     (property "Reference" "C11" (id 0) (at 199.39 82.55 90)
@@
     (pin "2")
   )
-  (symbol (lib_id "1001_un:R0603_DNP") (at 153.67 64.77 0) (unit 1)
+  (symbol (lib_id "1002_res:R0603_DNP") (at 153.67 64.77 0) (unit 1)
     (in_bom yes) (on_board yes)
     (property "Reference" "R20" (id 0) (at 158.75 63.5 0)
@@
     (pin "2")
   )
-  (symbol (lib_id "1001_un:R0603_100k") (at 198.12 74.93 180) (unit 1)
+  (symbol (lib_id "1002_res:R0603_100k") (at 198.12 74.93 180) (unit 1)
     (in_bom yes) (on_board yes)
     (property "Reference" "R24" (id 0) (at 200.66 72.39 0)
@@
     (pin "1")
   )
-  (symbol (lib_id "1001_un:c0603_50v0.1u") (at 147.32 102.87 90) (unit 1)
+  (symbol (lib_id "1003_cap:c0603_50v0.1u") (at 147.32 102.87 90) (unit 1)
     (in_bom yes) (on_board yes)
     (property "Reference" "C10" (id 0) (at 152.4 101.6 90))

Commit message: x
Parts:
- L2: symbol 1001_un:L3.3uH_7.4x6.6mm_30mhO_9.5A -> 1006_Inductance:L3.3uH_7.4x6.6mm_30mhO_9.5A
- U2: symbol 1001_un:dcdc_lt8612x -> 1009_ic:dcdc_lt8612x
Changed lines of the file:
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@@
     (pin "2")
   )
-  (symbol (lib_id "1001_un:dcdc_lt8612x") (at 110.49 92.71 0) (unit 1)
+  (symbol (lib_id "1009_ic:dcdc_lt8612x") (at 110.49 92.71 0) (unit 1)
     (in_bom yes) (on_board yes)
     (property "Reference" "U2" (id 0) (at 101.6 88.9 0)
@@
     (pin "2")
   )
-  (symbol (lib_id "1001_un:L3.3uH_7.4x6.6mm_30mhO_9.5A") (at 189.23 107.95 0) (unit 1)
+  (symbol (lib_id "1006_Inductance:L3.3uH_7.4x6.6mm_30mhO_9.5A") (at 189.23 107.95 0) (unit 1)
     (in_bom yes) (on_board yes)
     (property "Reference" "L2" (id 0) (at 189.23 104.14 0)

Commit message: x
Parts:
- C7: footprint 02_dyn_pcblib:C0805mix0603 -> 2004_cap:C0805mix0603
- D2: footprint 02_dyn_pcblib:LED0603 -> 2007_LED:LED0603
- L2: footprint 02_dyn_pcblib:L7.1x6.6mm -> 2005_inductance:L7.1x6.6mm
- R22: footprint 02_dyn_pcblib:R1206mix0603 -> 2003_res:R1206mix0603
- U2: footprint 02_dyn_pcblib:QFN-28-1EP_3x6mm_P0.5mm_EP1.7x4.75mmX -> 2006_qfn:QFN-28-1EP_3x6mm_P0.5mm_EP1.7x4.75mmX
Changed lines of the file:
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@@
       (effects (font (size 0.5 0.5)))
     )
-    (property "Footprint" "02_dyn_pcblib:C0805mix0603" (id 2) (at 65.151 130.937 0)
+    (property "Footprint" "2004_cap:C0805mix0603" (id 2) (at 65.151 130.937 0)
       (effects (font (size 1.27 1.27)) hide)
     )
@@
       (effects (font (size 0.5 0.5)))
     )
-    (property "Footprint" "02_dyn_pcblib:R1206mix0603" (id 2) (at 177.8 55.88 0)
+    (property "Footprint" "2003_res:R1206mix0603" (id 2) (at 177.8 55.88 0)
       (effects (font (size 1.27 1.27)) hide)
     )
@@
     )
     (property "Value" "dcdc_lt8612x" (id 1) (at 114.3 106.68 0))
-    (property "Footprint" "02_dyn_pcblib:QFN-28-1EP_3x6mm_P0.5mm_EP1.7x4.75mmX" (id 2) (at 116.84 64.77 0)
+    (property "Footprint" "2006_qfn:QFN-28-1EP_3x6mm_P0.5mm_EP1.7x4.75mmX" (id 2) (at 116.84 64.77 0)
       (effects (font (size 1.27 1.27)) hide)
     )
@@
       (effects (font (size 0.5 0.5)) (justify left))
     )
-    (property "Footprint" "02_dyn_pcblib:LED0603" (id 2) (at 93.98 73.66 0)
+    (property "Footprint" "2007_LED:LED0603" (id 2) (at 93.98 73.66 0)
       (effects (font (size 1.27 1.27)) hide)
     )
@@
       (effects (font (size 0.5 0.5)) (justify left))
     )
-    (property "Footprint" "02_dyn_pcblib:L7.1x6.6mm" (id 2) (at 187.96 97.79 0)
-      (effects (font (size 1.27 1.27)) hide)
-    )
+    (property "Footprint" "2005_inductance:L7.1x6.6mm" (id 2) (at 187.96 97.79 0)
+      (effects (font (size 1.27 1.27)) hide)
+    )
