File: kicad01_power_board_for_nuclear_team/kicad01_power_board_for_nuclear_team.kicad_pcb (KiCad board)
At the start: 2 copper layers, 100 x 100 mm, 63 parts, among them U301 dcdc_lt8612x, U401 dcdc_lt8612x, U501 dcdc_lt8612x

Commit message: x
Parts:
- added R201: R1206_0.0, 02_dyn_pcblib:R1206mix0603, F.Cu at (73.7, 99.1)
- added R224: R0603_1M, 02_dyn_pcblib:C0603, F.Cu at (114.3, 104.1)
- added R603: R0805_0.0, 02_dyn_pcblib:R0805mix0603, F.Cu at (109.2, 85.0)
- added R604: R0603_DNP, 02_dyn_pcblib:C0603, F.Cu at (117.7, 109.2)
- added R623: R0603_10k, 02_dyn_pcblib:C0603, F.Cu at (119.4, 104.1)
- added R624: R0603_10k, 02_dyn_pcblib:C0603, F.Cu at (113.4, 84.8)
- added R633: R0603_10k, 02_dyn_pcblib:C0603, F.Cu at (121.9, 109.2)
- added R634: R0603_10k, 02_dyn_pcblib:C0603, F.Cu at (123.4, 104.1)
- added R705: R0603_1M, 02_dyn_pcblib:C0603, F.Cu at (146.3, 63.5)
- added R718: R0603_1M, 02_dyn_pcblib:C0603, F.Cu at (143.6, 58.4)
- added R724: R0603_1M, 02_dyn_pcblib:C0603, F.Cu at (147.6, 58.4)
- C322, C324, C325, C365, C371, C422, C424, C425, C465, C471, C522, C524, C525, C565, C571: footprint Capacitor_SMD:C_0603_1608Metric -> 02_dyn_pcblib:C0603
- R311, R312, R313, R323, R331, R332, R351, R361, R362, R365, R411, R412, R413, R423, R431, R432, R451, R461, R462, R465, R511, R512, R513, R523, R531, R532, R551, R561, R562, R565: footprint Resistor_SMD:R_0603_1608Metric -> 02_dyn_pcblib:C0603
- R352, R452, R552: footprint Resistor_SMD:R_0603_1608Metric_Pad0.98x0.95mm_HandSolder -> 02_dyn_pcblib:C0603
- moved R531 92.5 mm to (66.0, 55.9)
- moved R562 89.3 mm to (75.8, 53.3)
- moved R532 84.8 mm to (79.8, 53.3)
- moved C524 84.6 mm to (88.9, 53.3)
- moved C571 83.9 mm to (83.8, 53.3)
- moved R552 80.1 mm to (94.0, 53.3)
- moved U501 77.4 mm to (67.5, 66.3)
- moved R523 76.1 mm to (97.6, 53.3)
- moved R513 74.5 mm to (86.4, 63.5)
- moved R565 73.3 mm to (91.4, 63.5)
- moved L571 70.7 mm to (79.0, 61.0)
- moved C525 69.8 mm to (97.6, 63.5)
- moved C565 68.2 mm to (104.1, 59.2)
- moved R511 67.1 mm to (101.6, 63.5)
- moved C522 66.7 mm to (80.4, 76.2)
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Connections:
- C321 pad 2: GND -> Net-(C321-Pad2)
- C322 pad 2: GND -> Net-(C322-Pad2)
- C324 pad 1: GND -> Net-(C324-Pad1)
- C371 pad 2: GND -> Net-(C321-Pad2)
- C421 pad 2: GND -> Net-(C421-Pad2)
- C422 pad 2: GND -> Net-(C422-Pad2)
- C424 pad 1: GND -> Net-(C424-Pad1)
- C471 pad 2: GND -> Net-(C421-Pad2)
- C521 pad 2: GND -> Net-(C521-Pad2)
- C522 pad 2: GND -> Net-(C522-Pad2)
- C524 pad 1: GND -> Net-(C524-Pad1)
- C571 pad 2: GND -> Net-(C521-Pad2)
- R313 pad 2: GND -> Net-(C322-Pad2)
- R323 pad 2: GND -> Net-(C322-Pad2)
- R331 pad 2: GND -> Net-(C322-Pad2)
- R361 pad 2: GND -> Net-(R361-Pad2)
- R413 pad 2: GND -> Net-(C422-Pad2)
- R423 pad 2: GND -> Net-(C422-Pad2)
- R431 pad 2: GND -> Net-(C422-Pad2)
- R461 pad 2: GND -> Net-(R461-Pad2)
- R513 pad 2: GND -> Net-(C522-Pad2)
- R523 pad 2: GND -> Net-(C522-Pad2)
- R531 pad 2: GND -> Net-(C522-Pad2)
- R561 pad 2: GND -> Net-(R561-Pad2)
- U301 pad 10: GND -> Net-(C321-Pad2)
- U301 pad 11: GND -> Net-(C321-Pad2)
- U301 pad 12: GND -> Net-(C321-Pad2)
- U301 pad 13: GND -> Net-(C321-Pad2)
- U301 pad 14: GND -> Net-(C321-Pad2)
- U301 pad 25: GND -> Net-(C322-Pad2)
- U301 pad 26: GND -> Net-(C322-Pad2)
- U301 pad 27: GND -> Net-(C322-Pad2)
- U301 pad 28: GND -> Net-(C322-Pad2)
- U301 pad 29: GND -> Net-(C321-Pad2)
- U301 pad 30: GND -> Net-(C321-Pad2)
- U301 pad 31: GND -> Net-(C321-Pad2)
- U301 pad 32: GND -> Net-(C321-Pad2)
- U301 pad 8: GND -> Net-(C321-Pad2)
- U301 pad 9: GND -> Net-(C321-Pad2)
- U401 pad 10: GND -> Net-(C421-Pad2)
- U401 pad 11: GND -> Net-(C421-Pad2)
- U401 pad 12: GND -> Net-(C421-Pad2)
- U401 pad 13: GND -> Net-(C421-Pad2)
- U401 pad 14: GND -> Net-(C421-Pad2)
- U401 pad 25: GND -> Net-(C422-Pad2)
- U401 pad 26: GND -> Net-(C422-Pad2)
- U401 pad 27: GND -> Net-(C422-Pad2)
- U401 pad 28: GND -> Net-(C422-Pad2)
- U401 pad 29: GND -> Net-(C421-Pad2)
- U401 pad 30: GND -> Net-(C421-Pad2)
- U401 pad 31: GND -> Net-(C421-Pad2)
- U401 pad 32: GND -> Net-(C421-Pad2)
- U401 pad 8: GND -> Net-(C421-Pad2)
- U401 pad 9: GND -> Net-(C421-Pad2)
- U501 pad 10: GND -> Net-(C521-Pad2)
- U501 pad 11: GND -> Net-(C521-Pad2)
- U501 pad 12: GND -> Net-(C521-Pad2)
- U501 pad 13: GND -> Net-(C521-Pad2)
- U501 pad 14: GND -> Net-(C521-Pad2)
- U501 pad 25: GND -> Net-(C522-Pad2)
- U501 pad 26: GND -> Net-(C522-Pad2)
- U501 pad 27: GND -> Net-(C522-Pad2)
- U501 pad 28: GND -> Net-(C522-Pad2)
- U501 pad 29: GND -> Net-(C521-Pad2)
- U501 pad 30: GND -> Net-(C521-Pad2)
- U501 pad 31: GND -> Net-(C521-Pad2)
- U501 pad 32: GND -> Net-(C521-Pad2)
- U501 pad 8: GND -> Net-(C521-Pad2)
- U501 pad 9: GND -> Net-(C521-Pad2)

Commit message: ix
Parts:
- removed R201: R1206_0.0, 02_dyn_pcblib:R1206mix0603
- removed R224, R705, R718, R724: R0603_1M, 02_dyn_pcblib:C0603
- added B801: nucleco_power_board_v101, 02_dyn_pcblib:nucleco_power_board_v101, F.Cu at (59.3, 152.4)
- added C201: c0805_35v10u, 02_dyn_pcblib:C0805mix0603, F.Cu at (60.8, 97.6)
- added C211: c0805_35v10u, 02_dyn_pcblib:C0805mix0603, F.Cu at (69.9, 97.4)
- added C701: c0805_35v10u, 02_dyn_pcblib:C0805mix0603, F.Cu at (71.3, 149.7)
- added C711: c0805_35v10u, 02_dyn_pcblib:C0805mix0603, F.Cu at (92.2, 149.9)
- added C721: c0805_35v10u, 02_dyn_pcblib:C0805mix0603, F.Cu at (151.7, 150.1)
- added H201: hdr_2x1_1-1123723-2, 02_dyn_pcblib:hdr_2x1_1-1123723-2, F.Cu at (66.9, 92.9)
- added H211: hdr_2x1_1-1123723-2, 02_dyn_pcblib:hdr_2x1_1-1123723-2, F.Cu at (76.4, 92.8)
- added H701: hdr_2x1_1-1123723-2, 02_dyn_pcblib:hdr_2x1_1-1123723-2, F.Cu at (63.7, 146.5)
- added H711: hdr_2x1_1-1123723-2, 02_dyn_pcblib:hdr_2x1_1-1123723-2, F.Cu at (96.8, 146.7)
- added H721: hdr_2x1_1-1123723-2, 02_dyn_pcblib:hdr_2x1_1-1123723-2, F.Cu at (143.1, 147.1)
- added PTC201: PTC_fuse_7A, 02_dyn_pcblib:ptc_fuse_2920, F.Cu at (65.4, 103.1)
- added Q251: nmos75v80a_IRFS3607TRLPBF, 02_dyn_pcblib:d2pak_TO263, F.Cu at (71.1, 114.2)
- added R211: R1206_0.0, 02_dyn_pcblib:R1206mix0603, F.Cu at (61.0, 141.0)
- added R221: R0603_1M, 02_dyn_pcblib:C0603, F.Cu at (61.7, 112.4)
- added R222: R0603_1M, 02_dyn_pcblib:C0603, F.Cu at (61.6, 116.9)
- moved C424 113.1 mm to (240.5, 41.6)
- moved C471 113.1 mm to (258.7, 56.8)
- moved C571 113.1 mm to (194.8, 31.4)
- moved D451 113.1 mm to (263.4, 56.8)
- moved R312 113.1 mm to (194.8, 82.2)
- moved R412 113.1 mm to (263.4, 46.7)
- moved R451 113.1 mm to (240.5, 56.8)
- moved R465 113.1 mm to (250.7, 56.8)
- moved C324 113.1 mm to (196.6, 92.4)
- moved C365 113.1 mm to (207.5, 82.2)
- moved C371 113.1 mm to (211.5, 87.3)
- moved C421 113.1 mm to (232.9, 64.4)
- moved C565 113.1 mm to (215.1, 37.3)
- moved D351 113.1 mm to (189.7, 77.1)
- moved L471 113.1 mm to (222.7, 34.0)
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Connections:
- C321 pad 2: Net-(C321-Pad2) -> GND
- C322 pad 2: Net-(C322-Pad2) -> GND
- C324 pad 1: Net-(C324-Pad1) -> GND
- C371 pad 2: Net-(C321-Pad2) -> GND
- C421 pad 2: Net-(C421-Pad2) -> GND
- C422 pad 2: Net-(C422-Pad2) -> GND
- C424 pad 1: Net-(C424-Pad1) -> GND
- C471 pad 2: Net-(C421-Pad2) -> GND
- C521 pad 2: Net-(C521-Pad2) -> GND
- C522 pad 2: Net-(C522-Pad2) -> GND
- C524 pad 1: Net-(C524-Pad1) -> GND
- C571 pad 2: Net-(C521-Pad2) -> GND
- R313 pad 2: Net-(C322-Pad2) -> GND
- R323 pad 2: Net-(C322-Pad2) -> GND
- R331 pad 2: Net-(C322-Pad2) -> GND
- R361 pad 2: Net-(R361-Pad2) -> GND
- R413 pad 2: Net-(C422-Pad2) -> GND
- R423 pad 2: Net-(C422-Pad2) -> GND
- R431 pad 2: Net-(C422-Pad2) -> GND
- R461 pad 2: Net-(R461-Pad2) -> GND
- R513 pad 2: Net-(C522-Pad2) -> GND
- R523 pad 2: Net-(C522-Pad2) -> GND
- R531 pad 2: Net-(C522-Pad2) -> GND
- R561 pad 2: Net-(R561-Pad2) -> GND
- U301 pad 10: Net-(C321-Pad2) -> GND
- U301 pad 11: Net-(C321-Pad2) -> GND
- U301 pad 12: Net-(C321-Pad2) -> GND
- U301 pad 13: Net-(C321-Pad2) -> GND
- U301 pad 14: Net-(C321-Pad2) -> GND
- U301 pad 25: Net-(C322-Pad2) -> GND
- U301 pad 26: Net-(C322-Pad2) -> GND
- U301 pad 27: Net-(C322-Pad2) -> GND
- U301 pad 28: Net-(C322-Pad2) -> GND
- U301 pad 29: Net-(C321-Pad2) -> GND
- U301 pad 30: Net-(C321-Pad2) -> GND
- U301 pad 31: Net-(C321-Pad2) -> GND
- U301 pad 32: Net-(C321-Pad2) -> GND
- U301 pad 8: Net-(C321-Pad2) -> GND
- U301 pad 9: Net-(C321-Pad2) -> GND
- U401 pad 10: Net-(C421-Pad2) -> GND
- U401 pad 11: Net-(C421-Pad2) -> GND
- U401 pad 12: Net-(C421-Pad2) -> GND
- U401 pad 13: Net-(C421-Pad2) -> GND
- U401 pad 14: Net-(C421-Pad2) -> GND
- U401 pad 25: Net-(C422-Pad2) -> GND
- U401 pad 26: Net-(C422-Pad2) -> GND
- U401 pad 27: Net-(C422-Pad2) -> GND
- U401 pad 28: Net-(C422-Pad2) -> GND
- U401 pad 29: Net-(C421-Pad2) -> GND
- U401 pad 30: Net-(C421-Pad2) -> GND
- U401 pad 31: Net-(C421-Pad2) -> GND
- U401 pad 32: Net-(C421-Pad2) -> GND
- U401 pad 8: Net-(C421-Pad2) -> GND
- U401 pad 9: Net-(C421-Pad2) -> GND
- U501 pad 10: Net-(C521-Pad2) -> GND
- U501 pad 11: Net-(C521-Pad2) -> GND
- U501 pad 12: Net-(C521-Pad2) -> GND
- U501 pad 13: Net-(C521-Pad2) -> GND
- U501 pad 14: Net-(C521-Pad2) -> GND
- U501 pad 25: Net-(C522-Pad2) -> GND
- U501 pad 26: Net-(C522-Pad2) -> GND
- U501 pad 27: Net-(C522-Pad2) -> GND
- U501 pad 28: Net-(C522-Pad2) -> GND
- U501 pad 29: Net-(C521-Pad2) -> GND
- U501 pad 30: Net-(C521-Pad2) -> GND
- U501 pad 31: Net-(C521-Pad2) -> GND
- U501 pad 32: Net-(C521-Pad2) -> GND
- U501 pad 8: Net-(C521-Pad2) -> GND
- U501 pad 9: Net-(C521-Pad2) -> GND
Routing:
- net GND: track 0.00 -> 160.9 mm
- net V24in: track 0.00 -> 64.1 mm
- net Net-(C201-Pad1): track 0.00 -> 29.8 mm
- net V24out: track 0.00 -> 20.2 mm
- net Net-(PTC201-Pad2): track 0.00 -> 12.2 mm
- net Net-(Q251-Pad1): track 0.00 -> 7.22 mm
- net V5out: track 0.00 -> 6.34 mm
Other:
- board size 100 x 100 mm -> 99.9 x 65 mm

Commit message: x
Parts:
- added C372: c0805_DNP, 02_dyn_pcblib:C0805mix0603, F.Cu at (196.7, 137.7)
- added C472: c0805_DNP, 02_dyn_pcblib:C0805mix0603, F.Cu at (280.3, 118.9)
- added C572: c0805_DNP, 02_dyn_pcblib:C0805mix0603, F.Cu at (172.2, 136.3)
- moved R491 132.8 mm to (314.9, 145.2)
- moved C571 108.0 mm to (170.1, 136.5), turned to 90 degrees
- moved C524 106.0 mm to (170.1, 133.1), turned to 90 degrees
- moved R552 105.9 mm to (171.8, 132.0), turned to -90 degrees
- moved C565 103.1 mm to (178.2, 133.5)
- moved R523 102.3 mm to (172.8, 127.2), turned to -90 degrees
- moved L571 100.2 mm to (165.6, 136.3), turned to -90 degrees
- moved R562 99.6 mm to (175.5, 130.3), turned to 90 degrees
- moved C525 98.6 mm to (166.6, 130.8)
- moved R532 95.8 mm to (178.1, 126.4)
- moved R531 94.1 mm to (178.1, 128.1), turned to 180 degrees
- moved R565 93.3 mm to (178.2, 131.7), turned to 180 degrees
- moved R511 93.1 mm to (168.7, 123.7), turned to 180 degrees
- moved D551 89.5 mm to (178.1, 135.4)
- moved C465 88.5 mm to (266.5, 121.6)
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Routing:
- net GND: track 160.9 -> 314.6 mm
- net V24in: track 64.1 -> 123.0 mm
- net Net-(C365-Pad2): track 0.00 -> 35.5 mm
- net Net-(C565-Pad2): track 0.00 -> 32.6 mm
- net Net-(C525-Pad1): track 0.00 -> 21.1 mm
- net Net-(C325-Pad1): track 0.00 -> 15.1 mm
- net Net-(C365-Pad1): track 0.00 -> 11.3 mm
- net Net-(C565-Pad1): track 0.00 -> 11.1 mm
- net Net-(R532-Pad1): track 0.00 -> 10.2 mm
- net Net-(R332-Pad1): track 0.00 -> 10.2 mm
- net Vgood5: track 0.00 -> 9.73 mm
- net Vgood3: track 0.00 -> 9.43 mm
- net Net-(R512-Pad1): track 0.00 -> 7.86 mm
- net Net-(R312-Pad1): track 0.00 -> 7.62 mm
- net Net-(C522-Pad1): track 0.00 -> 7.51 mm
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
Commit message: x
Parts:
- moved R491 189.7 mm to (125.3, 139.4)
- moved R412 167.4 mm to (120.5, 123.7), turned to 180 degrees
- moved C471 165.4 mm to (117.7, 137.1), turned to 90 degrees
- moved C472 161.5 mm to (119.8, 137.0), turned to -90 degrees
- moved D451 161.5 mm to (126.4, 135.9)
- moved C422 157.7 mm to (122.0, 127.0), turned to -90 degrees
- moved R432 156.1 mm to (125.6, 126.0)
- moved R462 154.6 mm to (123.1, 130.3)
- moved R411 154.4 mm to (116.2, 123.7), turned to 180 degrees
- moved R423 153.7 mm to (119.3, 127.7), turned to -90 degrees
- moved R465 148.9 mm to (126.4, 133.8), turned to 180 degrees
- moved C424 147.4 mm to (117.7, 133.8), turned to 90 degrees
- moved C421 147.1 mm to (112.4, 124.2), turned to 180 degrees
- moved R431 144.3 mm to (126.4, 127.7)
- moved R452 143.3 mm to (119.5, 132.8), turned to -90 degrees
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Routing:
- net GND: track 314.6 -> 396.9 mm
- net V24in: track 123.0 -> 176.9 mm
- net Net-(C465-Pad2): track 0.00 -> 28.2 mm
- net Net-(C425-Pad1): track 0.00 -> 15.1 mm
- net Net-(C465-Pad1): track 0.00 -> 13.2 mm
- net Net-(C565-Pad2): track 32.6 -> 43.7 mm
- net Net-(R432-Pad1): track 0.00 -> 10.2 mm
- net Net-(R412-Pad1): track 0.00 -> 9.92 mm
- net Vgood4: track 0.00 -> 7.56 mm
- net Net-(C422-Pad1): track 0.00 -> 6.59 mm
- net VOint4: track 0.00 -> 4.83 mm
- net Net-(D451-Pad1): track 0.00 -> 4.34 mm
- net Vsync5: track 0.00 -> 3.05 mm
- net Net-(D551-Pad1): track 1.67 -> 4.62 mm
- net Vsync4: track 0.00 -> 2.93 mm
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
Commit message: x
Routing:
- net GND: track 396.9 -> 572.7 mm, vias 0 -> 4
Changed lines of the file:
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@@
   (segment (start 61.655 116.0522) (end 61.655 113.1318) (width 0.25) (layer "F.Cu") (net 51))
   (segment (start 61.6042 116.103) (end 61.655 116.0522) (width 0.25) (layer "F.Cu") (net 51))
-  (segment (start 65.284 145.282) (end 65.284 116.7574) (width 0.25) (layer "F.Cu") (net 52))
   (segment (start 139.956 113.6115) (end 139.9435 113.6115) (width 0.25) (layer "F.Cu") (net 52))
   (segment (start 139.231 115.324) (end 139.231 115.824) (width 0.25) (layer "F.Cu") (net 52))
   (segment (start 83.913 126.3115) (end 85.3755 126.3115) (width 0.25) (layer "F.Cu") (net 52))
   (segment (start 143.69398 114.34852) (end 143.4335 114.609) (width 0.25) (layer "F.Cu") (net 52))
+  (segment (start 75.946 133.8326) (end 75.8758 133.9028) (width 0.25) (layer "F.Cu") (net 52))
   (segment (start 145.181 115.824) (end 146.919 115.824) (width 0.25) (layer "F.Cu") (net 52))
   (segment (start 140.463 114.609) (end 140.9785 114.609) (width 0.25) (layer "F.Cu") (net 52))
@@
   (segment (start 139.6155 113.6115) (end 138.91848 112.91448) (width 0.25) (layer "F.Cu") (net 52))
   (segment (start 89.863 126.3115) (end 89.83848 126.33602) (width 0.25) (layer "F.Cu") (net 52))
+  (segment (start 73.6854 100.5078) (end 73.533 100.3554) (width 0.25) (layer "F.Cu") (net 52))
   (segment (start 112.1395 124.432) (end 111.8855 124.178) (width 0.25) (layer "F.Cu") (net 52))
   (segment (start 140.956 113.6115) (end 140.956 113.077718) (width 0.25) (layer "F.Cu") (net 52))
@@
   (segment (start 85.6605 126.5965) (end 85.6605 127.0865) (width 0.25) (layer "F.Cu") (net 52))
   (segment (start 153.87348 115.74948) (end 153.87348 117.08948) (width 0.25) (layer "F.Cu") (net 52))
+  (segment (start 142.5956 133.8072) (end 143.0782 133.3246) (width 0.25) (layer "F.Cu") (net 52))
   (segment (start 119.2515 128.509) (end 121.2835 128.509) (width 0.25) (layer "F.Cu") (net 52))
   (segment (start 138.4215 123.0615) (end 137.03048 121.67048) (width 0.25) (layer "F.Cu") (net 52))
@@
   (segment (start 149.47648 115.26848) (end 149.93248 115.26848) (width 0.25) (layer "F.Cu") (net 52))
   (segment (start 143.6485 114.824) (end 143.4335 114.609) (width 0.25) (layer "F.Cu") (net 52))
+  (segment (start 145.161 133.5532) (end 144.7038 133.5532) (width 0.25) (layer "F.Cu") (net 52))
   (segment (start 139.9435 113.6115) (end 139.231 114.324) (width 0.25) (layer "F.Cu") (net 52))
   (segment (start 98.5855 123.2045) (end 98.1975 122.8165) (width 0.25) (layer "F.Cu") (net 52))
@@
   (segment (start 113.193 127.516) (end 113.408 127.301) (width 0.25) (layer "F.Cu") (net 52))
   (segment (start 82.0005 128.6065) (end 82.7955 127.8115) (width 0.25) (layer "F.Cu") (net 52))
+  (segment (start 142.621 100.5078) (end 142.5702 100.457) (width 0.25) (layer "F.Cu") (net 52))
+  (segment (start 134.9248 100.457) (end 131.9276 103.4542) (width 0.25) (layer "F.Cu") (net 52))
   (segment (start 140.456 113.6115) (end 139.361 112.5165) (width 0.25) (layer "F.Cu") (net 52))
   (segment (start 85.6605 127.5265) (end 88.1155 127.5265) (width 0.25) (layer "F.Cu") (net 52))
@@
   (segment (start 110.8695 124.94) (end 110.8695 128.242) (width 0.25) (layer "F.Cu") (net 52))
   (segment (start 112.373 126.3035) (end 111.6605 127.016) (width 0.25) (layer "F.Cu") (net 52))
+  (segment (start 75.946 100.5078) (end 73.6854 100.5078) (width 0.25) (layer "F.Cu") (net 52))
   (segment (start 89.1405 127.5265) (end 88.1155 127.5265) (width 0.25) (layer "F.Cu") (net 52))
   (segment (start 138.91848 112.91448) (end 138.91848 111.64402) (width 0.25) (layer "F.Cu") (net 52))
@@
   (segment (start 63.7286 146.685) (end 63.8048 146.7612) (width 0.25) (layer "F.Cu") (net 52))
   (segment (start 89.863 126.8115) (end 89.863 127.089) (width 0.25) (layer "F.Cu") (net 52))
+  (segment (start 75.8758 133.9028) (end 65.284 133.9028) (width 0.25) (layer "F.Cu") (net 52))
   (segment (start 137.03048 117.52452) (end 139.231 115.324) (width 0.25) (layer "F.Cu") (net 52))
   (segment (start 146.93648 115.84148) (end 146.94948 115.82848) (width 0.25) (layer "F.Cu") (net 52))
@@
   (segment (start 112.3855 126.964) (end 112.7225 127.301) (width 0.25) (layer "F.Cu") (net 52))
   (segment (start 82.780978 135.0015) (end 82.0005 134.221022) (width 0.25) (layer "F.Cu") (net 52))
+  (segment (start 142.5702 100.457) (end 134.9248 100.457) (width 0.25) (layer "F.Cu") (net 52))
   (segment (start 83.913 127.3115) (end 85.4455 127.3115) (width 0.25) (layer "F.Cu") (net 52))
   (segment (start 139.956 114.102) (end 140.463 114.609) (width 0.25) (layer "F.Cu") (net 52))
@@
   (segment (start 89.8905 135.0015) (end 89.8905 135.0835) (width 0.25) (layer "F.Cu") (net 52))
   (segment (start 143.4335 114.609) (end 140.9785 114.609) (width 0.25) (layer "F.Cu") (net 52))
+  (segment (start 143.0782 133.3246) (end 145.3896 133.3246) (width 0.25) (layer "F.Cu") (net 52))
   (segment (start 139.956 111.2015) (end 139.361 111.2015) (width 0.25) (layer "F.Cu") (net 52))
   (segment (start 117.7275 136.37) (end 111.3775 136.37) (width 0.25) (layer "F.Cu") (net 52))
@@
   (segment (start 89.863 126.8115) (end 88.3305 126.8115) (width 0.25) (layer "F.Cu") (net 52))
   (segment (start 127.1515 128.483) (end 127.1515 127.734) (width 0.25) (layer "F.Cu") (net 52))
+  (segment (start 131.9276 103.4542) (end 131.9276 126.111) (width 0.25) (layer "F.Cu") (net 52))
   (segment (start 140.456 113.6115) (end 140.456 114.0865) (width 0.25) (layer "F.Cu") (net 52))
   (segment (start 112.3855 126.3035) (end 112.3855 126.964) (width 0.25) (layer "F.Cu") (net 52))
@@
   (segment (start 112.7225 127.301) (end 113.408 127.301) (width 0.25) (layer "F.Cu") (net 52))
   (segment (start 85.638 125.599) (end 85.638 127.064) (width 0.25) (layer "F.Cu") (net 52))
+  (segment (start 131.9276 126.111) (end 139.6238 133.8072) (width 0.25) (layer "F.Cu") (net 52))
+  (segment (start 145.3896 133.3246) (end 145.161 133.5532) (width 0.25) (layer "F.Cu") (net 52))
   (segment (start 140.9785 114.609) (end 140.9785 115.539) (width 0.25) (layer "F.Cu") (net 52))
   (segment (start 145.181 114.824) (end 145.181 114.324) (width 0.25) (layer "F.Cu") (net 52))
@@
   (segment (start 83.913 127.3115) (end 83.913 126.8115) (width 0.25) (layer "F.Cu") (net 52))
   (segment (start 116.078 127.516) (end 115.863 127.301) (width 0.25) (layer "F.Cu") (net 52))
+  (segment (start 139.6238 133.8072) (end 142.5956 133.8072) (width 0.25) (layer "F.Cu") (net 52))
+  (segment (start 65.284 145.282) (end 65.284 133.9028) (width 0.25) (layer "F.Cu") (net 52))
   (segment (start 85.3755 126.3115) (end 85.6605 126.5965) (width 0.25) (layer "F.Cu") (net 52))
   (segment (start 84.638 125.599) (end 84.638 126.054) (width 0.25) (layer "F.Cu") (net 52))
@@
   (segment (start 98.5885 127.5775) (end 98.6145 127.5515) (width 0.25) (layer "F.Cu") (net 52))
   (segment (start 112.8855 126.7785) (end 113.408 127.301) (width 0.25) (layer "F.Cu") (net 52))
+  (segment (start 65.284 133.9028) (end 65.284 116.7574) (width 0.25) (layer "F.Cu") (net 52))
   (segment (start 110.8695 128.242) (end 111.1235 128.496) (width 0.25) (layer "F.Cu") (net 52))
+  (via (at 142.621 100.5078) (size 2.9) (drill 2.5) (layers "F.Cu" "B.Cu") (net 52))
+  (via (at 75.946 100.5078) (size 2.9) (drill 2.5) (layers "F.Cu" "B.Cu") (net 52))
+  (via (at 75.946 133.8326) (size 2.9) (drill 2.5) (layers "F.Cu" "B.Cu") (net 52))
+  (via (at 142.5956 133.8072) (size 2.9) (drill 2.5) (layers "F.Cu" "B.Cu") (net 52))
+  (segment (start 77.9526 135.8392) (end 78.4098 135.8392) (width 0.25) (layer "B.Cu") (net 52))
+  (segment (start 143.129 134.3406) (end 142.5956 133.8072) (width 0.25) (layer "B.Cu") (net 52))
   (segment (start 98.5012 150.8252) (end 96.7547 149.0787) (width 0.25) (layer "B.Cu") (net 52))
   (segment (start 89.9756 146.6684) (end 96.7547 146.6684) (width 0.25) (layer "B.Cu") (net 52))
+  (segment (start 84.4296 97.1804) (end 81.1276 100.4824) (width 0.25) (layer "B.Cu") (net 52))
+  (segment (start 144.4498 98.679) (end 144.4498 88.0364) (width 0.25) (layer "B.Cu") (net 52))
   (segment (start 143.129 147.1422) (end 143.129 147.2946) (width 0.25) (layer "B.Cu") (net 52))
+  (segment (start 83.058 95.8088) (end 84.4296 97.1804) (width 0.25) (layer "B.Cu") (net 52))
   (segment (start 96.7547 149.0787) (end 96.7547 146.6684) (width 0.25) (layer "B.Cu") (net 52))
   (segment (start 68.1228 150.876) (end 85.6488 150.876) (width 0.25) (layer "B.Cu") (net 52))
   (segment (start 63.7286 146.4818) (end 68.1228 150.876) (width 0.25) (layer "B.Cu") (net 52))
+  (segment (start 143.129 147.1422) (end 143.129 134.3406) (width 0.25) (layer "B.Cu") (net 52))
   (segment (start 85.6488 150.876) (end 89.916 146.6088) (width 0.25) (layer "B.Cu") (net 52))
+  (segment (start 75.9714 100.4824) (end 75.946 100.5078) (width 0.25) (layer "B.Cu") (net 52))
   (segment (start 143.1544 147.32) (end 139.6492 150.8252) (width 0.25) (layer "B.Cu") (net 52))
   (segment (start 139.6492 150.8252) (end 98.5012 150.8252) (width 0.25) (layer "B.Cu") (net 52))
   (segment (start 89.916 146.6088) (end 89.9756 146.6684) (width 0.25) (layer "B.Cu") (net 52))
+  (segment (start 75.946 133.8326) (end 77.9526 135.8392) (width 0.25) (layer "B.Cu") (net 52))
+  (segment (start 83.058 89.1032) (end 83.058 95.8088) (width 0.25) (layer "B.Cu") (net 52))
+  (segment (start 84.1248 88.0364) (end 83.058 89.1032) (width 0.25) (layer "B.Cu") (net 52))
+  (segment (start 142.621 100.5078) (end 144.4498 98.679) (width 0.25) (layer "B.Cu") (net 52))
+  (segment (start 81.1276 100.4824) (end 75.9714 100.4824) (width 0.25) (layer "B.Cu") (net 52))
   (segment (start 143.129 147.2946) (end 143.1544 147.32) (width 0.25) (layer "B.Cu") (net 52))
+  (segment (start 144.4498 88.0364) (end 84.1248 88.0364) (width 0.25) (layer "B.Cu") (net 52))
   (segment (start 65.405 106.5208) (end 66.7374 106.5208) (width 0.25) (layer "F.Cu") (net 53))
   (segment (start 66.7374 106.5208) (end 74.434 114.2174) (width 0.25) (layer "F.Cu") (net 53))
