File: kicad01_power_board_for_nuclear_team/kicad01_power_board_for_nuclear_team.kicad_pcb (KiCad board)
At the start: 2 copper layers, 99.9 x 65 mm, 88 parts, among them Q251 nmos75v80a_IRFS3607TRLPBF, U301 dcdc_lt8612x, U401 dcdc_lt8612x, U501 dcdc_lt8612x

Commit message: x
Parts:
- added H1: hole2mm50_7mm40, 02_dyn_pcblib:hole2mm50_7mm40, F.Cu at (142.7, 100.6)
- added H2: hole2mm50_7mm40, 02_dyn_pcblib:hole2mm50_7mm40, F.Cu at (75.9, 100.5)
- added H3: hole2mm50_7mm40, 02_dyn_pcblib:hole2mm50_7mm40, F.Cu at (75.9, 133.7)
- added H4: hole2mm50_7mm40, 02_dyn_pcblib:hole2mm50_7mm40, F.Cu at (142.5, 133.7)
- moved C211 17.1 mm to (86.1, 91.8)
- moved C201 5.36 mm to (61.9, 92.3)
- moved H211 3.24 mm to (79.5, 93.8), turned to 90 degrees
- moved H201 1.15 mm to (67.4, 93.9), turned to 90 degrees
Routing:
- net V24in: track 176.9 -> 304.9 mm, vias 0 -> 6
- net V18out: track 0.00 -> 57.4 mm
- net GND: track 572.7 -> 621.9 mm, vias 4 -> 0
- net V5out: track 6.17 -> 27.5 mm
- net Net-(C201-Pad1): track 29.8 -> 31.7 mm

Commit message: x
Parts:
- added U601: mcu_MSP430FR2433IRGER, 02_dyn_pcblib:QFN-24-1EP_4x4mm_P0.5mm_EP2.8x2.8mmX, F.Cu at (117.0, 97.3)
- Q251: value nmos75v80a_IRFS3607TRLPBF -> nmosTO263_75v80A
Routing:
- net GND: track 621.9 -> 640.3 mm

Commit message: x
Parts:
- B801: footprint 02_dyn_pcblib:nucleco_power_board_v101 -> 2008_h3d:nucleco_power_board_v101
- C201, C211, C321, C372, C421, C472, C521, C572, C701, C711, C721: footprint 02_dyn_pcblib:C0805mix0603 -> 2004_cap:C0805mix0603
- C322, C324, C325, C365, C371, C422, C424, C425, C465, C471, C522, C524, C525, C565, C571, R221, R222, R311, R312, R313, R323, R331, R332, R351, R352, R361, R362, R365, R411, R412, R413, R423, R431, R432, R451, R452, R461, R462, R465, R511, R512, R513, R523, R531, R532, R551, R552, R561, R562, R565, R604, R623, R624, R633, R634: footprint 02_dyn_pcblib:C0603 -> 2004_cap:C0603
- D351, D451, D551: footprint 02_dyn_pcblib:LED0603 -> 2007_LED:LED0603
- H1, H2, H3, H4: footprint 02_dyn_pcblib:hole2mm50_7mm40 -> 2002_hdr:hole2mm50_7mm40
- H201, H211, H701, H711, H721: footprint 02_dyn_pcblib:hdr_2x1_1-1123723-2 -> 2002_hdr:hdr_2x1_1-1123723-2
- L371, L471, L571: footprint 02_dyn_pcblib:L7.1x6.6mm -> 2005_inductance:L7.1x6.6mm
- PTC201: footprint 02_dyn_pcblib:ptc_fuse_2920 -> 2003_res:ptc_fuse_2920
- Q251: footprint 02_dyn_pcblib:d2pak_TO263 -> 2001_dyn_pcblib:d2pak_TO263
- R211, R391, R491, R591: footprint 02_dyn_pcblib:R1206mix0603 -> 2003_res:R1206mix0603
- R603: footprint 02_dyn_pcblib:R0805mix0603 -> 2003_res:R0805mix0603
- U301, U401, U501: footprint 02_dyn_pcblib:QFN-28-1EP_3x6mm_P0.5mm_EP1.7x4.75mmX -> 2006_qfn:QFN-28-1EP_3x6mm_P0.5mm_EP1.7x4.75mmX
- U601: footprint 02_dyn_pcblib:QFN-24-1EP_4x4mm_P0.5mm_EP2.8x2.8mmX -> 2006_qfn:QFN-24-1EP_4x4mm_P0.5mm_EP2.8x2.8mmX
Connections:
- R604 pad 1: Net-(R603-Pad2) -> Net-(C601-Pad2)
- R624 pad 1: Net-(R623-Pad2) -> Net-(R624-Pad1)
- R634 pad 1: Net-(R633-Pad2) -> Net-(R634-Pad1)
- U601 pad 10: unconnected-(U601-Pad10) -> Net-(R623-Pad2)
- U601 pad 11: unconnected-(U601-Pad11) -> Net-(R693-Pad1)
- U601 pad 12: unconnected-(U601-Pad12) -> Net-(R693-Pad2)
- U601 pad 18: unconnected-(U601-Pad18) -> Net-(C601-Pad1)
- U601 pad 19: unconnected-(U601-Pad19) -> Net-(R692-Pad1)
- U601 pad 20: unconnected-(U601-Pad20) -> Net-(R692-Pad2)
- U601 pad 21: unconnected-(U601-Pad21) -> Net-(R691-Pad2)
- U601 pad 22: unconnected-(U601-Pad22) -> Net-(R691-Pad1)
- U601 pad 23: unconnected-(U601-Pad23) -> Net-(C601-Pad1)
- U601 pad 24: unconnected-(U601-Pad24) -> Net-(C601-Pad2)
- U601 pad 25: unconnected-(U601-Pad25) -> Net-(C601-Pad1)
- U601 pad 26: unconnected-(U601-Pad26) -> Net-(C601-Pad1)
- U601 pad 27: unconnected-(U601-Pad27) -> Net-(C601-Pad1)
- U601 pad 28: unconnected-(U601-Pad28) -> Net-(C601-Pad1)
- U601 pad 3: unconnected-(U601-Pad3) -> Net-(R695-Pad1)
- U601 pad 4: unconnected-(U601-Pad4) -> Net-(R695-Pad2)
- U601 pad 5: unconnected-(U601-Pad5) -> Net-(R694-Pad1)
- U601 pad 6: unconnected-(U601-Pad6) -> Net-(R694-Pad2)
- U601 pad 7: unconnected-(U601-Pad7) -> Net-(R634-Pad1)
- U601 pad 8: unconnected-(U601-Pad8) -> Net-(R624-Pad1)
- U601 pad 9: unconnected-(U601-Pad9) -> Net-(R633-Pad2)
