File: kicad01_power_board_for_nuclear_team/kicad01_power_board_for_nuclear_team.kicad_pcb (KiCad board)
At the start: 2 copper layers, 99.9 x 65 mm, 93 parts, among them Q251 nmosTO263_75v80A, U301 dcdc_lt8612x, U401 dcdc_lt8612x, U501 dcdc_lt8612x, U601 mcu_MSP430FR2433IRGER

Commit message: x
Parts:
- added C601: c0603_50v1u, 2004_cap:C0603, F.Cu at (91.4, 76.2)
- added R691: R0603_DNP, 2003_res:R0603, F.Cu at (91.4, 78.7)
- added R692: R0603_DNP, 2003_res:R0603, F.Cu at (99.5, 76.2)
- added R693: R0603_DNP, 2003_res:R0603, F.Cu at (99.5, 78.7)
- added R694: R0603_DNP, 2003_res:R0603, F.Cu at (95.5, 76.2)
- added R695: R0603_DNP, 2003_res:R0603, F.Cu at (95.5, 78.7)
- R221, R222, R311, R312, R313, R323, R331, R332, R351, R352, R361, R362, R365, R411, R412, R413, R423, R431, R432, R451, R452, R461, R462, R465, R511, R512, R513, R523, R531, R532, R551, R552, R561, R562, R565, R604, R623, R624, R633, R634: footprint 2004_cap:C0603 -> 2003_res:R0603
- R603: value R0805_0.0 -> R0603_DNP; footprint 2003_res:R0805mix0603 -> 2003_res:R0603
Connections:
- R603 pad 2: Net-(R603-Pad2) -> Net-(C601-Pad2)

Commit message: x
Parts:
- added H602: p2mm54_1x4, 2002_hdr:p2mm54_1x4, F.Cu at (101.8, 103.8)
- added R611: R0603_DNP, 2003_res:R0603, F.Cu at (108.8, 99.1)
- added R643: R0603_DNP, 2003_res:R0603, F.Cu at (118.1, 101.9)
- added R644: R0603_DNP, 2003_res:R0603, F.Cu at (118.1, 103.6)
- added R696: R0603_DNP, 2003_res:R0603, F.Cu at (106.7, 105.4)
- added R697: R0603_DNP, 2003_res:R0603, F.Cu at (104.6, 102.9)
- moved R694 38.4 mm to (118.1, 107.2)
- moved R695 37.1 mm to (114.6, 110.5)
- moved R693 32.6 mm to (118.1, 105.4), turned to 180 degrees
- moved R691 29.7 mm to (113.0, 99.1), turned to -90 degrees
- moved R692 28.0 mm to (115.6, 99.1), turned to 90 degrees
- moved C601 27.9 mm to (110.5, 96.5), turned to 180 degrees
- moved R604 19.9 mm to (110.5, 94.0)
- moved R623 11.8 mm to (111.8, 109.2), turned to 90 degrees
- moved R624 9.21 mm to (106.7, 109.2), turned to -90 degrees
- moved R603 8.85 mm to (107.1, 94.0)
- moved U601 8.13 mm to (111.7, 103.5)
- moved R633 6.07 mm to (109.2, 109.2), turned to 90 degrees
- moved R634 4.10 mm to (104.1, 109.2), turned to -90 degrees
- moved C701 3.84 mm to (75.2, 149.7)
- moved H701 3.84 mm to (67.6, 146.5)
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Connections:
- net Net-(R312-Pad1) renamed Vena3
- net Net-(R412-Pad1) renamed Vena4
- C601 pad 1: Net-(C601-Pad1) -> GND
- R694 pad 2: Net-(R694-Pad2) -> Net-(R694-Pad1)
- U601 pad 1: unconnected-(U601-Pad1) -> SBWTdio
- U601 pad 11: Net-(R693-Pad1) -> Net-(R695-Pad1)
- U601 pad 12: Net-(R693-Pad2) -> Net-(R695-Pad2)
- U601 pad 13: unconnected-(U601-Pad13) -> Net-(R694-Pad1)
- U601 pad 14: unconnected-(U601-Pad14) -> Net-(R693-Pad2)
- U601 pad 15: unconnected-(U601-Pad15) -> Net-(R693-Pad1)
- U601 pad 16: unconnected-(U601-Pad16) -> Net-(R644-Pad2)
- U601 pad 17: unconnected-(U601-Pad17) -> Net-(R643-Pad2)
- U601 pad 18: Net-(C601-Pad1) -> GND
- U601 pad 2: unconnected-(U601-Pad2) -> SBWTck
- U601 pad 23: Net-(C601-Pad1) -> GND
- U601 pad 25: Net-(C601-Pad1) -> GND
- U601 pad 26: Net-(C601-Pad1) -> GND
- U601 pad 27: Net-(C601-Pad1) -> GND
- U601 pad 28: Net-(C601-Pad1) -> GND
- U601 pad 3: Net-(R695-Pad1) -> Net-(H602-Pad1)
- U601 pad 4: Net-(R695-Pad2) -> Net-(R697-Pad2)
- U601 pad 5: Net-(R694-Pad1) -> Net-(R696-Pad1)
- U601 pad 6: Net-(R694-Pad2) -> Net-(R696-Pad2)
Routing:
- net GND: track 640.3 -> 1015.3 mm
- net V24in: track 304.9 -> 518.6 mm
- net V18out: track 57.4 -> 133.7 mm
- net Vena3: track 7.87 -> 63.2 mm, vias 0 -> 2
- net Vsync4: track 2.93 -> 54.2 mm, vias 0 -> 2
- net V24out: track 20.2 -> 69.3 mm
- net Vsync3: track 3.36 -> 51.5 mm, vias 0 -> 2
- net VOint3: track 3.53 -> 49.7 mm, vias 0 -> 2
- net Vgood4: track 7.56 -> 47.0 mm, vias 0 -> 2
- net Net-(C465-Pad2): track 28.2 -> 66.8 mm
- net Vgood3: track 7.58 -> 43.0 mm, vias 0 -> 2
- net V5out: track 27.5 -> 62.1 mm
- net VOint4: track 4.83 -> 39.0 mm, vias 0 -> 2
- net Net-(C525-Pad1): track 21.1 -> 47.8 mm
- net Net-(C365-Pad2): track 35.3 -> 61.5 mm
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- added copper zone on B.Cu, net GND
- added copper zone on F.Cu, net GND

Commit message: x
Parts:
- H602: value p2mm54_1x4 -> PinHeader_1x04_P2.54mm_Vertical
Routing:
- net V24in: track 518.6 -> 597.9 mm, vias 6 -> 8
- net GND: track 1015.3 -> 1030.7 mm
- net Vena3: track 63.2 -> 55.0 mm
- net Net-(R692-Pad1): track 3.29 -> 4.00 mm
- net Net-(C201-Pad1): track 50.6 -> 50.0 mm
