File: kicad01_power_board_for_nuclear_team/003_dcdc_18v4a.kicad_sch (KiCad schematic)
At the start: 21 parts, among them U301 dcdc_lt8612x

Commit message: x
Connections:
- net GND: no longer names the net of C321.2, C371.2, U301.10 (PGND), U301.11 (GND), U301.12 (GND), U301.13 (GND), U301.14 (GND), U301.29 (GND), U301.30 (GND), U301.31 (GND), U301.32 (GND), U301.8 (PGND), U301.9 (PGND)
- net GND: no longer C322.2, C324.1, R313.2, R323.2, R331.2, R361.2, U301.25 (NC), U301.26 (NC), U301.27 (NC), U301.28 (NC)
- new net: C322.2, R313.2, R323.2, R331.2, U301.25 (NC), U301.26 (NC), U301.27 (NC), U301.28 (NC)
Changed lines of the file:
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@@
     (pin "2")
   )
-  (symbol (lib_id "01dyn_lib:R0603_100k") (at 190.5 66.04 180) (unit 1)
+  (symbol (lib_name "R0603_100k_1") (lib_id "01dyn_lib:R0603_100k") (at 190.5 66.04 180) (unit 1)
     (in_bom yes) (on_board yes)
     (property "Reference" "R365" (id 0) (at 193.04 63.5 0)
@@
     (pin "2")
   )
-  (symbol (lib_id "01dyn_lib:R0603_10k") (at 74.93 82.55 90) (unit 1)
+  (symbol (lib_name "R0603_10k_4") (lib_id "01dyn_lib:R0603_10k") (at 74.93 82.55 90) (unit 1)
     (in_bom yes) (on_board yes)
     (property "Reference" "R332" (id 0) (at 77.47 82.55 0)
@@
     (pin "2")
   )
-  (symbol (lib_id "power:GND") (at 81.28 71.12 0) (unit 1)
+  (symbol (lib_id "01dyn_lib:GND_1") (at 81.28 71.12 0) (unit 1)
     (in_bom yes) (on_board yes) (fields_autoplaced)
     (property "Reference" "#PWR0101" (id 0) (at 81.28 77.47 0)
       (effects (font (size 1.27 1.27)) hide)
     )
-    (property "Value" "GND" (id 1) (at 81.28 74.93 0))
+    (property "Value" "GND_1" (id 1) (at 81.28 74.93 0))
     (property "Footprint" "" (id 2) (at 81.28 71.12 0)
       (effects (font (size 1.27 1.27)) hide)
@@
     (pin "1")
   )
-  (symbol (lib_id "01dyn_lib:R0603_10k") (at 68.58 82.55 90) (unit 1)
+  (symbol (lib_name "R0603_10k_3") (lib_id "01dyn_lib:R0603_10k") (at 68.58 82.55 90) (unit 1)
     (in_bom yes) (on_board yes)
     (property "Reference" "R313" (id 0) (at 69.85 77.47 0)
@@
     (pin "2")
   )
-  (symbol (lib_id "01dyn_lib:R0603_10k") (at 172.72 66.04 180) (unit 1)
+  (symbol (lib_name "R0603_10k_2") (lib_id "01dyn_lib:R0603_10k") (at 172.72 66.04 180) (unit 1)
     (in_bom yes) (on_board yes)
     (property "Reference" "R362" (id 0) (at 172.72 63.5 0)
@@
     (pin "2")
   )
-  (symbol (lib_id "power:GND") (at 86.36 123.19 0) (unit 1)
+  (symbol (lib_id "01dyn_lib:GND_1") (at 86.36 123.19 0) (unit 1)
     (in_bom yes) (on_board yes) (fields_autoplaced)
     (property "Reference" "#PWR0104" (id 0) (at 86.36 129.54 0)
       (effects (font (size 1.27 1.27)) hide)
     )
-    (property "Value" "GND" (id 1) (at 86.36 127 0))
+    (property "Value" "GND_1" (id 1) (at 86.36 127 0))
     (property "Footprint" "" (id 2) (at 86.36 123.19 0)
       (effects (font (size 1.27 1.27)) hide)
@@
     (pin "1")
   )
-  (symbol (lib_id "01dyn_lib:R0603_100k") (at 64.77 81.28 90) (unit 1)
+  (symbol (lib_name "R0603_100k_2") (lib_id "01dyn_lib:R0603_100k") (at 64.77 81.28 90) (unit 1)
     (in_bom yes) (on_board yes)
     (property "Reference" "R312" (id 0) (at 63.5 83.82 0)
@@
     (pin "2")
   )
-  (symbol (lib_id "power:GND") (at 118.11 63.5 0) (unit 1)
+  (symbol (lib_id "01dyn_lib:GND_1") (at 118.11 63.5 0) (unit 1)
     (in_bom yes) (on_board yes) (fields_autoplaced)
     (property "Reference" "#PWR0102" (id 0) (at 118.11 69.85 0)
       (effects (font (size 1.27 1.27)) hide)
     )
-    (property "Value" "GND" (id 1) (at 118.11 67.31 0))
+    (property "Value" "GND_1" (id 1) (at 118.11 67.31 0))
     (property "Footprint" "" (id 2) (at 118.11 63.5 0)
       (effects (font (size 1.27 1.27)) hide)
@@
     (pin "1")
   )
-  (symbol (lib_id "power:GND") (at 147.32 72.39 0) (unit 1)
+  (symbol (lib_id "01dyn_lib:GND_1") (at 147.32 72.39 0) (unit 1)
     (in_bom yes) (on_board yes) (fields_autoplaced)
     (property "Reference" "#PWR0103" (id 0) (at 147.32 78.74 0)
       (effects (font (size 1.27 1.27)) hide)
     )
-    (property "Value" "GND" (id 1) (at 147.32 76.2 0))
+    (property "Value" "GND_1" (id 1) (at 147.32 76.2 0))
     (property "Footprint" "" (id 2) (at 147.32 72.39 0)
       (effects (font (size 1.27 1.27)) hide)
@@
     (pin "1")
   )
-  (symbol (lib_id "01dyn_lib:R0603_100k") (at 64.77 69.85 90) (unit 1)
+  (symbol (lib_name "R0603_100k_3") (lib_id "01dyn_lib:R0603_100k") (at 64.77 69.85 90) (unit 1)
     (in_bom yes) (on_board yes)
     (property "Reference" "R311" (id 0) (at 63.5 63.5 0)
@@
     (pin "2")
   )
-  (symbol (lib_id "01dyn_lib:R0603_10k") (at 160.02 66.04 180) (unit 1)
+  (symbol (lib_name "R0603_10k_1") (lib_id "01dyn_lib:R0603_10k") (at 160.02 66.04 180) (unit 1)
     (in_bom yes) (on_board yes)
     (property "Reference" "R361" (id 0) (at 162.56 63.5 0)
@@
     )
     (property "Value" "R0603_DNP" (id 1) (at 144.272 57.277 0)
-      (effects (font (size 0.5 0.5)))
+      (effects (font (size 0.5 0.5)) hide)
     )
     (property "Footprint" "Resistor_SMD:R_0603_1608Metric_Pad0.98x0.95mm_HandSolder" (id 2) (at 147.32 52.07 0)
@@
     (pin "2")
   )
-  (symbol (lib_id "01dyn_lib:c0603_100v10n") (at 190.5 71.12 270) (unit 1)
+  (symbol (lib_name "c0603_100v10n_1") (lib_id "01dyn_lib:c0603_100v10n") (at 190.5 71.12 270) (unit 1)
     (in_bom yes) (on_board yes)
     (property "Reference" "C365" (id 0) (at 191.77 73.66 90)

Commit message: ix
Parts:
- C321: symbol 01dyn_lib:c0805_35v10u -> 1001_un:c0805_35v10u
- C322, C365: footprint Capacitor_SMD:C_0603_1608Metric -> 02_dyn_pcblib:C0603; symbol 01dyn_lib:c0603_100v10n -> 1001_un:c0603_100v10n
- C324: footprint Capacitor_SMD:C_0603_1608Metric -> 02_dyn_pcblib:C0603; symbol 01dyn_lib:c0603_50v1u -> 1001_un:c0603_50v1u
- C325: footprint Capacitor_SMD:C_0603_1608Metric -> 02_dyn_pcblib:C0603; symbol 01dyn_lib:c0603_50v0.1u -> 1001_un:c0603_50v0.1u
- C371: footprint Capacitor_SMD:C_0603_1608Metric -> 02_dyn_pcblib:C0603; symbol 01dyn_lib:c0603_10v3.3u -> 1001_un:c0603_10v3.3u
- D351: symbol 01dyn_lib:LED0603_red -> 1001_un:LED0603_red
- L371: symbol 01dyn_lib:L3.3uH_7.4x6.6mm_30mhO_9.5A -> 1001_un:L3.3uH_7.4x6.6mm_30mhO_9.5A
- R311, R312, R323, R365: footprint Resistor_SMD:R_0603_1608Metric -> 02_dyn_pcblib:C0603; symbol 01dyn_lib:R0603_100k -> 1001_un:R0603_100k
- R313, R332, R351, R361, R362: footprint Resistor_SMD:R_0603_1608Metric -> 02_dyn_pcblib:C0603; symbol 01dyn_lib:R0603_10k -> 1001_un:R0603_10k
- R331: footprint Resistor_SMD:R_0603_1608Metric -> 02_dyn_pcblib:C0603; symbol 01dyn_lib:R0603_49.9k -> 1001_un:R0603_49.9k
- R352: footprint Resistor_SMD:R_0603_1608Metric_Pad0.98x0.95mm_HandSolder -> 02_dyn_pcblib:C0603; symbol 01dyn_lib:R0603_DNP -> 1001_un:R0603_DNP
- R391: symbol 01dyn_lib:R1206_0.0 -> 1001_un:R1206_0.0
- U301: symbol 01dyn_lib:dcdc_lt8612x -> 1001_un:dcdc_lt8612x
Connections:
- net GND: now reaches C322.2, R313.2, R323.2, R331.2, U301.25 (NC), U301.26 (NC), U301.27 (NC), U301.28 (NC)
- net GND: now also C321.2, C324.1, C371.2, R361.2, U301.10 (PGND), U301.11 (GND), U301.12 (GND), U301.13 (GND), U301.14 (GND), U301.29 (GND), U301.30 (GND), U301.31 (GND), U301.32 (GND), U301.8 (PGND), U301.9 (PGND)

Commit message: x
Parts:
- added C372: c0805_DNP, 02_dyn_pcblib:C0805mix0603, symbol 1003_cap:c0805_DNP
- C321: symbol 1001_un:c0805_35v10u -> 1003_cap:c0805_35v10u
- C322, C365: symbol 1001_un:c0603_100v10n -> 1003_cap:c0603_100v10n
- C324: symbol 1001_un:c0603_50v1u -> 1003_cap:c0603_50v1u
- C325: symbol 1001_un:c0603_50v0.1u -> 1003_cap:c0603_50v0.1u
- C371: symbol 1001_un:c0603_10v3.3u -> 1003_cap:c0603_10v3.3u
- D351: symbol 1001_un:LED0603_red -> 1004_led_mos:LED0603_red
- R311, R312, R323, R365: symbol 1001_un:R0603_100k -> 1002_res:R0603_100k
- R313, R332, R351, R361, R362: symbol 1001_un:R0603_10k -> 1002_res:R0603_10k
- R331: symbol 1001_un:R0603_49.9k -> 1002_res:R0603_49.9k
- R352: symbol 1001_un:R0603_DNP -> 1002_res:R0603_DNP
- R391: symbol 1001_un:R1206_0.0 -> 1002_res:R1206_0.0
Connections:
- net GND: now also C372.1
- net at C365.2, C371.1, L371.2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: now also C372.2
Changed lines of the file:
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@@
   (junction (at 152.4 101.6) (diameter 0) (color 0 0 0 0)
   )
+  (junction (at 200.66 120.65) (diameter 0) (color 0 0 0 0)
+  )
   (junction (at 68.58 91.44) (diameter 0) (color 0 0 0 0)
   )
@@
   (junction (at 152.4 104.14) (diameter 0) (color 0 0 0 0)
   )
+  (junction (at 200.66 104.14) (diameter 0) (color 0 0 0 0)
+  )
   (junction (at 106.68 66.04) (diameter 0) (color 0 0 0 0)
   )
@@
     (stroke (width 0) (type default) (color 0 0 0 0))
   )
+  (wire (pts (xy 209.55 120.65) (xy 200.66 120.65))
+    (stroke (width 0) (type default) (color 0 0 0 0))
+  )
   (wire (pts (xy 137.16 81.28) (xy 139.7 81.28))
     (stroke (width 0) (type default) (color 0 0 0 0))
@@
     (stroke (width 0) (type default) (color 0 0 0 0))
   )
-  (wire (pts (xy 200.66 99.06) (xy 200.66 107.95))
+  (wire (pts (xy 200.66 99.06) (xy 200.66 104.14))
     (stroke (width 0) (type default) (color 0 0 0 0))
   )
@@
     (stroke (width 0) (type default) (color 0 0 0 0))
   )
+  (wire (pts (xy 209.55 115.57) (xy 209.55 120.65))
+    (stroke (width 0) (type default) (color 0 0 0 0))
+  )
   (wire (pts (xy 85.09 86.36) (xy 91.44 86.36))
     (stroke (width 0) (type default) (color 0 0 0 0))
@@
     (stroke (width 0) (type default) (color 0 0 0 0))
   )
+  (wire (pts (xy 209.55 104.14) (xy 200.66 104.14))
+    (stroke (width 0) (type default) (color 0 0 0 0))
+  )
   (polyline (pts (xy 205.74 59.69) (xy 205.74 77.47))
     (stroke (width 0) (type default) (color 0 0 0 0))
@@
     (stroke (width 0) (type default) (color 0 0 0 0))
   )
+  (wire (pts (xy 209.55 107.95) (xy 209.55 104.14))
+    (stroke (width 0) (type default) (color 0 0 0 0))
+  )
   (wire (pts (xy 74.93 76.2) (xy 74.93 78.74))
     (stroke (width 0) (type default) (color 0 0 0 0))
@@
   )
   (wire (pts (xy 88.9 77.47) (xy 88.9 83.82))
+    (stroke (width 0) (type default) (color 0 0 0 0))
+  )
+  (wire (pts (xy 200.66 104.14) (xy 200.66 107.95))
     (stroke (width 0) (type default) (color 0 0 0 0))
   )
@@
     )
   )
-  (symbol (lib_id "1001_un:LED0603_red") (at 86.36 55.88 180) (unit 1)
+  (symbol (lib_id "1004_led_mos:LED0603_red") (at 86.36 55.88 180) (unit 1)
     (in_bom yes) (on_board yes)
     (property "Reference" "D351" (id 0) (at 90.17 54.61 0))
@@
     (pin "2")
   )
-  (symbol (lib_id "1001_un:R0603_100k") (at 190.5 66.04 180) (unit 1)
+  (symbol (lib_id "1002_res:R0603_100k") (at 190.5 66.04 180) (unit 1)
     (in_bom yes) (on_board yes)
     (property "Reference" "R365" (id 0) (at 193.04 63.5 0)
@@
     (pin "2")
   )
-  (symbol (lib_id "1001_un:R0603_10k") (at 74.93 82.55 90) (unit 1)
+  (symbol (lib_id "1002_res:R0603_10k") (at 74.93 82.55 90) (unit 1)
     (in_bom yes) (on_board yes)
     (property "Reference" "R332" (id 0) (at 77.47 82.55 0)
@@
     (pin "1")
   )
-  (symbol (lib_id "1001_un:R0603_10k") (at 68.58 82.55 90) (unit 1)
+  (symbol (lib_id "1002_res:R0603_10k") (at 68.58 82.55 90) (unit 1)
     (in_bom yes) (on_board yes)
     (property "Reference" "R313" (id 0) (at 69.85 77.47 0)
@@
     (pin "2")
   )
-  (symbol (lib_id "1001_un:R0603_10k") (at 172.72 66.04 180) (unit 1)
+  (symbol (lib_id "1002_res:R0603_10k") (at 172.72 66.04 180) (unit 1)
     (in_bom yes) (on_board yes)
     (property "Reference" "R362" (id 0) (at 172.72 63.5 0)
@@
     (pin "2")
   )
-  (symbol (lib_id "1001_un:R1206_0.0") (at 170.18 35.56 180) (unit 1)
+  (symbol (lib_id "1002_res:R1206_0.0") (at 170.18 35.56 180) (unit 1)
     (in_bom yes) (on_board yes) (fields_autoplaced)
     (property "Reference" "R391" (id 0) (at 170.18 30.48 0)
@@
     (pin "2")
   )
-  (symbol (lib_id "1001_un:R0603_100k") (at 88.9 72.39 90) (unit 1)
+  (symbol (lib_id "1002_res:R0603_100k") (at 88.9 72.39 90) (unit 1)
     (in_bom yes) (on_board yes)
     (property "Reference" "R323" (id 0) (at 87.63 69.85 0)
@@
     (pin "2")
   )
-  (symbol (lib_id "1001_un:c0805_35v10u") (at 58.42 109.22 180) (unit 1)
+  (symbol (lib_id "1003_cap:c0805_35v10u") (at 58.42 109.22 180) (unit 1)
     (in_bom yes) (on_board yes)
     (property "Reference" "C321" (id 0) (at 60.96 111.76 0))
@@
     (pin "1")
   )
-  (symbol (lib_id "1001_un:R0603_100k") (at 64.77 81.28 90) (unit 1)
+  (symbol (lib_id "1002_res:R0603_100k") (at 64.77 81.28 90) (unit 1)
     (in_bom yes) (on_board yes)
     (property "Reference" "R312" (id 0) (at 63.5 83.82 0)
@@
     (pin "2")
   )
-  (symbol (lib_id "1001_un:c0603_10v3.3u") (at 200.66 111.76 180) (unit 1)
+  (symbol (lib_id "1003_cap:c0603_10v3.3u") (at 200.66 111.76 180) (unit 1)
     (in_bom yes) (on_board yes)
     (property "Reference" "C371" (id 0) (at 201.93 109.22 0)
@@
     (pin "2")
   )
-  (symbol (lib_id "1001_un:c0603_50v0.1u") (at 139.7 93.98 90) (unit 1)
+  (symbol (lib_id "1003_cap:c0603_50v0.1u") (at 139.7 93.98 90) (unit 1)
     (in_bom yes) (on_board yes)
     (property "Reference" "C325" (id 0) (at 144.78 92.71 90))
@@
     (pin "9")
   )
-  (symbol (lib_id "1001_un:R0603_10k") (at 106.68 55.88 180) (unit 1)
+  (symbol (lib_id "1003_cap:c0805_DNP") (at 209.55 111.76 0) (unit 1)
+    (in_bom yes) (on_board yes)
+    (property "Reference" "C372" (id 0) (at 213.36 111.125 0)
+      (effects (font (size 1.5 1.5)) (justify left))
+    )
+    (property "Value" "c0805_DNP" (id 1) (at 207.01 111.76 0)
+      (effects (font (size 0.5 0.5)) (justify left))
+    )
+    (property "Footprint" "02_dyn_pcblib:C0805mix0603" (id 2) (at 210.439 98.933 0)
+      (effects (font (size 1.27 1.27)) hide)
+    )
+    (property "Datasheet" "~" (id 3) (at 209.4865 111.8235 0)
+      (effects (font (size 1.27 1.27)) hide)
+    )
+    (property "PartNum" "c0805_DNP" (id 4) (at 209.042 96.266 0)
+      (effects (font (size 1.27 1.27)) hide)
+    )
+    (pin "1")
+    (pin "2")
+  )
+  (symbol (lib_id "1002_res:R0603_10k") (at 106.68 55.88 180) (unit 1)
     (in_bom yes) (on_board yes)
     (property "Reference" "R351" (id 0) (at 111.76 54.61 0)
@@
     (pin "2")
   )
-  (symbol (lib_id "1001_un:R0603_49.9k") (at 74.93 72.39 90) (unit 1)
+  (symbol (lib_id "1002_res:R0603_49.9k") (at 74.93 72.39 90) (unit 1)
     (in_bom yes) (on_board yes)
     (property "Reference" "R331" (id 0) (at 73.66 69.85 0)
@@
     (pin "1")
   )
-  (symbol (lib_id "1001_un:R0603_100k") (at 64.77 69.85 90) (unit 1)
+  (symbol (lib_id "1002_res:R0603_100k") (at 64.77 69.85 90) (unit 1)
     (in_bom yes) (on_board yes)
     (property "Reference" "R311" (id 0) (at 63.5 63.5 0)
@@
     (pin "2")
   )
-  (symbol (lib_id "1001_un:R0603_10k") (at 160.02 66.04 180) (unit 1)
+  (symbol (lib_id "1002_res:R0603_10k") (at 160.02 66.04 180) (unit 1)
     (in_bom yes) (on_board yes)
     (property "Reference" "R361" (id 0) (at 162.56 63.5 0)
@@
     (pin "2")
   )
-  (symbol (lib_id "1001_un:c0603_100v10n") (at 85.09 81.28 0) (unit 1)
+  (symbol (lib_id "1003_cap:c0603_100v10n") (at 85.09 81.28 0) (unit 1)
     (in_bom yes) (on_board yes)
     (property "Reference" "C322" (id 0) (at 85.09 85.09 0)
@@
     (pin "2")
   )
-  (symbol (lib_id "1001_un:R0603_DNP") (at 146.05 55.88 0) (unit 1)
+  (symbol (lib_id "1002_res:R0603_DNP") (at 146.05 55.88 0) (unit 1)
     (in_bom yes) (on_board yes)
     (property "Reference" "R352" (id 0) (at 151.13 54.61 0)
@@
     (pin "2")
   )
-  (symbol (lib_id "1001_un:c0603_100v10n") (at 190.5 71.12 270) (unit 1)
+  (symbol (lib_id "1003_cap:c0603_100v10n") (at 190.5 71.12 270) (unit 1)
     (in_bom yes) (on_board yes)
     (property "Reference" "C365" (id 0) (at 191.77 73.66 90)
@@
     (pin "2")
   )
-  (symbol (lib_id "1001_un:c0603_50v1u") (at 128.27 67.31 180) (unit 1)
+  (symbol (lib_id "1003_cap:c0603_50v1u") (at 128.27 67.31 180) (unit 1)
     (in_bom yes) (on_board yes)
     (property "Reference" "C324" (id 0) (at 130.81 69.85 0))

Commit message: x
Parts:
- L371: symbol 1001_un:L3.3uH_7.4x6.6mm_30mhO_9.5A -> 1006_Inductance:L3.3uH_7.4x6.6mm_30mhO_9.5A
- U301: symbol 1001_un:dcdc_lt8612x -> 1009_ic:dcdc_lt8612x
Changed lines of the file:
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@@
     (pin "2")
   )
-  (symbol (lib_id "1001_un:dcdc_lt8612x") (at 102.87 83.82 0) (unit 1)
+  (symbol (lib_id "1009_ic:dcdc_lt8612x") (at 102.87 83.82 0) (unit 1)
     (in_bom yes) (on_board yes)
     (property "Reference" "U301" (id 0) (at 93.98 80.01 0)
@@
       (effects (font (size 1.5 1.5)) (justify left))
     )
-    (property "Value" "c0805_DNP" (id 1) (at 207.01 111.76 0)
-      (effects (font (size 0.5 0.5)) (justify left))
+    (property "Value" "c0805_DNP" (id 1) (at 209.677 111.887 0)
+      (effects (font (size 0.5 0.5)))
     )
     (property "Footprint" "02_dyn_pcblib:C0805mix0603" (id 2) (at 210.439 98.933 0)
@@
     (pin "2")
   )
-  (symbol (lib_id "1001_un:L3.3uH_7.4x6.6mm_30mhO_9.5A") (at 181.61 99.06 0) (unit 1)
+  (symbol (lib_id "1006_Inductance:L3.3uH_7.4x6.6mm_30mhO_9.5A") (at 181.61 99.06 0) (unit 1)
     (in_bom yes) (on_board yes)
     (property "Reference" "L371" (id 0) (at 181.61 95.25 0)

Commit message: x
Changed lines of the file:
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@@
     )
     (property "Value" "R0603_DNP" (id 1) (at 144.272 57.277 0)
-      (effects (font (size 0.5 0.5)) hide)
+      (effects (font (size 0.5 0.5)))
     )
     (property "Footprint" "02_dyn_pcblib:C0603" (id 2) (at 147.32 52.07 0)
