File: kicad01_power_board_for_nuclear_team/003_dcdc_18v4a.kicad_sch (KiCad schematic)
At the start: 22 parts, among them U301 dcdc_lt8612x

Commit message: x
Parts:
- C321, C372: footprint 02_dyn_pcblib:C0805mix0603 -> 2004_cap:C0805mix0603
- C322, C324, C325, C365, C371, R311, R312, R313, R323, R331, R332, R351, R352, R361, R362, R365: footprint 02_dyn_pcblib:C0603 -> 2004_cap:C0603
- D351: footprint 02_dyn_pcblib:LED0603 -> 2007_LED:LED0603
- L371: footprint 02_dyn_pcblib:L7.1x6.6mm -> 2005_inductance:L7.1x6.6mm
- R391: footprint 02_dyn_pcblib:R1206mix0603 -> 2003_res:R1206mix0603
- U301: footprint 02_dyn_pcblib:QFN-28-1EP_3x6mm_P0.5mm_EP1.7x4.75mmX -> 2006_qfn:QFN-28-1EP_3x6mm_P0.5mm_EP1.7x4.75mmX
Changed lines of the file:
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@@
       (effects (font (size 0.5 0.5)) (justify left))
     )
-    (property "Footprint" "02_dyn_pcblib:LED0603" (id 2) (at 86.36 64.77 0)
+    (property "Footprint" "2007_LED:LED0603" (id 2) (at 86.36 64.77 0)
       (effects (font (size 1.27 1.27)) hide)
     )
@@
       (effects (font (size 0.5 0.5)))
     )
-    (property "Footprint" "02_dyn_pcblib:C0603" (id 2) (at 189.23 69.85 0)
+    (property "Footprint" "2004_cap:C0603" (id 2) (at 189.23 69.85 0)
       (effects (font (size 1.27 1.27)) hide)
     )
@@
       (effects (font (size 0.5 0.5)))
     )
-    (property "Footprint" "02_dyn_pcblib:C0603" (id 2) (at 71.12 81.28 0)
+    (property "Footprint" "2004_cap:C0603" (id 2) (at 71.12 81.28 0)
       (effects (font (size 1.27 1.27)) hide)
     )
@@
       (effects (font (size 0.5 0.5)))
     )
-    (property "Footprint" "02_dyn_pcblib:C0603" (id 2) (at 64.77 81.28 0)
+    (property "Footprint" "2004_cap:C0603" (id 2) (at 64.77 81.28 0)
       (effects (font (size 1.27 1.27)) hide)
     )
@@
       (effects (font (size 0.5 0.5)))
     )
-    (property "Footprint" "02_dyn_pcblib:C0603" (id 2) (at 171.45 69.85 0)
+    (property "Footprint" "2004_cap:C0603" (id 2) (at 171.45 69.85 0)
       (effects (font (size 1.27 1.27)) hide)
     )
@@
       (effects (font (size 0.5 0.5)))
     )
-    (property "Footprint" "02_dyn_pcblib:R1206mix0603" (id 2) (at 170.18 46.99 0)
+    (property "Footprint" "2003_res:R1206mix0603" (id 2) (at 170.18 46.99 0)
       (effects (font (size 1.27 1.27)) hide)
     )
@@
       (effects (font (size 0.5 0.5)))
     )
-    (property "Footprint" "02_dyn_pcblib:C0603" (id 2) (at 85.09 71.12 0)
+    (property "Footprint" "2004_cap:C0603" (id 2) (at 85.09 71.12 0)
       (effects (font (size 1.27 1.27)) hide)
     )
@@
       (effects (font (size 0.5 0.5)))
     )
-    (property "Footprint" "02_dyn_pcblib:C0805mix0603" (id 2) (at 57.531 122.047 0)
+    (property "Footprint" "2004_cap:C0805mix0603" (id 2) (at 57.531 122.047 0)
       (effects (font (size 1.27 1.27)) hide)
     )
@@
       (effects (font (size 0.5 0.5)))
     )
-    (property "Footprint" "02_dyn_pcblib:C0603" (id 2) (at 60.96 80.01 0)
+    (property "Footprint" "2004_cap:C0603" (id 2) (at 60.96 80.01 0)
       (effects (font (size 1.27 1.27)) hide)
     )
@@
       (effects (font (size 0.5 0.5)))
     )
-    (property "Footprint" "02_dyn_pcblib:C0603" (id 2) (at 199.771 124.587 0)
+    (property "Footprint" "2004_cap:C0603" (id 2) (at 199.771 124.587 0)
       (effects (font (size 1.27 1.27)) hide)
     )
@@
       (effects (font (size 0.5 0.5)))
     )
-    (property "Footprint" "02_dyn_pcblib:C0603" (id 2) (at 126.873 93.091 0)
+    (property "Footprint" "2004_cap:C0603" (id 2) (at 126.873 93.091 0)
       (effects (font (size 1.27 1.27)) hide)
     )
@@
     )
     (property "Value" "dcdc_lt8612x" (id 1) (at 106.68 97.79 0))
-    (property "Footprint" "02_dyn_pcblib:QFN-28-1EP_3x6mm_P0.5mm_EP1.7x4.75mmX" (id 2) (at 109.22 55.88 0)
+    (property "Footprint" "2006_qfn:QFN-28-1EP_3x6mm_P0.5mm_EP1.7x4.75mmX" (id 2) (at 109.22 55.88 0)
       (effects (font (size 1.27 1.27)) hide)
     )
@@
       (effects (font (size 0.5 0.5)))
     )
-    (property "Footprint" "02_dyn_pcblib:C0805mix0603" (id 2) (at 210.439 98.933 0)
+    (property "Footprint" "2004_cap:C0805mix0603" (id 2) (at 210.439 98.933 0)
       (effects (font (size 1.27 1.27)) hide)
     )
@@
       (effects (font (size 0.5 0.5)))
     )
-    (property "Footprint" "02_dyn_pcblib:C0603" (id 2) (at 105.41 59.69 0)
+    (property "Footprint" "2004_cap:C0603" (id 2) (at 105.41 59.69 0)
       (effects (font (size 1.27 1.27)) hide)
     )
@@
       (effects (font (size 0.5 0.5)))
     )
-    (property "Footprint" "02_dyn_pcblib:C0603" (id 2) (at 71.12 71.12 0)
+    (property "Footprint" "2004_cap:C0603" (id 2) (at 71.12 71.12 0)
       (effects (font (size 1.27 1.27)) hide)
     )
@@
       (effects (font (size 0.5 0.5)) (justify left))
     )
-    (property "Footprint" "02_dyn_pcblib:L7.1x6.6mm" (id 2) (at 180.34 88.9 0)
+    (property "Footprint" "2005_inductance:L7.1x6.6mm" (id 2) (at 180.34 88.9 0)
       (effects (font (size 1.27 1.27)) hide)
     )
@@
       (effects (font (size 0.5 0.5)))
     )
-    (property "Footprint" "02_dyn_pcblib:C0603" (id 2) (at 60.96 68.58 0)
+    (property "Footprint" "2004_cap:C0603" (id 2) (at 60.96 68.58 0)
       (effects (font (size 1.27 1.27)) hide)
     )
@@
       (effects (font (size 0.5 0.5)))
     )
-    (property "Footprint" "02_dyn_pcblib:C0603" (id 2) (at 158.75 69.85 0)
+    (property "Footprint" "2004_cap:C0603" (id 2) (at 158.75 69.85 0)
       (effects (font (size 1.27 1.27)) hide)
     )
@@
       (effects (font (size 0.5 0.5)))
     )
-    (property "Footprint" "02_dyn_pcblib:C0603" (id 2) (at 85.979 68.453 0)
+    (property "Footprint" "2004_cap:C0603" (id 2) (at 85.979 68.453 0)
       (effects (font (size 1.27 1.27)) hide)
     )
@@
       (effects (font (size 0.5 0.5)))
     )
-    (property "Footprint" "02_dyn_pcblib:C0603" (id 2) (at 147.32 52.07 0)
+    (property "Footprint" "2004_cap:C0603" (id 2) (at 147.32 52.07 0)
       (effects (font (size 1.27 1.27)) hide)
     )
@@
       (effects (font (size 0.5 0.5)))
     )
-    (property "Footprint" "02_dyn_pcblib:C0603" (id 2) (at 203.327 72.009 0)
+    (property "Footprint" "2004_cap:C0603" (id 2) (at 203.327 72.009 0)
       (effects (font (size 1.27 1.27)) hide)
     )
@@
       (effects (font (size 0.5 0.5)))
     )
-    (property "Footprint" "02_dyn_pcblib:C0603" (id 2) (at 127.381 80.137 0)
-      (effects (font (size 1.27 1.27)) hide)
-    )
+    (property "Footprint" "2004_cap:C0603" (id 2) (at 127.381 80.137 0)
+      (effects (font (size 1.27 1.27)) hide)
+    )

Commit message: x
Parts:
- R311, R312, R313, R323, R331, R332, R351, R352, R361, R362, R365: footprint 2004_cap:C0603 -> 2003_res:R0603
Connections:
- net Vena3: now reaches R312.1, R313.1, U301.4 (EN/UV)
Changed lines of the file:
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@@
   (junction (at 88.9 77.47) (diameter 0) (color 0 0 0 0)
   )
+  (junction (at 64.77 91.44) (diameter 0) (color 0 0 0 0)
+  )
   (junction (at 109.22 66.04) (diameter 0) (color 0 0 0 0)
   )
@@
   )
   (polyline (pts (xy 60.96 60.96) (xy 71.12 60.96))
+    (stroke (width 0) (type default) (color 0 0 0 0))
+  )
+  (wire (pts (xy 45.72 91.44) (xy 64.77 91.44))
     (stroke (width 0) (type default) (color 0 0 0 0))
   )
@@
     )
   )
+  (global_label "Vena3" (shape input) (at 45.72 91.44 180) (fields_autoplaced)
+    (effects (font (size 1.27 1.27)) (justify right))
+    (property "Intersheet References" "${INTERSHEET_REFS}" (id 0) (at 37.6221 91.3606 0)
+      (effects (font (size 1.27 1.27)) (justify right) hide)
+    )
+  )
   (global_label "Vgood3" (shape input) (at 139.7 81.28 0) (fields_autoplaced)
     (effects (font (size 1.27 1.27)) (justify left))
@@
       (effects (font (size 0.5 0.5)))
     )
-    (property "Footprint" "2004_cap:C0603" (id 2) (at 189.23 69.85 0)
+    (property "Footprint" "2003_res:R0603" (id 2) (at 189.23 69.85 0)
       (effects (font (size 1.27 1.27)) hide)
     )
@@
       (effects (font (size 0.5 0.5)))
     )
-    (property "Footprint" "2004_cap:C0603" (id 2) (at 71.12 81.28 0)
+    (property "Footprint" "2003_res:R0603" (id 2) (at 71.12 81.28 0)
       (effects (font (size 1.27 1.27)) hide)
     )
@@
       (effects (font (size 0.5 0.5)))
     )
-    (property "Footprint" "2004_cap:C0603" (id 2) (at 64.77 81.28 0)
+    (property "Footprint" "2003_res:R0603" (id 2) (at 64.77 81.28 0)
       (effects (font (size 1.27 1.27)) hide)
     )
@@
       (effects (font (size 0.5 0.5)))
     )
-    (property "Footprint" "2004_cap:C0603" (id 2) (at 171.45 69.85 0)
+    (property "Footprint" "2003_res:R0603" (id 2) (at 171.45 69.85 0)
       (effects (font (size 1.27 1.27)) hide)
     )
@@
       (effects (font (size 0.5 0.5)))
     )
-    (property "Footprint" "2004_cap:C0603" (id 2) (at 85.09 71.12 0)
+    (property "Footprint" "2003_res:R0603" (id 2) (at 85.09 71.12 0)
       (effects (font (size 1.27 1.27)) hide)
     )
@@
       (effects (font (size 0.5 0.5)))
     )
-    (property "Footprint" "2004_cap:C0603" (id 2) (at 60.96 80.01 0)
+    (property "Footprint" "2003_res:R0603" (id 2) (at 60.96 80.01 0)
       (effects (font (size 1.27 1.27)) hide)
     )
@@
       (effects (font (size 0.5 0.5)))
     )
-    (property "Footprint" "2004_cap:C0603" (id 2) (at 105.41 59.69 0)
+    (property "Footprint" "2003_res:R0603" (id 2) (at 105.41 59.69 0)
       (effects (font (size 1.27 1.27)) hide)
     )
@@
       (effects (font (size 0.5 0.5)))
     )
-    (property "Footprint" "2004_cap:C0603" (id 2) (at 71.12 71.12 0)
+    (property "Footprint" "2003_res:R0603" (id 2) (at 71.12 71.12 0)
       (effects (font (size 1.27 1.27)) hide)
     )
@@
       (effects (font (size 0.5 0.5)))
     )
-    (property "Footprint" "2004_cap:C0603" (id 2) (at 60.96 68.58 0)
+    (property "Footprint" "2003_res:R0603" (id 2) (at 60.96 68.58 0)
       (effects (font (size 1.27 1.27)) hide)
     )
@@
       (effects (font (size 0.5 0.5)))
     )
-    (property "Footprint" "2004_cap:C0603" (id 2) (at 158.75 69.85 0)
+    (property "Footprint" "2003_res:R0603" (id 2) (at 158.75 69.85 0)
       (effects (font (size 1.27 1.27)) hide)
     )
@@
       (effects (font (size 0.5 0.5)))
     )
-    (property "Footprint" "2004_cap:C0603" (id 2) (at 147.32 52.07 0)
-      (effects (font (size 1.27 1.27)) hide)
-    )
+    (property "Footprint" "2003_res:R0603" (id 2) (at 147.32 52.07 0)
+      (effects (font (size 1.27 1.27)) hide)
+    )
