File: kicad01_power_board_for_nuclear_team/004_dcdc_18v4a.kicad_sch (KiCad schematic)
At the start: 21 parts, among them U401 dcdc_lt8612x

Commit message: x
Connections:
- net GND: no longer names the net of C421.2, C471.2, U401.10 (PGND), U401.11 (GND), U401.12 (GND), U401.13 (GND), U401.14 (GND), U401.29 (GND), U401.30 (GND), U401.31 (GND), U401.32 (GND), U401.8 (PGND), U401.9 (PGND)
- net GND: no longer C422.2, C424.1, R413.2, R423.2, R431.2, R461.2, U401.25 (NC), U401.26 (NC), U401.27 (NC), U401.28 (NC)
- new net: C422.2, R413.2, R423.2, R431.2, U401.25 (NC), U401.26 (NC), U401.27 (NC), U401.28 (NC)
Changed lines of the file:
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@@
     (pin "2")
   )
-  (symbol (lib_id "power:GND") (at 88.9 80.01 0) (unit 1)
+  (symbol (lib_id "01dyn_lib:GND_1") (at 88.9 80.01 0) (unit 1)
     (in_bom yes) (on_board yes) (fields_autoplaced)
     (property "Reference" "#PWR0108" (id 0) (at 88.9 86.36 0)
       (effects (font (size 1.27 1.27)) hide)
     )
-    (property "Value" "GND" (id 1) (at 88.9 83.82 0))
+    (property "Value" "GND_1" (id 1) (at 88.9 83.82 0))
     (property "Footprint" "" (id 2) (at 88.9 80.01 0)
       (effects (font (size 1.27 1.27)) hide)
@@
     (pin "2")
   )
-  (symbol (lib_id "01dyn_lib:R0603_100k") (at 72.39 90.17 90) (unit 1)
+  (symbol (lib_name "R0603_100k_3") (lib_id "01dyn_lib:R0603_100k") (at 72.39 90.17 90) (unit 1)
     (in_bom yes) (on_board yes)
     (property "Reference" "R412" (id 0) (at 71.12 92.71 0)
@@
     (pin "2")
   )
-  (symbol (lib_id "power:GND") (at 125.73 72.39 0) (unit 1)
+  (symbol (lib_id "01dyn_lib:GND_1") (at 125.73 72.39 0) (unit 1)
     (in_bom yes) (on_board yes) (fields_autoplaced)
     (property "Reference" "#PWR0106" (id 0) (at 125.73 78.74 0)
       (effects (font (size 1.27 1.27)) hide)
     )
-    (property "Value" "GND" (id 1) (at 125.73 76.2 0))
+    (property "Value" "GND_1" (id 1) (at 125.73 76.2 0))
     (property "Footprint" "" (id 2) (at 125.73 72.39 0)
       (effects (font (size 1.27 1.27)) hide)
@@
       (effects (font (size 1.5 1.5)))
     )
-    (property "Value" "R1206_0.0" (id 1) (at 177.8 41.91 0)
+    (property "Value" "R1206_0.0" (id 1) (at 179.578 43.053 0)
       (effects (font (size 0.5 0.5)))
     )
@@
     (pin "2")
   )
-  (symbol (lib_id "01dyn_lib:R0603_100k") (at 96.52 81.28 90) (unit 1)
+  (symbol (lib_name "R0603_100k_2") (lib_id "01dyn_lib:R0603_100k") (at 96.52 81.28 90) (unit 1)
     (in_bom yes) (on_board yes)
     (property "Reference" "R423" (id 0) (at 95.25 78.74 0)
@@
     (pin "2")
   )
-  (symbol (lib_id "01dyn_lib:R0603_10k") (at 82.55 91.44 90) (unit 1)
+  (symbol (lib_name "R0603_10k_3") (lib_id "01dyn_lib:R0603_10k") (at 82.55 91.44 90) (unit 1)
     (in_bom yes) (on_board yes)
     (property "Reference" "R432" (id 0) (at 85.09 91.44 0)
@@
     (pin "2")
   )
-  (symbol (lib_id "01dyn_lib:R0603_10k") (at 167.64 74.93 180) (unit 1)
+  (symbol (lib_name "R0603_10k_1") (lib_id "01dyn_lib:R0603_10k") (at 167.64 74.93 180) (unit 1)
     (in_bom yes) (on_board yes)
     (property "Reference" "R461" (id 0) (at 170.18 72.39 0)
@@
     (pin "2")
   )
-  (symbol (lib_id "01dyn_lib:R0603_10k") (at 180.34 74.93 180) (unit 1)
+  (symbol (lib_name "R0603_10k_2") (lib_id "01dyn_lib:R0603_10k") (at 180.34 74.93 180) (unit 1)
     (in_bom yes) (on_board yes)
     (property "Reference" "R462" (id 0) (at 180.34 72.39 0)
@@
     (pin "2")
   )
-  (symbol (lib_id "power:GND") (at 154.94 81.28 0) (unit 1)
+  (symbol (lib_id "01dyn_lib:GND_1") (at 154.94 81.28 0) (unit 1)
     (in_bom yes) (on_board yes) (fields_autoplaced)
     (property "Reference" "#PWR0107" (id 0) (at 154.94 87.63 0)
       (effects (font (size 1.27 1.27)) hide)
     )
-    (property "Value" "GND" (id 1) (at 154.94 85.09 0))
+    (property "Value" "GND_1" (id 1) (at 154.94 85.09 0))
     (property "Footprint" "" (id 2) (at 154.94 81.28 0)
       (effects (font (size 1.27 1.27)) hide)
@@
     (pin "1")
   )
-  (symbol (lib_id "01dyn_lib:R0603_10k") (at 76.2 91.44 90) (unit 1)
+  (symbol (lib_name "R0603_10k_4") (lib_id "01dyn_lib:R0603_10k") (at 76.2 91.44 90) (unit 1)
     (in_bom yes) (on_board yes)
     (property "Reference" "R413" (id 0) (at 77.47 86.36 0)
@@
     (pin "2")
   )
-  (symbol (lib_id "01dyn_lib:c0603_100v10n") (at 198.12 80.01 270) (unit 1)
+  (symbol (lib_name "c0603_100v10n_1") (lib_id "01dyn_lib:c0603_100v10n") (at 198.12 80.01 270) (unit 1)
     (in_bom yes) (on_board yes)
     (property "Reference" "C465" (id 0) (at 199.39 82.55 90)
@@
     )
     (property "Value" "R0603_DNP" (id 1) (at 151.892 66.167 0)
-      (effects (font (size 0.5 0.5)))
+      (effects (font (size 0.5 0.5)) hide)
     )
     (property "Footprint" "Resistor_SMD:R_0603_1608Metric_Pad0.98x0.95mm_HandSolder" (id 2) (at 154.94 60.96 0)
@@
     (pin "2")
   )
-  (symbol (lib_id "01dyn_lib:R0603_100k") (at 198.12 74.93 180) (unit 1)
+  (symbol (lib_name "R0603_100k_1") (lib_id "01dyn_lib:R0603_100k") (at 198.12 74.93 180) (unit 1)
     (in_bom yes) (on_board yes)
     (property "Reference" "R465" (id 0) (at 200.66 72.39 0)
@@
     (pin "2")
   )
-  (symbol (lib_id "power:GND") (at 93.98 132.08 0) (unit 1)
+  (symbol (lib_id "01dyn_lib:GND_1") (at 93.98 132.08 0) (unit 1)
     (in_bom yes) (on_board yes) (fields_autoplaced)
     (property "Reference" "#PWR0105" (id 0) (at 93.98 138.43 0)
       (effects (font (size 1.27 1.27)) hide)
     )
-    (property "Value" "GND" (id 1) (at 93.98 135.89 0))
+    (property "Value" "GND_1" (id 1) (at 93.98 135.89 0))
     (property "Footprint" "" (id 2) (at 93.98 132.08 0)
       (effects (font (size 1.27 1.27)) hide)

Commit message: ix
Parts:
- C421: symbol 01dyn_lib:c0805_35v10u -> 1001_un:c0805_35v10u
- C422, C465: footprint Capacitor_SMD:C_0603_1608Metric -> 02_dyn_pcblib:C0603; symbol 01dyn_lib:c0603_100v10n -> 1001_un:c0603_100v10n
- C424: footprint Capacitor_SMD:C_0603_1608Metric -> 02_dyn_pcblib:C0603; symbol 01dyn_lib:c0603_50v1u -> 1001_un:c0603_50v1u
- C425: footprint Capacitor_SMD:C_0603_1608Metric -> 02_dyn_pcblib:C0603; symbol 01dyn_lib:c0603_50v0.1u -> 1001_un:c0603_50v0.1u
- C471: footprint Capacitor_SMD:C_0603_1608Metric -> 02_dyn_pcblib:C0603; symbol 01dyn_lib:c0603_10v3.3u -> 1001_un:c0603_10v3.3u
- D451: symbol 01dyn_lib:LED0603_red -> 1001_un:LED0603_red
- L471: symbol 01dyn_lib:L3.3uH_7.4x6.6mm_30mhO_9.5A -> 1001_un:L3.3uH_7.4x6.6mm_30mhO_9.5A
- R411, R412, R423, R465: footprint Resistor_SMD:R_0603_1608Metric -> 02_dyn_pcblib:C0603; symbol 01dyn_lib:R0603_100k -> 1001_un:R0603_100k
- R413, R432, R451, R461, R462: footprint Resistor_SMD:R_0603_1608Metric -> 02_dyn_pcblib:C0603; symbol 01dyn_lib:R0603_10k -> 1001_un:R0603_10k
- R431: footprint Resistor_SMD:R_0603_1608Metric -> 02_dyn_pcblib:C0603; symbol 01dyn_lib:R0603_49.9k -> 1001_un:R0603_49.9k
- R452: footprint Resistor_SMD:R_0603_1608Metric_Pad0.98x0.95mm_HandSolder -> 02_dyn_pcblib:C0603; symbol 01dyn_lib:R0603_DNP -> 1001_un:R0603_DNP
- R491: symbol 01dyn_lib:R1206_0.0 -> 1001_un:R1206_0.0
- U401: symbol 01dyn_lib:dcdc_lt8612x -> 1001_un:dcdc_lt8612x
Connections:
- net GND: now reaches C424.1
- net GND: now also C421.2, C422.2, C471.2, R413.2, R423.2, R431.2, R461.2, U401.10 (PGND), U401.11 (GND), U401.12 (GND), U401.13 (GND), U401.14 (GND), U401.25 (NC), U401.26 (NC), U401.27 (NC), U401.28 (NC), U401.29 (GND), U401.30 (GND), U401.31 (GND), U401.32 (GND), U401.8 (PGND), U401.9 (PGND)

Commit message: x
Parts:
- added C472: c0805_DNP, 02_dyn_pcblib:C0805mix0603, symbol 1003_cap:c0805_DNP
- C421: symbol 1001_un:c0805_35v10u -> 1003_cap:c0805_35v10u
- C422, C465: symbol 1001_un:c0603_100v10n -> 1003_cap:c0603_100v10n
- C424: symbol 1001_un:c0603_50v1u -> 1003_cap:c0603_50v1u
- C425: symbol 1001_un:c0603_50v0.1u -> 1003_cap:c0603_50v0.1u
- C471: symbol 1001_un:c0603_10v3.3u -> 1003_cap:c0603_10v3.3u
- D451: symbol 1001_un:LED0603_red -> 1004_led_mos:LED0603_red
- R411, R412, R423, R465: symbol 1001_un:R0603_100k -> 1002_res:R0603_100k
- R413, R432, R451, R461, R462: symbol 1001_un:R0603_10k -> 1002_res:R0603_10k
- R431: symbol 1001_un:R0603_49.9k -> 1002_res:R0603_49.9k
- R452: symbol 1001_un:R0603_DNP -> 1002_res:R0603_DNP
- R491: symbol 1001_un:R1206_0.0 -> 1002_res:R1206_0.0
Connections:
- net GND: now also C472.1
- net at C465.2, C471.1, L471.2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: now also C472.2
Changed lines of the file:
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@@
   (junction (at 119.38 74.93) (diameter 0) (color 0 0 0 0)
   )
+  (junction (at 208.28 111.76) (diameter 0) (color 0 0 0 0)
+  )
   (junction (at 66.04 64.77) (diameter 0) (color 0 0 0 0)
   )
@@
   (junction (at 208.28 107.95) (diameter 0) (color 0 0 0 0)
   )
+  (junction (at 208.28 129.54) (diameter 0) (color 0 0 0 0)
+  )
   (wire (pts (xy 109.22 124.46) (xy 109.22 129.54))
     (stroke (width 0) (type default) (color 0 0 0 0))
@@
     (stroke (width 0) (type default) (color 0 0 0 0))
   )
-  (wire (pts (xy 208.28 107.95) (xy 208.28 116.84))
+  (wire (pts (xy 208.28 107.95) (xy 208.28 111.76))
     (stroke (width 0) (type default) (color 0 0 0 0))
   )
@@
     (stroke (width 0) (type default) (color 0 0 0 0))
   )
+  (wire (pts (xy 217.17 116.84) (xy 217.17 111.76))
+    (stroke (width 0) (type default) (color 0 0 0 0))
+  )
+  (wire (pts (xy 208.28 111.76) (xy 208.28 116.84))
+    (stroke (width 0) (type default) (color 0 0 0 0))
+  )
   (wire (pts (xy 116.84 74.93) (xy 116.84 87.63))
     (stroke (width 0) (type default) (color 0 0 0 0))
@@
     (stroke (width 0) (type default) (color 0 0 0 0))
   )
+  (wire (pts (xy 208.28 111.76) (xy 217.17 111.76))
+    (stroke (width 0) (type default) (color 0 0 0 0))
+  )
   (wire (pts (xy 119.38 129.54) (xy 121.92 129.54))
     (stroke (width 0) (type default) (color 0 0 0 0))
@@
     (stroke (width 0) (type default) (color 0 0 0 0))
   )
+  (wire (pts (xy 217.17 124.46) (xy 217.17 129.54))
+    (stroke (width 0) (type default) (color 0 0 0 0))
+  )
   (wire (pts (xy 181.61 44.45) (xy 208.28 44.45))
     (stroke (width 0) (type default) (color 0 0 0 0))
   )
   (polyline (pts (xy 73.66 66.04) (xy 76.2 69.85))
+    (stroke (width 0) (type default) (color 0 0 0 0))
+  )
+  (wire (pts (xy 217.17 129.54) (xy 208.28 129.54))
     (stroke (width 0) (type default) (color 0 0 0 0))
   )
@@
     )
   )
-  (symbol (lib_id "1001_un:c0603_50v1u") (at 135.89 76.2 180) (unit 1)
+  (symbol (lib_id "1003_cap:c0603_50v1u") (at 135.89 76.2 180) (unit 1)
     (in_bom yes) (on_board yes)
     (property "Reference" "C424" (id 0) (at 138.43 78.74 0))
@@
     (pin "1")
   )
-  (symbol (lib_id "1001_un:c0603_10v3.3u") (at 208.28 120.65 180) (unit 1)
+  (symbol (lib_id "1003_cap:c0603_10v3.3u") (at 208.28 120.65 180) (unit 1)
     (in_bom yes) (on_board yes)
     (property "Reference" "C471" (id 0) (at 209.55 118.11 0)
@@
     (pin "2")
   )
-  (symbol (lib_id "1001_un:R0603_10k") (at 114.3 64.77 180) (unit 1)
+  (symbol (lib_id "1002_res:R0603_10k") (at 114.3 64.77 180) (unit 1)
     (in_bom yes) (on_board yes)
     (property "Reference" "R451" (id 0) (at 119.38 63.5 0)
@@
     (pin "2")
   )
-  (symbol (lib_id "1001_un:R0603_100k") (at 72.39 90.17 90) (unit 1)
+  (symbol (lib_id "1002_res:R0603_100k") (at 72.39 90.17 90) (unit 1)
     (in_bom yes) (on_board yes)
     (property "Reference" "R412" (id 0) (at 71.12 92.71 0)
@@
     (pin "2")
   )
-  (symbol (lib_id "1001_un:c0805_35v10u") (at 66.04 118.11 180) (unit 1)
+  (symbol (lib_id "1003_cap:c0805_35v10u") (at 66.04 118.11 180) (unit 1)
     (in_bom yes) (on_board yes)
     (property "Reference" "C421" (id 0) (at 68.58 120.65 0))
@@
     (pin "1")
   )
-  (symbol (lib_id "1001_un:R1206_0.0") (at 177.8 44.45 180) (unit 1)
+  (symbol (lib_id "1002_res:R1206_0.0") (at 177.8 44.45 180) (unit 1)
     (in_bom yes) (on_board yes) (fields_autoplaced)
     (property "Reference" "R491" (id 0) (at 177.8 39.37 0)
@@
     (pin "2")
   )
-  (symbol (lib_id "1001_un:R0603_100k") (at 96.52 81.28 90) (unit 1)
+  (symbol (lib_id "1002_res:R0603_100k") (at 96.52 81.28 90) (unit 1)
     (in_bom yes) (on_board yes)
     (property "Reference" "R423" (id 0) (at 95.25 78.74 0)
@@
     (pin "2")
   )
-  (symbol (lib_id "1001_un:R0603_10k") (at 82.55 91.44 90) (unit 1)
+  (symbol (lib_id "1002_res:R0603_10k") (at 82.55 91.44 90) (unit 1)
     (in_bom yes) (on_board yes)
     (property "Reference" "R432" (id 0) (at 85.09 91.44 0)
@@
     (pin "2")
   )
-  (symbol (lib_id "1001_un:R0603_49.9k") (at 82.55 81.28 90) (unit 1)
+  (symbol (lib_id "1002_res:R0603_49.9k") (at 82.55 81.28 90) (unit 1)
     (in_bom yes) (on_board yes)
     (property "Reference" "R431" (id 0) (at 81.28 78.74 0)
@@
     (pin "2")
   )
-  (symbol (lib_id "1001_un:R0603_100k") (at 72.39 78.74 90) (unit 1)
+  (symbol (lib_id "1002_res:R0603_100k") (at 72.39 78.74 90) (unit 1)
     (in_bom yes) (on_board yes)
     (property "Reference" "R411" (id 0) (at 71.12 72.39 0)
@@
     (pin "9")
   )
-  (symbol (lib_id "1001_un:c0603_100v10n") (at 92.71 90.17 0) (unit 1)
+  (symbol (lib_id "1003_cap:c0603_100v10n") (at 92.71 90.17 0) (unit 1)
     (in_bom yes) (on_board yes)
     (property "Reference" "C422" (id 0) (at 92.71 93.98 0)
@@
     (pin "2")
   )
-  (symbol (lib_id "1001_un:R0603_10k") (at 167.64 74.93 180) (unit 1)
+  (symbol (lib_id "1003_cap:c0805_DNP") (at 217.17 120.65 0) (unit 1)
+    (in_bom yes) (on_board yes)
+    (property "Reference" "C472" (id 0) (at 220.98 120.015 0)
+      (effects (font (size 1.5 1.5)) (justify left))
+    )
+    (property "Value" "c0805_DNP" (id 1) (at 214.63 120.65 0)
+      (effects (font (size 0.5 0.5)) (justify left))
+    )
+    (property "Footprint" "02_dyn_pcblib:C0805mix0603" (id 2) (at 218.059 107.823 0)
+      (effects (font (size 1.27 1.27)) hide)
+    )
+    (property "Datasheet" "~" (id 3) (at 217.1065 120.7135 0)
+      (effects (font (size 1.27 1.27)) hide)
+    )
+    (property "PartNum" "c0805_DNP" (id 4) (at 216.662 105.156 0)
+      (effects (font (size 1.27 1.27)) hide)
+    )
+    (pin "1")
+    (pin "2")
+  )
+  (symbol (lib_id "1002_res:R0603_10k") (at 167.64 74.93 180) (unit 1)
     (in_bom yes) (on_board yes)
     (property "Reference" "R461" (id 0) (at 170.18 72.39 0)
@@
     (pin "2")
   )
-  (symbol (lib_id "1001_un:R0603_10k") (at 180.34 74.93 180) (unit 1)
+  (symbol (lib_id "1002_res:R0603_10k") (at 180.34 74.93 180) (unit 1)
     (in_bom yes) (on_board yes)
     (property "Reference" "R462" (id 0) (at 180.34 72.39 0)
@@
     (pin "2")
   )
-  (symbol (lib_id "1001_un:LED0603_red") (at 93.98 64.77 180) (unit 1)
+  (symbol (lib_id "1004_led_mos:LED0603_red") (at 93.98 64.77 180) (unit 1)
     (in_bom yes) (on_board yes)
     (property "Reference" "D451" (id 0) (at 97.79 63.5 0))
@@
     (pin "1")
   )
-  (symbol (lib_id "1001_un:R0603_10k") (at 76.2 91.44 90) (unit 1)
+  (symbol (lib_id "1002_res:R0603_10k") (at 76.2 91.44 90) (unit 1)
     (in_bom yes) (on_board yes)
     (property "Reference" "R413" (id 0) (at 77.47 86.36 0)
@@
     (pin "2")
   )
-  (symbol (lib_id "1001_un:c0603_100v10n") (at 198.12 80.01 270) (unit 1)
+  (symbol (lib_id "1003_cap:c0603_100v10n") (at 198.12 80.01 270) (unit 1)
     (in_bom yes) (on_board yes)
     (property "Reference" "C465" (id 0) (at 199.39 82.55 90)
@@
     (pin "2")
   )
-  (symbol (lib_id "1001_un:R0603_DNP") (at 153.67 64.77 0) (unit 1)
+  (symbol (lib_id "1002_res:R0603_DNP") (at 153.67 64.77 0) (unit 1)
     (in_bom yes) (on_board yes)
     (property "Reference" "R452" (id 0) (at 158.75 63.5 0)
@@
     (pin "2")
   )
-  (symbol (lib_id "1001_un:R0603_100k") (at 198.12 74.93 180) (unit 1)
+  (symbol (lib_id "1002_res:R0603_100k") (at 198.12 74.93 180) (unit 1)
     (in_bom yes) (on_board yes)
     (property "Reference" "R465" (id 0) (at 200.66 72.39 0)
@@
     (pin "1")
   )
-  (symbol (lib_id "1001_un:c0603_50v0.1u") (at 147.32 102.87 90) (unit 1)
+  (symbol (lib_id "1003_cap:c0603_50v0.1u") (at 147.32 102.87 90) (unit 1)
     (in_bom yes) (on_board yes)
     (property "Reference" "C425" (id 0) (at 152.4 101.6 90))

Commit message: x
Parts:
- L471: symbol 1001_un:L3.3uH_7.4x6.6mm_30mhO_9.5A -> 1006_Inductance:L3.3uH_7.4x6.6mm_30mhO_9.5A
- U401: symbol 1001_un:dcdc_lt8612x -> 1009_ic:dcdc_lt8612x
Changed lines of the file:
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@@
     (pin "2")
   )
-  (symbol (lib_id "1001_un:dcdc_lt8612x") (at 110.49 92.71 0) (unit 1)
+  (symbol (lib_id "1009_ic:dcdc_lt8612x") (at 110.49 92.71 0) (unit 1)
     (in_bom yes) (on_board yes)
     (property "Reference" "U401" (id 0) (at 101.6 88.9 0)
@@
       (effects (font (size 1.5 1.5)) (justify left))
     )
-    (property "Value" "c0805_DNP" (id 1) (at 214.63 120.65 0)
-      (effects (font (size 0.5 0.5)) (justify left))
+    (property "Value" "c0805_DNP" (id 1) (at 217.297 120.777 0)
+      (effects (font (size 0.5 0.5)))
     )
     (property "Footprint" "02_dyn_pcblib:C0805mix0603" (id 2) (at 218.059 107.823 0)
@@
     (pin "2")
   )
-  (symbol (lib_id "1001_un:L3.3uH_7.4x6.6mm_30mhO_9.5A") (at 189.23 107.95 0) (unit 1)
+  (symbol (lib_id "1006_Inductance:L3.3uH_7.4x6.6mm_30mhO_9.5A") (at 189.23 107.95 0) (unit 1)
     (in_bom yes) (on_board yes)
     (property "Reference" "L471" (id 0) (at 189.23 104.14 0)

Commit message: x
Changed lines of the file:
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@@
     )
     (property "Value" "R0603_DNP" (id 1) (at 151.892 66.167 0)
-      (effects (font (size 0.5 0.5)) hide)
+      (effects (font (size 0.5 0.5)))
     )
     (property "Footprint" "02_dyn_pcblib:C0603" (id 2) (at 154.94 60.96 0)
