File: kicad01_power_board_for_nuclear_team/004_dcdc_18v4a.kicad_sch (KiCad schematic)
At the start: 22 parts, among them U401 dcdc_lt8612x

Commit message: x
Parts:
- C421, C472: footprint 02_dyn_pcblib:C0805mix0603 -> 2004_cap:C0805mix0603
- C422, C424, C425, C465, C471, R411, R412, R413, R423, R431, R432, R451, R452, R461, R462, R465: footprint 02_dyn_pcblib:C0603 -> 2004_cap:C0603
- D451: footprint 02_dyn_pcblib:LED0603 -> 2007_LED:LED0603
- L471: footprint 02_dyn_pcblib:L7.1x6.6mm -> 2005_inductance:L7.1x6.6mm
- R491: footprint 02_dyn_pcblib:R1206mix0603 -> 2003_res:R1206mix0603
- U401: footprint 02_dyn_pcblib:QFN-28-1EP_3x6mm_P0.5mm_EP1.7x4.75mmX -> 2006_qfn:QFN-28-1EP_3x6mm_P0.5mm_EP1.7x4.75mmX
Changed lines of the file:
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@@
       (effects (font (size 0.5 0.5)))
     )
-    (property "Footprint" "02_dyn_pcblib:C0603" (id 2) (at 135.001 89.027 0)
+    (property "Footprint" "2004_cap:C0603" (id 2) (at 135.001 89.027 0)
       (effects (font (size 1.27 1.27)) hide)
     )
@@
       (effects (font (size 0.5 0.5)))
     )
-    (property "Footprint" "02_dyn_pcblib:C0603" (id 2) (at 207.391 133.477 0)
+    (property "Footprint" "2004_cap:C0603" (id 2) (at 207.391 133.477 0)
       (effects (font (size 1.27 1.27)) hide)
     )
@@
       (effects (font (size 0.5 0.5)))
     )
-    (property "Footprint" "02_dyn_pcblib:C0603" (id 2) (at 113.03 68.58 0)
+    (property "Footprint" "2004_cap:C0603" (id 2) (at 113.03 68.58 0)
       (effects (font (size 1.27 1.27)) hide)
     )
@@
       (effects (font (size 0.5 0.5)))
     )
-    (property "Footprint" "02_dyn_pcblib:C0603" (id 2) (at 68.58 88.9 0)
+    (property "Footprint" "2004_cap:C0603" (id 2) (at 68.58 88.9 0)
       (effects (font (size 1.27 1.27)) hide)
     )
@@
       (effects (font (size 0.5 0.5)))
     )
-    (property "Footprint" "02_dyn_pcblib:C0805mix0603" (id 2) (at 65.151 130.937 0)
+    (property "Footprint" "2004_cap:C0805mix0603" (id 2) (at 65.151 130.937 0)
       (effects (font (size 1.27 1.27)) hide)
     )
@@
       (effects (font (size 0.5 0.5)))
     )
-    (property "Footprint" "02_dyn_pcblib:R1206mix0603" (id 2) (at 177.8 55.88 0)
+    (property "Footprint" "2003_res:R1206mix0603" (id 2) (at 177.8 55.88 0)
       (effects (font (size 1.27 1.27)) hide)
     )
@@
       (effects (font (size 0.5 0.5)))
     )
-    (property "Footprint" "02_dyn_pcblib:C0603" (id 2) (at 92.71 80.01 0)
+    (property "Footprint" "2004_cap:C0603" (id 2) (at 92.71 80.01 0)
       (effects (font (size 1.27 1.27)) hide)
     )
@@
       (effects (font (size 0.5 0.5)))
     )
-    (property "Footprint" "02_dyn_pcblib:C0603" (id 2) (at 78.74 90.17 0)
+    (property "Footprint" "2004_cap:C0603" (id 2) (at 78.74 90.17 0)
       (effects (font (size 1.27 1.27)) hide)
     )
@@
       (effects (font (size 0.5 0.5)))
     )
-    (property "Footprint" "02_dyn_pcblib:C0603" (id 2) (at 78.74 80.01 0)
+    (property "Footprint" "2004_cap:C0603" (id 2) (at 78.74 80.01 0)
       (effects (font (size 1.27 1.27)) hide)
     )
@@
       (effects (font (size 0.5 0.5)))
     )
-    (property "Footprint" "02_dyn_pcblib:C0603" (id 2) (at 68.58 77.47 0)
+    (property "Footprint" "2004_cap:C0603" (id 2) (at 68.58 77.47 0)
       (effects (font (size 1.27 1.27)) hide)
     )
@@
     )
     (property "Value" "dcdc_lt8612x" (id 1) (at 114.3 106.68 0))
-    (property "Footprint" "02_dyn_pcblib:QFN-28-1EP_3x6mm_P0.5mm_EP1.7x4.75mmX" (id 2) (at 116.84 64.77 0)
+    (property "Footprint" "2006_qfn:QFN-28-1EP_3x6mm_P0.5mm_EP1.7x4.75mmX" (id 2) (at 116.84 64.77 0)
       (effects (font (size 1.27 1.27)) hide)
     )
@@
       (effects (font (size 0.5 0.5)))
     )
-    (property "Footprint" "02_dyn_pcblib:C0603" (id 2) (at 93.599 77.343 0)
+    (property "Footprint" "2004_cap:C0603" (id 2) (at 93.599 77.343 0)
       (effects (font (size 1.27 1.27)) hide)
     )
@@
       (effects (font (size 0.5 0.5)))
     )
-    (property "Footprint" "02_dyn_pcblib:C0805mix0603" (id 2) (at 218.059 107.823 0)
+    (property "Footprint" "2004_cap:C0805mix0603" (id 2) (at 218.059 107.823 0)
       (effects (font (size 1.27 1.27)) hide)
     )
@@
       (effects (font (size 0.5 0.5)))
     )
-    (property "Footprint" "02_dyn_pcblib:C0603" (id 2) (at 166.37 78.74 0)
+    (property "Footprint" "2004_cap:C0603" (id 2) (at 166.37 78.74 0)
       (effects (font (size 1.27 1.27)) hide)
     )
@@
       (effects (font (size 0.5 0.5)))
     )
-    (property "Footprint" "02_dyn_pcblib:C0603" (id 2) (at 179.07 78.74 0)
+    (property "Footprint" "2004_cap:C0603" (id 2) (at 179.07 78.74 0)
       (effects (font (size 1.27 1.27)) hide)
     )
@@
       (effects (font (size 0.5 0.5)) (justify left))
     )
-    (property "Footprint" "02_dyn_pcblib:LED0603" (id 2) (at 93.98 73.66 0)
+    (property "Footprint" "2007_LED:LED0603" (id 2) (at 93.98 73.66 0)
       (effects (font (size 1.27 1.27)) hide)
     )
@@
       (effects (font (size 0.5 0.5)))
     )
-    (property "Footprint" "02_dyn_pcblib:C0603" (id 2) (at 72.39 90.17 0)
+    (property "Footprint" "2004_cap:C0603" (id 2) (at 72.39 90.17 0)
       (effects (font (size 1.27 1.27)) hide)
     )
@@
       (effects (font (size 0.5 0.5)))
     )
-    (property "Footprint" "02_dyn_pcblib:C0603" (id 2) (at 210.947 80.899 0)
+    (property "Footprint" "2004_cap:C0603" (id 2) (at 210.947 80.899 0)
       (effects (font (size 1.27 1.27)) hide)
     )
@@
       (effects (font (size 0.5 0.5)))
     )
-    (property "Footprint" "02_dyn_pcblib:C0603" (id 2) (at 154.94 60.96 0)
+    (property "Footprint" "2004_cap:C0603" (id 2) (at 154.94 60.96 0)
       (effects (font (size 1.27 1.27)) hide)
     )
@@
       (effects (font (size 0.5 0.5)) (justify left))
     )
-    (property "Footprint" "02_dyn_pcblib:L7.1x6.6mm" (id 2) (at 187.96 97.79 0)
+    (property "Footprint" "2005_inductance:L7.1x6.6mm" (id 2) (at 187.96 97.79 0)
       (effects (font (size 1.27 1.27)) hide)
     )
@@
       (effects (font (size 0.5 0.5)))
     )
-    (property "Footprint" "02_dyn_pcblib:C0603" (id 2) (at 196.85 78.74 0)
+    (property "Footprint" "2004_cap:C0603" (id 2) (at 196.85 78.74 0)
       (effects (font (size 1.27 1.27)) hide)
     )
@@
       (effects (font (size 0.5 0.5)))
     )
-    (property "Footprint" "02_dyn_pcblib:C0603" (id 2) (at 134.493 101.981 0)
-      (effects (font (size 1.27 1.27)) hide)
-    )
+    (property "Footprint" "2004_cap:C0603" (id 2) (at 134.493 101.981 0)
+      (effects (font (size 1.27 1.27)) hide)
+    )

Commit message: x
Parts:
- R411, R412, R413, R423, R431, R432, R451, R452, R461, R462, R465: footprint 2004_cap:C0603 -> 2003_res:R0603
Connections:
- net Vena4: now reaches R412.1, R413.1, U401.4 (EN/UV)
Changed lines of the file:
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@@
   (junction (at 93.98 115.57) (diameter 0) (color 0 0 0 0)
   )
+  (junction (at 72.39 100.33) (diameter 0) (color 0 0 0 0)
+  )
   (junction (at 160.02 105.41) (diameter 0) (color 0 0 0 0)
   )
@@
   )
   (polyline (pts (xy 77.47 66.04) (xy 77.47 60.96))
+    (stroke (width 0) (type default) (color 0 0 0 0))
+  )
+  (wire (pts (xy 57.15 100.33) (xy 72.39 100.33))
     (stroke (width 0) (type default) (color 0 0 0 0))
   )
@@
     )
   )
+  (global_label "Vena4" (shape input) (at 57.15 100.33 180) (fields_autoplaced)
+    (effects (font (size 1.27 1.27)) (justify right))
+    (property "Intersheet References" "${INTERSHEET_REFS}" (id 0) (at 49.0521 100.2506 0)
+      (effects (font (size 1.27 1.27)) (justify right) hide)
+    )
+  )
   (global_label "Vsync4" (shape input) (at 100.33 82.55 0) (fields_autoplaced)
     (effects (font (size 1.27 1.27)) (justify left))
@@
       (effects (font (size 0.5 0.5)))
     )
-    (property "Footprint" "2004_cap:C0603" (id 2) (at 113.03 68.58 0)
+    (property "Footprint" "2003_res:R0603" (id 2) (at 113.03 68.58 0)
       (effects (font (size 1.27 1.27)) hide)
     )
@@
       (effects (font (size 0.5 0.5)))
     )
-    (property "Footprint" "2004_cap:C0603" (id 2) (at 68.58 88.9 0)
+    (property "Footprint" "2003_res:R0603" (id 2) (at 68.58 88.9 0)
       (effects (font (size 1.27 1.27)) hide)
     )
@@
       (effects (font (size 0.5 0.5)))
     )
-    (property "Footprint" "2004_cap:C0603" (id 2) (at 92.71 80.01 0)
+    (property "Footprint" "2003_res:R0603" (id 2) (at 92.71 80.01 0)
       (effects (font (size 1.27 1.27)) hide)
     )
@@
       (effects (font (size 0.5 0.5)))
     )
-    (property "Footprint" "2004_cap:C0603" (id 2) (at 78.74 90.17 0)
+    (property "Footprint" "2003_res:R0603" (id 2) (at 78.74 90.17 0)
       (effects (font (size 1.27 1.27)) hide)
     )
@@
       (effects (font (size 0.5 0.5)))
     )
-    (property "Footprint" "2004_cap:C0603" (id 2) (at 78.74 80.01 0)
+    (property "Footprint" "2003_res:R0603" (id 2) (at 78.74 80.01 0)
       (effects (font (size 1.27 1.27)) hide)
     )
@@
       (effects (font (size 0.5 0.5)))
     )
-    (property "Footprint" "2004_cap:C0603" (id 2) (at 68.58 77.47 0)
+    (property "Footprint" "2003_res:R0603" (id 2) (at 68.58 77.47 0)
       (effects (font (size 1.27 1.27)) hide)
     )
@@
       (effects (font (size 0.5 0.5)))
     )
-    (property "Footprint" "2004_cap:C0603" (id 2) (at 166.37 78.74 0)
+    (property "Footprint" "2003_res:R0603" (id 2) (at 166.37 78.74 0)
       (effects (font (size 1.27 1.27)) hide)
     )
@@
       (effects (font (size 0.5 0.5)))
     )
-    (property "Footprint" "2004_cap:C0603" (id 2) (at 179.07 78.74 0)
+    (property "Footprint" "2003_res:R0603" (id 2) (at 179.07 78.74 0)
       (effects (font (size 1.27 1.27)) hide)
     )
@@
       (effects (font (size 0.5 0.5)))
     )
-    (property "Footprint" "2004_cap:C0603" (id 2) (at 72.39 90.17 0)
+    (property "Footprint" "2003_res:R0603" (id 2) (at 72.39 90.17 0)
       (effects (font (size 1.27 1.27)) hide)
     )
@@
       (effects (font (size 0.5 0.5)))
     )
-    (property "Footprint" "2004_cap:C0603" (id 2) (at 154.94 60.96 0)
+    (property "Footprint" "2003_res:R0603" (id 2) (at 154.94 60.96 0)
       (effects (font (size 1.27 1.27)) hide)
     )
@@
       (effects (font (size 0.5 0.5)))
     )
-    (property "Footprint" "2004_cap:C0603" (id 2) (at 196.85 78.74 0)
-      (effects (font (size 1.27 1.27)) hide)
-    )
+    (property "Footprint" "2003_res:R0603" (id 2) (at 196.85 78.74 0)
+      (effects (font (size 1.27 1.27)) hide)
+    )
