File: kicad01_power_board_for_nuclear_team/005_dcdc_5v3a.kicad_sch (KiCad schematic)
At the start: 21 parts, among them U501 dcdc_lt8612x

Commit message: x
Parts:
- C522, C524, C525, C565, C571: footprint Capacitor_SMD:C_0603_1608Metric -> 02_dyn_pcblib:C0603
- R511, R512, R513, R523, R531, R532, R551, R561, R562, R565: footprint Resistor_SMD:R_0603_1608Metric -> 02_dyn_pcblib:C0603
- R552: footprint Resistor_SMD:R_0603_1608Metric_Pad0.98x0.95mm_HandSolder -> 02_dyn_pcblib:C0603
Connections:
- net GND: no longer names the net of C521.2, C571.2, U501.10 (PGND), U501.11 (GND), U501.12 (GND), U501.13 (GND), U501.14 (GND), U501.29 (GND), U501.30 (GND), U501.31 (GND), U501.32 (GND), U501.8 (PGND), U501.9 (PGND)
- net GND: no longer C522.2, C524.1, R513.2, R523.2, R531.2, R561.2, U501.25 (NC), U501.26 (NC), U501.27 (NC), U501.28 (NC)
- new net: C522.2, R513.2, R523.2, R531.2, U501.25 (NC), U501.26 (NC), U501.27 (NC), U501.28 (NC)

Commit message: ix
Parts:
- C521: symbol 01dyn_lib:c0805_35v10u -> 1001_un:c0805_35v10u
- C522, C565: symbol 01dyn_lib:c0603_100v10n -> 1001_un:c0603_100v10n
- C524: symbol 01dyn_lib:c0603_50v1u -> 1001_un:c0603_50v1u
- C525: symbol 01dyn_lib:c0603_50v0.1u -> 1001_un:c0603_50v0.1u
- C571: symbol 01dyn_lib:c0603_10v3.3u -> 1001_un:c0603_10v3.3u
- D551: symbol 01dyn_lib:LED0603_red -> 1001_un:LED0603_red
- L571: symbol 01dyn_lib:L3.3uH_7.4x6.6mm_30mhO_9.5A -> 1001_un:L3.3uH_7.4x6.6mm_30mhO_9.5A
- R511, R512, R523, R565: symbol 01dyn_lib:R0603_100k -> 1001_un:R0603_100k
- R513, R532, R551, R561, R562: symbol 01dyn_lib:R0603_10k -> 1001_un:R0603_10k
- R531: symbol 01dyn_lib:R0603_49.9k -> 1001_un:R0603_49.9k
- R552: symbol 01dyn_lib:R0603_DNP -> 1001_un:R0603_DNP
- R591: symbol 01dyn_lib:R1206_0.0 -> 1001_un:R1206_0.0
- U501: symbol 01dyn_lib:dcdc_lt8612x -> 1001_un:dcdc_lt8612x
Connections:
- net GND: now reaches C522.2, R513.2, R523.2, R531.2, U501.25 (NC), U501.26 (NC), U501.27 (NC), U501.28 (NC)
- net GND: now also C521.2, C524.1, C571.2, R561.2, U501.10 (PGND), U501.11 (GND), U501.12 (GND), U501.13 (GND), U501.14 (GND), U501.29 (GND), U501.30 (GND), U501.31 (GND), U501.32 (GND), U501.8 (PGND), U501.9 (PGND)
Other:
- note added: "Output : 0.97/(Rx61+Rx62)*(Rx61+Rx62+Rx63) 0.97/(0.1+22.6)*(0.1+22.6+100)==5.243v"
- note removed: "Output : 0.97/(Rx61+Rx62)*(Rx61+Rx62+Rx63) 0.97/(1+4.7)*(1+4.7+100)==17.988v"
Changed lines of the file:
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@@
     (effects (font (size 2 2)) (justify left bottom))
   )
-  (text "Output : \n0.97/(Rx61+Rx62)*(Rx61+Rx62+Rx63)\n0.97/(1+4.7)*(1+4.7+100)==17.988v"
-    (at 153.67 60.96 0)
+  (text "Output : \n0.97/(Rx61+Rx62)*(Rx61+Rx62+Rx63)\n0.97/(0.1+22.6)*(0.1+22.6+100)==5.243v"
+    (at 148.59 60.96 0)
     (effects (font (size 2 2)) (justify left bottom))
   )
@@
     )
   )
-  (symbol (lib_id "01dyn_lib:R1206_0.0") (at 187.96 46.99 180) (unit 1)
+  (symbol (lib_id "1001_un:R1206_0.0") (at 187.96 46.99 180) (unit 1)
     (in_bom yes) (on_board yes) (fields_autoplaced)
     (property "Reference" "R591" (id 0) (at 187.96 41.91 0)
@@
     (pin "2")
   )
-  (symbol (lib_name "R0603_100k_3") (lib_id "01dyn_lib:R0603_100k") (at 208.28 77.47 180) (unit 1)
+  (symbol (lib_id "1001_un:R0603_100k") (at 208.28 77.47 180) (unit 1)
     (in_bom yes) (on_board yes)
     (property "Reference" "R565" (id 0) (at 210.82 74.93 0)
@@
     (pin "2")
   )
-  (symbol (lib_name "R0603_100k_1") (lib_id "01dyn_lib:R0603_100k") (at 82.55 92.71 90) (unit 1)
+  (symbol (lib_id "1001_un:R0603_100k") (at 82.55 92.71 90) (unit 1)
     (in_bom yes) (on_board yes)
     (property "Reference" "R512" (id 0) (at 81.28 95.25 0)
@@
     (pin "2")
   )
-  (symbol (lib_name "R0603_10k_4") (lib_id "01dyn_lib:R0603_10k") (at 86.36 93.98 90) (unit 1)
+  (symbol (lib_id "1001_un:R0603_10k") (at 86.36 93.98 90) (unit 1)
     (in_bom yes) (on_board yes)
     (property "Reference" "R513" (id 0) (at 87.63 88.9 0)
@@
     (pin "2")
   )
-  (symbol (lib_id "01dyn_lib:c0603_10v3.3u") (at 218.44 123.19 180) (unit 1)
+  (symbol (lib_id "1001_un:c0603_10v3.3u") (at 218.44 123.19 180) (unit 1)
     (in_bom yes) (on_board yes)
     (property "Reference" "C571" (id 0) (at 219.71 120.65 0)
@@
     (pin "2")
   )
-  (symbol (lib_id "01dyn_lib:GND_1") (at 104.14 134.62 0) (unit 1)
+  (symbol (lib_id "power:GND") (at 104.14 134.62 0) (unit 1)
     (in_bom yes) (on_board yes) (fields_autoplaced)
     (property "Reference" "#PWR0111" (id 0) (at 104.14 140.97 0)
       (effects (font (size 1.27 1.27)) hide)
     )
-    (property "Value" "GND_1" (id 1) (at 104.14 138.43 0))
+    (property "Value" "GND" (id 1) (at 104.14 138.43 0))
     (property "Footprint" "" (id 2) (at 104.14 134.62 0)
       (effects (font (size 1.27 1.27)) hide)
@@
     (pin "1")
   )
-  (symbol (lib_id "01dyn_lib:R0603_DNP") (at 163.83 67.31 0) (unit 1)
+  (symbol (lib_id "1001_un:R0603_DNP") (at 163.83 67.31 0) (unit 1)
     (in_bom yes) (on_board yes)
     (property "Reference" "R552" (id 0) (at 168.91 66.04 0)
@@
     (pin "2")
   )
-  (symbol (lib_id "01dyn_lib:c0805_35v10u") (at 76.2 120.65 180) (unit 1)
+  (symbol (lib_id "1001_un:c0805_35v10u") (at 76.2 120.65 180) (unit 1)
     (in_bom yes) (on_board yes)
     (property "Reference" "C521" (id 0) (at 78.74 123.19 0))
@@
     (pin "2")
   )
-  (symbol (lib_name "c0603_100v10n_1") (lib_id "01dyn_lib:c0603_100v10n") (at 208.28 82.55 270) (unit 1)
+  (symbol (lib_id "1001_un:c0603_100v10n") (at 208.28 82.55 270) (unit 1)
     (in_bom yes) (on_board yes)
     (property "Reference" "C565" (id 0) (at 209.55 85.09 90)
@@
     (pin "2")
   )
-  (symbol (lib_name "R0603_10k_3") (lib_id "01dyn_lib:R0603_10k") (at 124.46 67.31 180) (unit 1)
+  (symbol (lib_id "1001_un:R0603_10k") (at 124.46 67.31 180) (unit 1)
     (in_bom yes) (on_board yes)
     (property "Reference" "R551" (id 0) (at 129.54 66.04 0)
@@
     (pin "2")
   )
-  (symbol (lib_id "01dyn_lib:c0603_50v1u") (at 146.05 78.74 180) (unit 1)
+  (symbol (lib_id "1001_un:c0603_50v1u") (at 146.05 78.74 180) (unit 1)
     (in_bom yes) (on_board yes)
     (property "Reference" "C524" (id 0) (at 148.59 81.28 0))
@@
     (pin "2")
   )
-  (symbol (lib_id "01dyn_lib:c0603_100v10n") (at 102.87 92.71 0) (unit 1)
+  (symbol (lib_id "1001_un:c0603_100v10n") (at 102.87 92.71 0) (unit 1)
     (in_bom yes) (on_board yes)
     (property "Reference" "C522" (id 0) (at 102.87 96.52 0)
@@
     (pin "2")
   )
-  (symbol (lib_name "R0603_100k_2") (lib_id "01dyn_lib:R0603_100k") (at 82.55 81.28 90) (unit 1)
+  (symbol (lib_id "1001_un:R0603_100k") (at 82.55 81.28 90) (unit 1)
     (in_bom yes) (on_board yes)
     (property "Reference" "R511" (id 0) (at 81.28 74.93 0)
@@
     (pin "2")
   )
-  (symbol (lib_id "01dyn_lib:R0603_10k") (at 92.71 93.98 90) (unit 1)
+  (symbol (lib_id "1001_un:R0603_10k") (at 92.71 93.98 90) (unit 1)
     (in_bom yes) (on_board yes)
     (property "Reference" "R532" (id 0) (at 95.25 93.98 0)
@@
     (pin "2")
   )
-  (symbol (lib_id "01dyn_lib:L3.3uH_7.4x6.6mm_30mhO_9.5A") (at 199.39 110.49 0) (unit 1)
+  (symbol (lib_id "1001_un:L3.3uH_7.4x6.6mm_30mhO_9.5A") (at 199.39 110.49 0) (unit 1)
     (in_bom yes) (on_board yes)
     (property "Reference" "L571" (id 0) (at 199.39 106.68 0)
@@
     (pin "2")
   )
-  (symbol (lib_id "01dyn_lib:R0603_100k") (at 106.68 83.82 90) (unit 1)
+  (symbol (lib_id "1001_un:R0603_100k") (at 106.68 83.82 90) (unit 1)
     (in_bom yes) (on_board yes)
     (property "Reference" "R523" (id 0) (at 105.41 81.28 0)
@@
     (pin "2")
   )
-  (symbol (lib_name "R0603_10k_1") (lib_id "01dyn_lib:R0603_10k") (at 177.8 77.47 180) (unit 1)
+  (symbol (lib_id "1001_un:R0603_10k") (at 177.8 77.47 180) (unit 1)
     (in_bom yes) (on_board yes)
     (property "Reference" "R561" (id 0) (at 180.34 74.93 0)
@@
     (pin "2")
   )
-  (symbol (lib_id "01dyn_lib:GND_1") (at 165.1 83.82 0) (unit 1)
+  (symbol (lib_id "power:GND") (at 165.1 83.82 0) (unit 1)
     (in_bom yes) (on_board yes) (fields_autoplaced)
     (property "Reference" "#PWR0110" (id 0) (at 165.1 90.17 0)
       (effects (font (size 1.27 1.27)) hide)
     )
-    (property "Value" "GND_1" (id 1) (at 165.1 87.63 0))
+    (property "Value" "GND" (id 1) (at 165.1 87.63 0))
     (property "Footprint" "" (id 2) (at 165.1 83.82 0)
       (effects (font (size 1.27 1.27)) hide)
@@
     (pin "1")
   )
-  (symbol (lib_id "01dyn_lib:R0603_49.9k") (at 92.71 83.82 90) (unit 1)
+  (symbol (lib_id "1001_un:R0603_49.9k") (at 92.71 83.82 90) (unit 1)
     (in_bom yes) (on_board yes)
     (property "Reference" "R531" (id 0) (at 91.44 81.28 0)
@@
     (pin "2")
   )
-  (symbol (lib_id "01dyn_lib:c0603_50v0.1u") (at 157.48 105.41 90) (unit 1)
+  (symbol (lib_id "1001_un:c0603_50v0.1u") (at 157.48 105.41 90) (unit 1)
     (in_bom yes) (on_board yes)
     (property "Reference" "C525" (id 0) (at 162.56 104.14 90))
@@
     (pin "2")
   )
-  (symbol (lib_id "01dyn_lib:dcdc_lt8612x") (at 120.65 95.25 0) (unit 1)
+  (symbol (lib_id "1001_un:dcdc_lt8612x") (at 120.65 95.25 0) (unit 1)
     (in_bom yes) (on_board yes)
     (property "Reference" "U501" (id 0) (at 111.76 91.44 0)
@@
     (pin "9")
   )
-  (symbol (lib_id "01dyn_lib:LED0603_red") (at 104.14 67.31 180) (unit 1)
+  (symbol (lib_id "1001_un:LED0603_red") (at 104.14 67.31 180) (unit 1)
     (in_bom yes) (on_board yes)
     (property "Reference" "D551" (id 0) (at 107.95 66.04 0))
@@
     (pin "2")
   )
-  (symbol (lib_id "01dyn_lib:GND_1") (at 135.89 74.93 0) (unit 1)
+  (symbol (lib_id "power:GND") (at 135.89 74.93 0) (unit 1)
     (in_bom yes) (on_board yes) (fields_autoplaced)
     (property "Reference" "#PWR0109" (id 0) (at 135.89 81.28 0)
       (effects (font (size 1.27 1.27)) hide)
     )
-    (property "Value" "GND_1" (id 1) (at 135.89 78.74 0))
+    (property "Value" "GND" (id 1) (at 135.89 78.74 0))
     (property "Footprint" "" (id 2) (at 135.89 74.93 0)
       (effects (font (size 1.27 1.27)) hide)
@@
     (pin "1")
   )
-  (symbol (lib_id "01dyn_lib:GND_1") (at 99.06 82.55 0) (unit 1)
+  (symbol (lib_id "power:GND") (at 99.06 82.55 0) (unit 1)
     (in_bom yes) (on_board yes) (fields_autoplaced)
     (property "Reference" "#PWR0112" (id 0) (at 99.06 88.9 0)
       (effects (font (size 1.27 1.27)) hide)
     )
-    (property "Value" "GND_1" (id 1) (at 99.06 86.36 0))
+    (property "Value" "GND" (id 1) (at 99.06 86.36 0))
     (property "Footprint" "" (id 2) (at 99.06 82.55 0)
       (effects (font (size 1.27 1.27)) hide)
@@
     (pin "1")
   )
-  (symbol (lib_name "R0603_10k_2") (lib_id "01dyn_lib:R0603_10k") (at 190.5 77.47 180) (unit 1)
+  (symbol (lib_id "1001_un:R0603_10k") (at 190.5 77.47 180) (unit 1)
     (in_bom yes) (on_board yes)
     (property "Reference" "R562" (id 0) (at 190.5 74.93 0)

Commit message: x
Parts:
- added C572: c0805_DNP, 02_dyn_pcblib:C0805mix0603, symbol 1003_cap:c0805_DNP
- C521: symbol 1001_un:c0805_35v10u -> 1003_cap:c0805_35v10u
- C522, C565: symbol 1001_un:c0603_100v10n -> 1003_cap:c0603_100v10n
- C524: symbol 1001_un:c0603_50v1u -> 1003_cap:c0603_50v1u
- C525: symbol 1001_un:c0603_50v0.1u -> 1003_cap:c0603_50v0.1u
- C571: symbol 1001_un:c0603_10v3.3u -> 1003_cap:c0603_10v3.3u
- D551: symbol 1001_un:LED0603_red -> 1004_led_mos:LED0603_red
- R511, R512, R523, R565: symbol 1001_un:R0603_100k -> 1002_res:R0603_100k
- R513, R532, R551, R561, R562: symbol 1001_un:R0603_10k -> 1002_res:R0603_10k
- R531: symbol 1001_un:R0603_49.9k -> 1002_res:R0603_49.9k
- R552: symbol 1001_un:R0603_DNP -> 1002_res:R0603_DNP
- R591: symbol 1001_un:R1206_0.0 -> 1002_res:R1206_0.0
Connections:
- net GND: now also C572.1
- net at C565.2, C571.1, L571.2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: now also C572.2
Changed lines of the file:
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@@
   (junction (at 102.87 77.47) (diameter 0) (color 0 0 0 0)
   )
+  (junction (at 218.44 114.3) (diameter 0) (color 0 0 0 0)
+  )
   (junction (at 127 77.47) (diameter 0) (color 0 0 0 0)
   )
@@
   (junction (at 106.68 77.47) (diameter 0) (color 0 0 0 0)
   )
+  (junction (at 218.44 132.08) (diameter 0) (color 0 0 0 0)
+  )
   (junction (at 218.44 77.47) (diameter 0) (color 0 0 0 0)
   )
@@
     (stroke (width 0) (type default) (color 0 0 0 0))
   )
+  (wire (pts (xy 218.44 114.3) (xy 227.33 114.3))
+    (stroke (width 0) (type default) (color 0 0 0 0))
+  )
   (wire (pts (xy 129.54 132.08) (xy 132.08 132.08))
     (stroke (width 0) (type default) (color 0 0 0 0))
@@
     (stroke (width 0) (type default) (color 0 0 0 0))
   )
-  (wire (pts (xy 218.44 110.49) (xy 218.44 119.38))
+  (wire (pts (xy 218.44 110.49) (xy 218.44 114.3))
     (stroke (width 0) (type default) (color 0 0 0 0))
   )
@@
     (stroke (width 0) (type default) (color 0 0 0 0))
   )
+  (wire (pts (xy 227.33 127) (xy 227.33 132.08))
+    (stroke (width 0) (type default) (color 0 0 0 0))
+  )
   (wire (pts (xy 76.2 132.08) (xy 104.14 132.08))
     (stroke (width 0) (type default) (color 0 0 0 0))
@@
     (stroke (width 0) (type default) (color 0 0 0 0))
   )
+  (wire (pts (xy 227.33 132.08) (xy 218.44 132.08))
+    (stroke (width 0) (type default) (color 0 0 0 0))
+  )
   (wire (pts (xy 129.54 127) (xy 129.54 132.08))
     (stroke (width 0) (type default) (color 0 0 0 0))
@@
     (stroke (width 0) (type default) (color 0 0 0 0))
   )
+  (wire (pts (xy 227.33 119.38) (xy 227.33 114.3))
+    (stroke (width 0) (type default) (color 0 0 0 0))
+  )
   (wire (pts (xy 104.14 118.11) (xy 104.14 115.57))
     (stroke (width 0) (type default) (color 0 0 0 0))
@@
   )
   (wire (pts (xy 104.14 110.49) (xy 104.14 107.95))
+    (stroke (width 0) (type default) (color 0 0 0 0))
+  )
+  (wire (pts (xy 218.44 114.3) (xy 218.44 119.38))
     (stroke (width 0) (type default) (color 0 0 0 0))
   )
@@
     )
   )
-  (symbol (lib_id "1001_un:R1206_0.0") (at 187.96 46.99 180) (unit 1)
+  (symbol (lib_id "1002_res:R1206_0.0") (at 187.96 46.99 180) (unit 1)
     (in_bom yes) (on_board yes) (fields_autoplaced)
     (property "Reference" "R591" (id 0) (at 187.96 41.91 0)
@@
     (pin "2")
   )
-  (symbol (lib_id "1001_un:R0603_100k") (at 208.28 77.47 180) (unit 1)
+  (symbol (lib_id "1002_res:R0603_100k") (at 208.28 77.47 180) (unit 1)
     (in_bom yes) (on_board yes)
     (property "Reference" "R565" (id 0) (at 210.82 74.93 0)
@@
     (pin "2")
   )
-  (symbol (lib_id "1001_un:R0603_100k") (at 82.55 92.71 90) (unit 1)
+  (symbol (lib_id "1002_res:R0603_100k") (at 82.55 92.71 90) (unit 1)
     (in_bom yes) (on_board yes)
     (property "Reference" "R512" (id 0) (at 81.28 95.25 0)
@@
     (pin "2")
   )
-  (symbol (lib_id "1001_un:R0603_10k") (at 86.36 93.98 90) (unit 1)
+  (symbol (lib_id "1002_res:R0603_10k") (at 86.36 93.98 90) (unit 1)
     (in_bom yes) (on_board yes)
     (property "Reference" "R513" (id 0) (at 87.63 88.9 0)
@@
     (pin "2")
   )
-  (symbol (lib_id "1001_un:c0603_10v3.3u") (at 218.44 123.19 180) (unit 1)
+  (symbol (lib_id "1003_cap:c0603_10v3.3u") (at 218.44 123.19 180) (unit 1)
     (in_bom yes) (on_board yes)
     (property "Reference" "C571" (id 0) (at 219.71 120.65 0)
@@
     (pin "1")
   )
-  (symbol (lib_id "1001_un:R0603_DNP") (at 163.83 67.31 0) (unit 1)
+  (symbol (lib_id "1002_res:R0603_DNP") (at 163.83 67.31 0) (unit 1)
     (in_bom yes) (on_board yes)
     (property "Reference" "R552" (id 0) (at 168.91 66.04 0)
@@
     (pin "2")
   )
-  (symbol (lib_id "1001_un:c0805_35v10u") (at 76.2 120.65 180) (unit 1)
+  (symbol (lib_id "1003_cap:c0805_35v10u") (at 76.2 120.65 180) (unit 1)
     (in_bom yes) (on_board yes)
     (property "Reference" "C521" (id 0) (at 78.74 123.19 0))
@@
     (pin "2")
   )
-  (symbol (lib_id "1001_un:c0603_100v10n") (at 208.28 82.55 270) (unit 1)
+  (symbol (lib_id "1003_cap:c0603_100v10n") (at 208.28 82.55 270) (unit 1)
     (in_bom yes) (on_board yes)
     (property "Reference" "C565" (id 0) (at 209.55 85.09 90)
@@
     (pin "2")
   )
-  (symbol (lib_id "1001_un:R0603_10k") (at 124.46 67.31 180) (unit 1)
+  (symbol (lib_id "1002_res:R0603_10k") (at 124.46 67.31 180) (unit 1)
     (in_bom yes) (on_board yes)
     (property "Reference" "R551" (id 0) (at 129.54 66.04 0)
@@
     (pin "2")
   )
-  (symbol (lib_id "1001_un:c0603_50v1u") (at 146.05 78.74 180) (unit 1)
+  (symbol (lib_id "1003_cap:c0603_50v1u") (at 146.05 78.74 180) (unit 1)
     (in_bom yes) (on_board yes)
     (property "Reference" "C524" (id 0) (at 148.59 81.28 0))
@@
     (pin "2")
   )
-  (symbol (lib_id "1001_un:c0603_100v10n") (at 102.87 92.71 0) (unit 1)
+  (symbol (lib_id "1003_cap:c0603_100v10n") (at 102.87 92.71 0) (unit 1)
     (in_bom yes) (on_board yes)
     (property "Reference" "C522" (id 0) (at 102.87 96.52 0)
@@
     (pin "2")
   )
-  (symbol (lib_id "1001_un:R0603_100k") (at 82.55 81.28 90) (unit 1)
+  (symbol (lib_id "1002_res:R0603_100k") (at 82.55 81.28 90) (unit 1)
     (in_bom yes) (on_board yes)
     (property "Reference" "R511" (id 0) (at 81.28 74.93 0)
@@
     (pin "2")
   )
-  (symbol (lib_id "1001_un:R0603_10k") (at 92.71 93.98 90) (unit 1)
+  (symbol (lib_id "1003_cap:c0805_DNP") (at 227.33 123.19 0) (unit 1)
+    (in_bom yes) (on_board yes)
+    (property "Reference" "C572" (id 0) (at 231.14 122.555 0)
+      (effects (font (size 1.5 1.5)) (justify left))
+    )
+    (property "Value" "c0805_DNP" (id 1) (at 224.79 123.19 0)
+      (effects (font (size 0.5 0.5)) (justify left))
+    )
+    (property "Footprint" "02_dyn_pcblib:C0805mix0603" (id 2) (at 228.219 110.363 0)
+      (effects (font (size 1.27 1.27)) hide)
+    )
+    (property "Datasheet" "~" (id 3) (at 227.2665 123.2535 0)
+      (effects (font (size 1.27 1.27)) hide)
+    )
+    (property "PartNum" "c0805_DNP" (id 4) (at 226.822 107.696 0)
+      (effects (font (size 1.27 1.27)) hide)
+    )
+    (pin "1")
+    (pin "2")
+  )
+  (symbol (lib_id "1002_res:R0603_10k") (at 92.71 93.98 90) (unit 1)
     (in_bom yes) (on_board yes)
     (property "Reference" "R532" (id 0) (at 95.25 93.98 0)
@@
     (pin "2")
   )
-  (symbol (lib_id "1001_un:R0603_100k") (at 106.68 83.82 90) (unit 1)
+  (symbol (lib_id "1002_res:R0603_100k") (at 106.68 83.82 90) (unit 1)
     (in_bom yes) (on_board yes)
     (property "Reference" "R523" (id 0) (at 105.41 81.28 0)
@@
     (pin "2")
   )
-  (symbol (lib_id "1001_un:R0603_10k") (at 177.8 77.47 180) (unit 1)
+  (symbol (lib_id "1002_res:R0603_10k") (at 177.8 77.47 180) (unit 1)
     (in_bom yes) (on_board yes)
     (property "Reference" "R561" (id 0) (at 180.34 74.93 0)
@@
     (pin "1")
   )
-  (symbol (lib_id "1001_un:R0603_49.9k") (at 92.71 83.82 90) (unit 1)
+  (symbol (lib_id "1002_res:R0603_49.9k") (at 92.71 83.82 90) (unit 1)
     (in_bom yes) (on_board yes)
     (property "Reference" "R531" (id 0) (at 91.44 81.28 0)
@@
     (pin "2")
   )
-  (symbol (lib_id "1001_un:c0603_50v0.1u") (at 157.48 105.41 90) (unit 1)
+  (symbol (lib_id "1003_cap:c0603_50v0.1u") (at 157.48 105.41 90) (unit 1)
     (in_bom yes) (on_board yes)
     (property "Reference" "C525" (id 0) (at 162.56 104.14 90))
@@
     (pin "9")
   )
-  (symbol (lib_id "1001_un:LED0603_red") (at 104.14 67.31 180) (unit 1)
+  (symbol (lib_id "1004_led_mos:LED0603_red") (at 104.14 67.31 180) (unit 1)
     (in_bom yes) (on_board yes)
     (property "Reference" "D551" (id 0) (at 107.95 66.04 0))
@@
     (pin "1")
   )
-  (symbol (lib_id "1001_un:R0603_10k") (at 190.5 77.47 180) (unit 1)
+  (symbol (lib_id "1002_res:R0603_10k") (at 190.5 77.47 180) (unit 1)
     (in_bom yes) (on_board yes)
     (property "Reference" "R562" (id 0) (at 190.5 74.93 0)

Commit message: x
Parts:
- L571: symbol 1001_un:L3.3uH_7.4x6.6mm_30mhO_9.5A -> 1006_Inductance:L3.3uH_7.4x6.6mm_30mhO_9.5A
- U501: symbol 1001_un:dcdc_lt8612x -> 1009_ic:dcdc_lt8612x
Changed lines of the file:
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@@
       (effects (font (size 1.5 1.5)) (justify left))
     )
-    (property "Value" "c0805_DNP" (id 1) (at 224.79 123.19 0)
-      (effects (font (size 0.5 0.5)) (justify left))
+    (property "Value" "c0805_DNP" (id 1) (at 227.457 123.317 0)
+      (effects (font (size 0.5 0.5)))
     )
     (property "Footprint" "02_dyn_pcblib:C0805mix0603" (id 2) (at 228.219 110.363 0)
@@
     (pin "2")
   )
-  (symbol (lib_id "1001_un:L3.3uH_7.4x6.6mm_30mhO_9.5A") (at 199.39 110.49 0) (unit 1)
+  (symbol (lib_id "1006_Inductance:L3.3uH_7.4x6.6mm_30mhO_9.5A") (at 199.39 110.49 0) (unit 1)
     (in_bom yes) (on_board yes)
     (property "Reference" "L571" (id 0) (at 199.39 106.68 0)
@@
     (pin "2")
   )
-  (symbol (lib_id "1001_un:dcdc_lt8612x") (at 120.65 95.25 0) (unit 1)
+  (symbol (lib_id "1009_ic:dcdc_lt8612x") (at 120.65 95.25 0) (unit 1)
     (in_bom yes) (on_board yes)
     (property "Reference" "U501" (id 0) (at 111.76 91.44 0)

Commit message: x
Changed lines of the file:
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@@
     )
     (property "Value" "R0603_DNP" (id 1) (at 162.052 68.707 0)
-      (effects (font (size 0.5 0.5)) hide)
+      (effects (font (size 0.5 0.5)))
     )
     (property "Footprint" "02_dyn_pcblib:C0603" (id 2) (at 165.1 63.5 0)
