File: kicad01_power_board_for_nuclear_team/005_dcdc_5v3a.kicad_sch (KiCad schematic)
At the start: 22 parts, among them U501 dcdc_lt8612x

Commit message: x
Parts:
- C521, C572: footprint 02_dyn_pcblib:C0805mix0603 -> 2004_cap:C0805mix0603
- C522, C524, C525, C565, C571, R511, R512, R513, R523, R531, R532, R551, R552, R561, R562, R565: footprint 02_dyn_pcblib:C0603 -> 2004_cap:C0603
- D551: footprint 02_dyn_pcblib:LED0603 -> 2007_LED:LED0603
- L571: footprint 02_dyn_pcblib:L7.1x6.6mm -> 2005_inductance:L7.1x6.6mm
- R591: footprint 02_dyn_pcblib:R1206mix0603 -> 2003_res:R1206mix0603
- U501: footprint 02_dyn_pcblib:QFN-28-1EP_3x6mm_P0.5mm_EP1.7x4.75mmX -> 2006_qfn:QFN-28-1EP_3x6mm_P0.5mm_EP1.7x4.75mmX
Changed lines of the file:
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@@
       (effects (font (size 0.5 0.5)))
     )
-    (property "Footprint" "02_dyn_pcblib:R1206mix0603" (id 2) (at 187.96 58.42 0)
+    (property "Footprint" "2003_res:R1206mix0603" (id 2) (at 187.96 58.42 0)
       (effects (font (size 1.27 1.27)) hide)
     )
@@
       (effects (font (size 0.5 0.5)))
     )
-    (property "Footprint" "02_dyn_pcblib:C0603" (id 2) (at 207.01 81.28 0)
+    (property "Footprint" "2004_cap:C0603" (id 2) (at 207.01 81.28 0)
       (effects (font (size 1.27 1.27)) hide)
     )
@@
       (effects (font (size 0.5 0.5)))
     )
-    (property "Footprint" "02_dyn_pcblib:C0603" (id 2) (at 78.74 91.44 0)
+    (property "Footprint" "2004_cap:C0603" (id 2) (at 78.74 91.44 0)
       (effects (font (size 1.27 1.27)) hide)
     )
@@
       (effects (font (size 0.5 0.5)))
     )
-    (property "Footprint" "02_dyn_pcblib:C0603" (id 2) (at 82.55 92.71 0)
+    (property "Footprint" "2004_cap:C0603" (id 2) (at 82.55 92.71 0)
       (effects (font (size 1.27 1.27)) hide)
     )
@@
       (effects (font (size 0.5 0.5)))
     )
-    (property "Footprint" "02_dyn_pcblib:C0603" (id 2) (at 217.551 136.017 0)
+    (property "Footprint" "2004_cap:C0603" (id 2) (at 217.551 136.017 0)
       (effects (font (size 1.27 1.27)) hide)
     )
@@
       (effects (font (size 0.5 0.5)))
     )
-    (property "Footprint" "02_dyn_pcblib:C0603" (id 2) (at 165.1 63.5 0)
+    (property "Footprint" "2004_cap:C0603" (id 2) (at 165.1 63.5 0)
       (effects (font (size 1.27 1.27)) hide)
     )
@@
       (effects (font (size 0.5 0.5)))
     )
-    (property "Footprint" "02_dyn_pcblib:C0805mix0603" (id 2) (at 75.311 133.477 0)
+    (property "Footprint" "2004_cap:C0805mix0603" (id 2) (at 75.311 133.477 0)
       (effects (font (size 1.27 1.27)) hide)
     )
@@
       (effects (font (size 0.5 0.5)))
     )
-    (property "Footprint" "02_dyn_pcblib:C0603" (id 2) (at 221.107 83.439 0)
+    (property "Footprint" "2004_cap:C0603" (id 2) (at 221.107 83.439 0)
       (effects (font (size 1.27 1.27)) hide)
     )
@@
       (effects (font (size 0.5 0.5)))
     )
-    (property "Footprint" "02_dyn_pcblib:C0603" (id 2) (at 123.19 71.12 0)
+    (property "Footprint" "2004_cap:C0603" (id 2) (at 123.19 71.12 0)
       (effects (font (size 1.27 1.27)) hide)
     )
@@
       (effects (font (size 0.5 0.5)))
     )
-    (property "Footprint" "02_dyn_pcblib:C0603" (id 2) (at 145.161 91.567 0)
+    (property "Footprint" "2004_cap:C0603" (id 2) (at 145.161 91.567 0)
       (effects (font (size 1.27 1.27)) hide)
     )
@@
       (effects (font (size 0.5 0.5)))
     )
-    (property "Footprint" "02_dyn_pcblib:C0603" (id 2) (at 103.759 79.883 0)
+    (property "Footprint" "2004_cap:C0603" (id 2) (at 103.759 79.883 0)
       (effects (font (size 1.27 1.27)) hide)
     )
@@
       (effects (font (size 0.5 0.5)))
     )
-    (property "Footprint" "02_dyn_pcblib:C0603" (id 2) (at 78.74 80.01 0)
+    (property "Footprint" "2004_cap:C0603" (id 2) (at 78.74 80.01 0)
       (effects (font (size 1.27 1.27)) hide)
     )
@@
       (effects (font (size 0.5 0.5)))
     )
-    (property "Footprint" "02_dyn_pcblib:C0805mix0603" (id 2) (at 228.219 110.363 0)
+    (property "Footprint" "2004_cap:C0805mix0603" (id 2) (at 228.219 110.363 0)
       (effects (font (size 1.27 1.27)) hide)
     )
@@
       (effects (font (size 0.5 0.5)))
     )
-    (property "Footprint" "02_dyn_pcblib:C0603" (id 2) (at 88.9 92.71 0)
+    (property "Footprint" "2004_cap:C0603" (id 2) (at 88.9 92.71 0)
       (effects (font (size 1.27 1.27)) hide)
     )
@@
       (effects (font (size 0.5 0.5)) (justify left))
     )
-    (property "Footprint" "02_dyn_pcblib:L7.1x6.6mm" (id 2) (at 198.12 100.33 0)
+    (property "Footprint" "2005_inductance:L7.1x6.6mm" (id 2) (at 198.12 100.33 0)
       (effects (font (size 1.27 1.27)) hide)
     )
@@
       (effects (font (size 0.5 0.5)))
     )
-    (property "Footprint" "02_dyn_pcblib:C0603" (id 2) (at 102.87 82.55 0)
+    (property "Footprint" "2004_cap:C0603" (id 2) (at 102.87 82.55 0)
       (effects (font (size 1.27 1.27)) hide)
     )
@@
       (effects (font (size 0.5 0.5)))
     )
-    (property "Footprint" "02_dyn_pcblib:C0603" (id 2) (at 176.53 81.28 0)
+    (property "Footprint" "2004_cap:C0603" (id 2) (at 176.53 81.28 0)
       (effects (font (size 1.27 1.27)) hide)
     )
@@
       (effects (font (size 0.5 0.5)))
     )
-    (property "Footprint" "02_dyn_pcblib:C0603" (id 2) (at 88.9 82.55 0)
+    (property "Footprint" "2004_cap:C0603" (id 2) (at 88.9 82.55 0)
       (effects (font (size 1.27 1.27)) hide)
     )
@@
       (effects (font (size 0.5 0.5)))
     )
-    (property "Footprint" "02_dyn_pcblib:C0603" (id 2) (at 144.653 104.521 0)
+    (property "Footprint" "2004_cap:C0603" (id 2) (at 144.653 104.521 0)
       (effects (font (size 1.27 1.27)) hide)
     )
@@
     )
     (property "Value" "dcdc_lt8612x" (id 1) (at 124.46 109.22 0))
-    (property "Footprint" "02_dyn_pcblib:QFN-28-1EP_3x6mm_P0.5mm_EP1.7x4.75mmX" (id 2) (at 127 67.31 0)
+    (property "Footprint" "2006_qfn:QFN-28-1EP_3x6mm_P0.5mm_EP1.7x4.75mmX" (id 2) (at 127 67.31 0)
       (effects (font (size 1.27 1.27)) hide)
     )
@@
       (effects (font (size 0.5 0.5)) (justify left))
     )
-    (property "Footprint" "02_dyn_pcblib:LED0603" (id 2) (at 104.14 76.2 0)
+    (property "Footprint" "2007_LED:LED0603" (id 2) (at 104.14 76.2 0)
       (effects (font (size 1.27 1.27)) hide)
     )
@@
       (effects (font (size 0.5 0.5)))
     )
-    (property "Footprint" "02_dyn_pcblib:C0603" (id 2) (at 189.23 81.28 0)
-      (effects (font (size 1.27 1.27)) hide)
-    )
+    (property "Footprint" "2004_cap:C0603" (id 2) (at 189.23 81.28 0)
+      (effects (font (size 1.27 1.27)) hide)
+    )
