File: kicad01_power_board_for_nuclear_team/006_msp430.kicad_sch (KiCad schematic)
At the start: 0 parts

Commit message: x
Parts:
- added R603: R0805_0.0, 02_dyn_pcblib:R0805mix0603, symbol 01dyn_lib:R0805_0.0
- added R604: R0603_DNP, Resistor_SMD:R_0603_1608Metric_Pad0.98x0.95mm_HandSolder, symbol 01dyn_lib:R0603_DNP
- added R623, R624, R633, R634: R0603_10k, Resistor_SMD:R_0603_1608Metric, symbol 01dyn_lib:R0603_10k
Connections:
- new net: R603.2, R604.1
- new net: R623.2, R624.1
- new net: R633.2, R634.1
- new net VOint3: R623.1
- new net VOint4: R624.2
- new net Vgood3: R633.1
- new net Vgood4: R634.2
- new net Vsync3: R603.1
- new net Vsync4: R604.2
Changed lines of the file:
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@@
 (kicad_sch (version 20211123) (generator eeschema)
   (paper "A4")
+  (wire (pts (xy 63.5 72.39) (xy 69.85 72.39))
+    (stroke (width 0) (type default) (color 0 0 0 0))
+  )
+  (wire (pts (xy 109.22 72.39) (xy 114.3 72.39))
+    (stroke (width 0) (type default) (color 0 0 0 0))
+  )
+  (wire (pts (xy 77.47 54.61) (xy 101.6 54.61))
+    (stroke (width 0) (type default) (color 0 0 0 0))
+  )
+  (wire (pts (xy 109.22 63.5) (xy 114.3 63.5))
+    (stroke (width 0) (type default) (color 0 0 0 0))
+  )
+  (wire (pts (xy 77.47 72.39) (xy 101.6 72.39))
+    (stroke (width 0) (type default) (color 0 0 0 0))
+  )
+  (wire (pts (xy 77.47 63.5) (xy 101.6 63.5))
+    (stroke (width 0) (type default) (color 0 0 0 0))
+  )
+  (wire (pts (xy 63.5 63.5) (xy 69.85 63.5))
+    (stroke (width 0) (type default) (color 0 0 0 0))
+  )
+  (wire (pts (xy 63.5 54.61) (xy 69.85 54.61))
+    (stroke (width 0) (type default) (color 0 0 0 0))
+  )
+  (wire (pts (xy 109.22 54.61) (xy 114.3 54.61))
+    (stroke (width 0) (type default) (color 0 0 0 0))
+  )
+  (global_label "VOint3" (shape input) (at 63.5 63.5 180) (fields_autoplaced)
+    (effects (font (size 1.27 1.27)) (justify right))
+    (property "Intersheet References" "${INTERSHEET_REFS}" (id 0) (at 54.9788 63.4206 0)
+      (effects (font (size 1.27 1.27)) (justify right) hide)
+    )
+  )
+  (global_label "Vgood3" (shape input) (at 63.5 72.39 180) (fields_autoplaced)
+    (effects (font (size 1.27 1.27)) (justify right))
+    (property "Intersheet References" "${INTERSHEET_REFS}" (id 0) (at 54.1926 72.4694 0)
+      (effects (font (size 1.27 1.27)) (justify right) hide)
+    )
+  )
+  (global_label "Vsync4" (shape input) (at 114.3 54.61 0) (fields_autoplaced)
+    (effects (font (size 1.27 1.27)) (justify left))
+    (property "Intersheet References" "${INTERSHEET_REFS}" (id 0) (at 123.2445 54.5306 0)
+      (effects (font (size 1.27 1.27)) (justify left) hide)
+    )
+  )
+  (global_label "Vsync3" (shape input) (at 63.5 54.61 180) (fields_autoplaced)
+    (effects (font (size 1.27 1.27)) (justify right))
+    (property "Intersheet References" "${INTERSHEET_REFS}" (id 0) (at 54.5555 54.6894 0)
+      (effects (font (size 1.27 1.27)) (justify right) hide)
+    )
+  )
+  (global_label "Vgood4" (shape input) (at 114.3 72.39 0) (fields_autoplaced)
+    (effects (font (size 1.27 1.27)) (justify left))
+    (property "Intersheet References" "${INTERSHEET_REFS}" (id 0) (at 123.6074 72.3106 0)
+      (effects (font (size 1.27 1.27)) (justify left) hide)
+    )
+  )
+  (global_label "VOint4" (shape input) (at 114.3 63.5 0) (fields_autoplaced)
+    (effects (font (size 1.27 1.27)) (justify left))
+    (property "Intersheet References" "${INTERSHEET_REFS}" (id 0) (at 122.8212 63.4206 0)
+      (effects (font (size 1.27 1.27)) (justify left) hide)
+    )
+  )
+  (symbol (lib_id "01dyn_lib:R0805_0.0") (at 73.66 54.61 0) (unit 1)
+    (in_bom yes) (on_board yes) (fields_autoplaced)
+    (property "Reference" "R603" (id 0) (at 73.66 49.53 0)
+      (effects (font (size 1.5 1.5)))
+    )
+    (property "Value" "R0805_0.0" (id 1) (at 71.882 56.007 0)
+      (effects (font (size 0.5 0.5)))
+    )
+    (property "Footprint" "02_dyn_pcblib:R0805mix0603" (id 2) (at 72.39 41.91 0)
+      (effects (font (size 1.27 1.27)) hide)
+    )
+    (property "Datasheet" "~" (id 3) (at 73.66 54.61 90)
+      (effects (font (size 1.27 1.27)) hide)
+    )
+    (property "PartNum" "RC0805JR-070RL" (id 4) (at 73.533 52.705 0)
+      (effects (font (size 1.27 1.27)) hide)
+    )
+    (property "PartDesc" "0 Ohms Jumper 0.125W, 1/8W Chip Resistor 0805 (2012 Metric) Moisture Resistant Thick Film" (id 5) (at 71.12 45.72 0)
+      (effects (font (size 1.27 1.27)) hide)
+    )
+    (pin "1")
+    (pin "2")
+  )
+  (symbol (lib_id "01dyn_lib:R0603_10k") (at 105.41 63.5 0) (unit 1)
+    (in_bom yes) (on_board yes) (fields_autoplaced)
+    (property "Reference" "R624" (id 0) (at 105.41 58.42 0)
+      (effects (font (size 1.5 1.5)))
+    )
+    (property "Value" "R0603_10k" (id 1) (at 103.632 64.897 0)
+      (effects (font (size 0.5 0.5)))
+    )
+    (property "Footprint" "Resistor_SMD:R_0603_1608Metric" (id 2) (at 106.68 59.69 0)
+      (effects (font (size 1.27 1.27)) hide)
+    )
+    (property "Datasheet" "~" (id 3) (at 105.41 63.5 90)
+      (effects (font (size 1.27 1.27)) hide)
+    )
+    (property "PartNum" "ERJ-PA3F1002V" (id 4) (at 105.537 61.595 0)
+      (effects (font (size 1.27 1.27)) hide)
+    )
+    (pin "1")
+    (pin "2")
+  )
+  (symbol (lib_name "R0603_10k_2") (lib_id "01dyn_lib:R0603_10k") (at 73.66 63.5 0) (unit 1)
+    (in_bom yes) (on_board yes) (fields_autoplaced)
+    (property "Reference" "R623" (id 0) (at 73.66 58.42 0)
+      (effects (font (size 1.5 1.5)))
+    )
+    (property "Value" "R0603_10k" (id 1) (at 71.882 64.897 0)
+      (effects (font (size 0.5 0.5)))
+    )
+    (property "Footprint" "Resistor_SMD:R_0603_1608Metric" (id 2) (at 74.93 59.69 0)
+      (effects (font (size 1.27 1.27)) hide)
+    )
+    (property "Datasheet" "~" (id 3) (at 73.66 63.5 90)
+      (effects (font (size 1.27 1.27)) hide)
+    )
+    (property "PartNum" "ERJ-PA3F1002V" (id 4) (at 73.787 61.595 0)
+      (effects (font (size 1.27 1.27)) hide)
+    )
+    (pin "1")
+    (pin "2")
+  )
+  (symbol (lib_id "01dyn_lib:R0603_DNP") (at 105.41 54.61 0) (unit 1)
+    (in_bom yes) (on_board yes) (fields_autoplaced)
+    (property "Reference" "R604" (id 0) (at 105.41 49.53 0)
+      (effects (font (size 1.5 1.5)))
+    )
+    (property "Value" "R0603_DNP" (id 1) (at 103.632 56.007 0)
+      (effects (font (size 0.5 0.5)) hide)
+    )
+    (property "Footprint" "Resistor_SMD:R_0603_1608Metric_Pad0.98x0.95mm_HandSolder" (id 2) (at 106.68 50.8 0)
+      (effects (font (size 1.27 1.27)) hide)
+    )
+    (property "Datasheet" "~" (id 3) (at 105.41 54.61 90)
+      (effects (font (size 1.27 1.27)) hide)
+    )
+    (property "PartNum" "R0603_DNP" (id 4) (at 105.283 52.705 0)
+      (effects (font (size 1.27 1.27)) hide)
+    )
+    (property "Notice" "This DNP resistor use handly footprint, which is larger than the normal standard footprint" (id 5) (at 102.87 45.72 0)
+      (effects (font (size 1.27 1.27)) hide)
+    )
+    (pin "1")
+    (pin "2")
+  )
+  (symbol (lib_name "R0603_10k_3") (lib_id "01dyn_lib:R0603_10k") (at 73.66 72.39 0) (unit 1)
+    (in_bom yes) (on_board yes) (fields_autoplaced)
+    (property "Reference" "R633" (id 0) (at 73.66 67.31 0)
+      (effects (font (size 1.5 1.5)))
+    )
+    (property "Value" "R0603_10k" (id 1) (at 71.882 73.787 0)
+      (effects (font (size 0.5 0.5)))
+    )
+    (property "Footprint" "Resistor_SMD:R_0603_1608Metric" (id 2) (at 74.93 68.58 0)
+      (effects (font (size 1.27 1.27)) hide)
+    )
+    (property "Datasheet" "~" (id 3) (at 73.66 72.39 90)
+      (effects (font (size 1.27 1.27)) hide)
+    )
+    (property "PartNum" "ERJ-PA3F1002V" (id 4) (at 73.787 70.485 0)
+      (effects (font (size 1.27 1.27)) hide)
+    )
+    (pin "1")
+    (pin "2")
+  )
+  (symbol (lib_name "R0603_10k_1") (lib_id "01dyn_lib:R0603_10k") (at 105.41 72.39 0) (unit 1)
+    (in_bom yes) (on_board yes) (fields_autoplaced)
+    (property "Reference" "R634" (id 0) (at 105.41 67.31 0)
+      (effects (font (size 1.5 1.5)))
+    )
+    (property "Value" "R0603_10k" (id 1) (at 103.632 73.787 0)
+      (effects (font (size 0.5 0.5)))
+    )
+    (property "Footprint" "Resistor_SMD:R_0603_1608Metric" (id 2) (at 106.68 68.58 0)
+      (effects (font (size 1.27 1.27)) hide)
+    )
+    (property "Datasheet" "~" (id 3) (at 105.41 72.39 90)
+      (effects (font (size 1.27 1.27)) hide)
+    )
+    (property "PartNum" "ERJ-PA3F1002V" (id 4) (at 105.537 70.485 0)
+      (effects (font (size 1.27 1.27)) hide)
+    )
+    (pin "1")
+    (pin "2")
+  )
 )

Commit message: ix
Parts:
- R603: symbol 01dyn_lib:R0805_0.0 -> 1001_un:R0805_0.0
- R604: footprint Resistor_SMD:R_0603_1608Metric_Pad0.98x0.95mm_HandSolder -> 02_dyn_pcblib:C0603; symbol 01dyn_lib:R0603_DNP -> 1001_un:R0603_DNP
- R623, R624, R633, R634: footprint Resistor_SMD:R_0603_1608Metric -> 02_dyn_pcblib:C0603; symbol 01dyn_lib:R0603_10k -> 1001_un:R0603_10k
Changed lines of the file:
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@@
     )
   )
-  (symbol (lib_id "01dyn_lib:R0805_0.0") (at 73.66 54.61 0) (unit 1)
+  (symbol (lib_id "1001_un:R0805_0.0") (at 73.66 54.61 0) (unit 1)
     (in_bom yes) (on_board yes) (fields_autoplaced)
     (property "Reference" "R603" (id 0) (at 73.66 49.53 0)
@@
     (pin "2")
   )
-  (symbol (lib_id "01dyn_lib:R0603_10k") (at 105.41 63.5 0) (unit 1)
+  (symbol (lib_id "1001_un:R0603_10k") (at 105.41 63.5 0) (unit 1)
     (in_bom yes) (on_board yes) (fields_autoplaced)
     (property "Reference" "R624" (id 0) (at 105.41 58.42 0)
@@
       (effects (font (size 0.5 0.5)))
     )
-    (property "Footprint" "Resistor_SMD:R_0603_1608Metric" (id 2) (at 106.68 59.69 0)
+    (property "Footprint" "02_dyn_pcblib:C0603" (id 2) (at 106.68 59.69 0)
       (effects (font (size 1.27 1.27)) hide)
     )
@@
     (pin "2")
   )
-  (symbol (lib_name "R0603_10k_2") (lib_id "01dyn_lib:R0603_10k") (at 73.66 63.5 0) (unit 1)
+  (symbol (lib_id "1001_un:R0603_10k") (at 73.66 63.5 0) (unit 1)
     (in_bom yes) (on_board yes) (fields_autoplaced)
     (property "Reference" "R623" (id 0) (at 73.66 58.42 0)
@@
       (effects (font (size 0.5 0.5)))
     )
-    (property "Footprint" "Resistor_SMD:R_0603_1608Metric" (id 2) (at 74.93 59.69 0)
+    (property "Footprint" "02_dyn_pcblib:C0603" (id 2) (at 74.93 59.69 0)
       (effects (font (size 1.27 1.27)) hide)
     )
@@
     (pin "2")
   )
-  (symbol (lib_id "01dyn_lib:R0603_DNP") (at 105.41 54.61 0) (unit 1)
+  (symbol (lib_id "1001_un:R0603_DNP") (at 105.41 54.61 0) (unit 1)
     (in_bom yes) (on_board yes) (fields_autoplaced)
     (property "Reference" "R604" (id 0) (at 105.41 49.53 0)
@@
       (effects (font (size 0.5 0.5)) hide)
     )
-    (property "Footprint" "Resistor_SMD:R_0603_1608Metric_Pad0.98x0.95mm_HandSolder" (id 2) (at 106.68 50.8 0)
+    (property "Footprint" "02_dyn_pcblib:C0603" (id 2) (at 106.68 50.8 0)
       (effects (font (size 1.27 1.27)) hide)
     )
@@
     (pin "2")
   )
-  (symbol (lib_name "R0603_10k_3") (lib_id "01dyn_lib:R0603_10k") (at 73.66 72.39 0) (unit 1)
+  (symbol (lib_id "1001_un:R0603_10k") (at 73.66 72.39 0) (unit 1)
     (in_bom yes) (on_board yes) (fields_autoplaced)
     (property "Reference" "R633" (id 0) (at 73.66 67.31 0)
@@
       (effects (font (size 0.5 0.5)))
     )
-    (property "Footprint" "Resistor_SMD:R_0603_1608Metric" (id 2) (at 74.93 68.58 0)
+    (property "Footprint" "02_dyn_pcblib:C0603" (id 2) (at 74.93 68.58 0)
       (effects (font (size 1.27 1.27)) hide)
     )
@@
     (pin "2")
   )
-  (symbol (lib_name "R0603_10k_1") (lib_id "01dyn_lib:R0603_10k") (at 105.41 72.39 0) (unit 1)
+  (symbol (lib_id "1001_un:R0603_10k") (at 105.41 72.39 0) (unit 1)
     (in_bom yes) (on_board yes) (fields_autoplaced)
     (property "Reference" "R634" (id 0) (at 105.41 67.31 0)
@@
       (effects (font (size 0.5 0.5)))
     )
-    (property "Footprint" "Resistor_SMD:R_0603_1608Metric" (id 2) (at 106.68 68.58 0)
+    (property "Footprint" "02_dyn_pcblib:C0603" (id 2) (at 106.68 68.58 0)
       (effects (font (size 1.27 1.27)) hide)
     )

Commit message: x
Parts:
- R603: symbol 1001_un:R0805_0.0 -> 1002_res:R0805_0.0
- R604: symbol 1001_un:R0603_DNP -> 1002_res:R0603_DNP
- R623, R624, R633, R634: symbol 1001_un:R0603_10k -> 1002_res:R0603_10k
Changed lines of the file:
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@@
     )
   )
-  (symbol (lib_id "1001_un:R0805_0.0") (at 73.66 54.61 0) (unit 1)
+  (symbol (lib_id "1002_res:R0805_0.0") (at 73.66 54.61 0) (unit 1)
     (in_bom yes) (on_board yes) (fields_autoplaced)
     (property "Reference" "R603" (id 0) (at 73.66 49.53 0)
@@
     (pin "2")
   )
-  (symbol (lib_id "1001_un:R0603_10k") (at 105.41 63.5 0) (unit 1)
+  (symbol (lib_id "1002_res:R0603_10k") (at 105.41 63.5 0) (unit 1)
     (in_bom yes) (on_board yes) (fields_autoplaced)
     (property "Reference" "R624" (id 0) (at 105.41 58.42 0)
@@
     (pin "2")
   )
-  (symbol (lib_id "1001_un:R0603_10k") (at 73.66 63.5 0) (unit 1)
+  (symbol (lib_id "1002_res:R0603_10k") (at 73.66 63.5 0) (unit 1)
     (in_bom yes) (on_board yes) (fields_autoplaced)
     (property "Reference" "R623" (id 0) (at 73.66 58.42 0)
@@
     (pin "2")
   )
-  (symbol (lib_id "1001_un:R0603_DNP") (at 105.41 54.61 0) (unit 1)
+  (symbol (lib_id "1002_res:R0603_DNP") (at 105.41 54.61 0) (unit 1)
     (in_bom yes) (on_board yes) (fields_autoplaced)
     (property "Reference" "R604" (id 0) (at 105.41 49.53 0)
@@
     (pin "2")
   )
-  (symbol (lib_id "1001_un:R0603_10k") (at 73.66 72.39 0) (unit 1)
+  (symbol (lib_id "1002_res:R0603_10k") (at 73.66 72.39 0) (unit 1)
     (in_bom yes) (on_board yes) (fields_autoplaced)
     (property "Reference" "R633" (id 0) (at 73.66 67.31 0)
@@
     (pin "2")
   )
-  (symbol (lib_id "1001_un:R0603_10k") (at 105.41 72.39 0) (unit 1)
+  (symbol (lib_id "1002_res:R0603_10k") (at 105.41 72.39 0) (unit 1)
     (in_bom yes) (on_board yes) (fields_autoplaced)
     (property "Reference" "R634" (id 0) (at 105.41 67.31 0)

Commit message: x
Parts:
- added C601: c0603_50v1u, 02_dyn_pcblib:C0603, symbol 1003_cap:c0603_50v1u
- added R691, R692, R693, R694, R695: R0603_DNP, 02_dyn_pcblib:C0603, symbol 1002_res:R0603_DNP
- added U601: mcu_MSP430FR2433IRGER, 02_dyn_pcblib:QFN-24-1EP_4x4mm_P0.5mm_EP2.8x2.8mmX, symbol 1009_ic:mcu_MSP430FR2433IRGER
- R603: value R0805_0.0 -> R0603_DNP; footprint 02_dyn_pcblib:R0805mix0603 -> 02_dyn_pcblib:C0603; symbol 1002_res:R0805_0.0 -> 1002_res:R0603_DNP; Notice (none) -> This DNP resistor use handly footprint, which is larger tha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; PartDesc 0 Ohms Jumper 0.125W, 1/8W Chip Resistor 0805 (2012 Metric)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 -> (none); PartNum RC0805JR-070RL -> R0603_DNP
Connections:
- net at R603.2, R604.1: now also C601.2, U601.24 (dVCC)
- net at R623.2: now also U601.10 (P1.3/A3/i2cSCL); no longer R624.1
- net at R634.1: now also U601.7 (P1.0/A0); no longer R633.2
- new net: C601.1, U601.18 (DvssGND), U601.23 (DvssGND), U601.25 (GND), U601.26 (GND), U601.27 (GND), U601.28 (GND)
- new net: R693.1, U601.11 (P2.2)
- new net: R693.2, U601.12 (P3.0)
- new net: R692.1, U601.19 (P2.7)
- new net: R692.2, U601.20 (p3.2)
- new net: R691.2, U601.21 (p2.0)
- new net: R691.1, U601.22 (p2.1)
- new net: R695.1, U601.3 (P1.4/A4)
- new net: R695.2, U601.4 (P1.5/A5)
- new net: R694.1, U601.5 (P1.6/A6)
- new net: R694.2, U601.6 (P1.7/A7)
- new net: R624.1, U601.8 (P1.1/A1)
- new net: R633.2, U601.9 (P1.2/A2/i2cSDA)
Other:
- moved on the sheet: R603, R604, R623, R624, R633, R634

Commit message: x
Parts:
- C601, R603, R604, R623, R624, R633, R634, R691, R692, R693, R694, R695: footprint 02_dyn_pcblib:C0603 -> 2004_cap:C0603
- U601: footprint 02_dyn_pcblib:QFN-24-1EP_4x4mm_P0.5mm_EP2.8x2.8mmX -> 2006_qfn:QFN-24-1EP_4x4mm_P0.5mm_EP2.8x2.8mmX
Changed lines of the file:
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@@
       (effects (font (size 1.5 1.5)))
     )
-    (property "Value" "c0603_50v1u" (id 1) (at 121.92 74.93 90)
-      (effects (font (size 0.5 0.5)))
-    )
-    (property "Footprint" "02_dyn_pcblib:C0603" (id 2) (at 109.093 77.851 0)
+    (property "Value" "c0603_50v1u" (id 1) (at 122.047 78.613 0)
+      (effects (font (size 0.5 0.5)))
+    )
+    (property "Footprint" "2004_cap:C0603" (id 2) (at 109.093 77.851 0)
       (effects (font (size 1.27 1.27)) hide)
     )
@@
       (effects (font (size 0.9 0.9)))
     )
-    (property "Footprint" "02_dyn_pcblib:QFN-24-1EP_4x4mm_P0.5mm_EP2.8x2.8mmX" (id 2) (at 130.81 74.93 0)
+    (property "Footprint" "2006_qfn:QFN-24-1EP_4x4mm_P0.5mm_EP2.8x2.8mmX" (id 2) (at 130.81 74.93 0)
       (effects (font (size 1.27 1.27)) hide)
     )
@@
       (effects (font (size 0.5 0.5)))
     )
-    (property "Footprint" "02_dyn_pcblib:C0603" (id 2) (at 99.06 80.01 0)
+    (property "Footprint" "2004_cap:C0603" (id 2) (at 99.06 80.01 0)
       (effects (font (size 1.27 1.27)) hide)
     )
@@
       (effects (font (size 0.5 0.5)))
     )
-    (property "Footprint" "02_dyn_pcblib:C0603" (id 2) (at 111.76 162.56 0)
+    (property "Footprint" "2004_cap:C0603" (id 2) (at 111.76 162.56 0)
       (effects (font (size 1.27 1.27)) hide)
     )
@@
       (effects (font (size 0.5 0.5)))
     )
-    (property "Footprint" "02_dyn_pcblib:C0603" (id 2) (at 128.27 90.17 0)
+    (property "Footprint" "2004_cap:C0603" (id 2) (at 128.27 90.17 0)
       (effects (font (size 1.27 1.27)) hide)
     )
@@
       (effects (font (size 0.5 0.5)))
     )
-    (property "Footprint" "02_dyn_pcblib:C0603" (id 2) (at 99.06 129.54 0)
+    (property "Footprint" "2004_cap:C0603" (id 2) (at 99.06 129.54 0)
       (effects (font (size 1.27 1.27)) hide)
     )
@@
       (effects (font (size 0.5 0.5)))
     )
-    (property "Footprint" "02_dyn_pcblib:C0603" (id 2) (at 87.63 129.54 0)
+    (property "Footprint" "2004_cap:C0603" (id 2) (at 87.63 129.54 0)
       (effects (font (size 1.27 1.27)) hide)
     )
@@
       (effects (font (size 0.5 0.5)))
     )
-    (property "Footprint" "02_dyn_pcblib:C0603" (id 2) (at 114.3 167.64 0)
+    (property "Footprint" "2004_cap:C0603" (id 2) (at 114.3 167.64 0)
       (effects (font (size 1.27 1.27)) hide)
     )
@@
       (effects (font (size 0.5 0.5)))
     )
-    (property "Footprint" "02_dyn_pcblib:C0603" (id 2) (at 135.89 90.17 0)
+    (property "Footprint" "2004_cap:C0603" (id 2) (at 135.89 90.17 0)
       (effects (font (size 1.27 1.27)) hide)
     )
@@
       (effects (font (size 0.5 0.5)))
     )
-    (property "Footprint" "02_dyn_pcblib:C0603" (id 2) (at 95.25 82.55 0)
+    (property "Footprint" "2004_cap:C0603" (id 2) (at 95.25 82.55 0)
       (effects (font (size 1.27 1.27)) hide)
     )
@@
       (effects (font (size 0.5 0.5)))
     )
-    (property "Footprint" "02_dyn_pcblib:C0603" (id 2) (at 135.89 152.4 0)
+    (property "Footprint" "2004_cap:C0603" (id 2) (at 135.89 152.4 0)
       (effects (font (size 1.27 1.27)) hide)
     )
@@
       (effects (font (size 0.5 0.5)))
     )
-    (property "Footprint" "02_dyn_pcblib:C0603" (id 2) (at 114.3 161.29 0)
+    (property "Footprint" "2004_cap:C0603" (id 2) (at 114.3 161.29 0)
       (effects (font (size 1.27 1.27)) hide)
     )
@@
       (effects (font (size 0.5 0.5)))
     )
-    (property "Footprint" "02_dyn_pcblib:C0603" (id 2) (at 111.76 153.67 0)
-      (effects (font (size 1.27 1.27)) hide)
-    )
+    (property "Footprint" "2004_cap:C0603" (id 2) (at 111.76 153.67 0)
+      (effects (font (size 1.27 1.27)) hide)
+    )

Commit message: x
Parts:
- R603, R604, R623, R624, R633, R634, R691, R692, R693, R694, R695: footprint 2004_cap:C0603 -> 2003_res:R0603
Changed lines of the file:
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@@
       (effects (font (size 0.5 0.5)))
     )
-    (property "Footprint" "2004_cap:C0603" (id 2) (at 99.06 80.01 0)
+    (property "Footprint" "2003_res:R0603" (id 2) (at 99.06 80.01 0)
       (effects (font (size 1.27 1.27)) hide)
     )
@@
       (effects (font (size 0.5 0.5)))
     )
-    (property "Footprint" "2004_cap:C0603" (id 2) (at 111.76 162.56 0)
+    (property "Footprint" "2003_res:R0603" (id 2) (at 111.76 162.56 0)
       (effects (font (size 1.27 1.27)) hide)
     )
@@
       (effects (font (size 0.5 0.5)))
     )
-    (property "Footprint" "2004_cap:C0603" (id 2) (at 128.27 90.17 0)
+    (property "Footprint" "2003_res:R0603" (id 2) (at 128.27 90.17 0)
       (effects (font (size 1.27 1.27)) hide)
     )
@@
       (effects (font (size 0.5 0.5)))
     )
-    (property "Footprint" "2004_cap:C0603" (id 2) (at 99.06 129.54 0)
+    (property "Footprint" "2003_res:R0603" (id 2) (at 99.06 129.54 0)
       (effects (font (size 1.27 1.27)) hide)
     )
@@
       (effects (font (size 0.5 0.5)))
     )
-    (property "Footprint" "2004_cap:C0603" (id 2) (at 87.63 129.54 0)
+    (property "Footprint" "2003_res:R0603" (id 2) (at 87.63 129.54 0)
       (effects (font (size 1.27 1.27)) hide)
     )
@@
       (effects (font (size 0.5 0.5)))
     )
-    (property "Footprint" "2004_cap:C0603" (id 2) (at 114.3 167.64 0)
+    (property "Footprint" "2003_res:R0603" (id 2) (at 114.3 167.64 0)
       (effects (font (size 1.27 1.27)) hide)
     )
@@
       (effects (font (size 0.5 0.5)))
     )
-    (property "Footprint" "2004_cap:C0603" (id 2) (at 135.89 90.17 0)
+    (property "Footprint" "2003_res:R0603" (id 2) (at 135.89 90.17 0)
       (effects (font (size 1.27 1.27)) hide)
     )
@@
       (effects (font (size 0.5 0.5)))
     )
-    (property "Footprint" "2004_cap:C0603" (id 2) (at 95.25 82.55 0)
+    (property "Footprint" "2003_res:R0603" (id 2) (at 95.25 82.55 0)
       (effects (font (size 1.27 1.27)) hide)
     )
@@
       (effects (font (size 0.5 0.5)))
     )
-    (property "Footprint" "2004_cap:C0603" (id 2) (at 135.89 152.4 0)
+    (property "Footprint" "2003_res:R0603" (id 2) (at 135.89 152.4 0)
       (effects (font (size 1.27 1.27)) hide)
     )
@@
       (effects (font (size 0.5 0.5)))
     )
-    (property "Footprint" "2004_cap:C0603" (id 2) (at 114.3 161.29 0)
+    (property "Footprint" "2003_res:R0603" (id 2) (at 114.3 161.29 0)
       (effects (font (size 1.27 1.27)) hide)
     )
@@
       (effects (font (size 0.5 0.5)))
     )
-    (property "Footprint" "2004_cap:C0603" (id 2) (at 111.76 153.67 0)
-      (effects (font (size 1.27 1.27)) hide)
-    )
+    (property "Footprint" "2003_res:R0603" (id 2) (at 111.76 153.67 0)
+      (effects (font (size 1.27 1.27)) hide)
+    )

Commit message: x
Parts:
- added H602: p2mm54_1x4, 2002_hdr:p2mm54_1x4, symbol 1008_hdr:p2mm54_1x4
- added R611, R644, R693, R694, R695: R0603_DNP, 2003_res:R0603, symbol 1002_res:R0603_DNP
- renumbered R693 to R643, R694 to R696, R695 to R697
Connections:
- net GND: now reaches C601.1, U601.18 (DvssGND), U601.23 (DvssGND), U601.25 (GND), U601.26 (GND), U601.27 (GND), U601.28 (GND)
- net GND: now also H602.4
- net at C601.2, R603.2, R604.1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: now also R611.1
- net SBWTdio: now reaches U601.1 (SBWTdio)
- net SBWTdio: now also H602.3, R611.2
- net at U601.11 (P2.2): now also R695.1; no longer R643.1
- net at U601.12 (P3.0): now also R695.2; no longer R643.2
- net at U601.13 (P2.3): now also R694.1, R694.2
- net at U601.14 (P3.1): now also R693.2
- net at U601.15 (P2.4): now also R693.1
- net at U601.16 (P2.5): now also R644.2
- net at U601.17 (P2.6): now also R643.2
- net SBWTck: now reaches U601.2 (SBWTck)
- net SBWTck: now also H602.2
- net at R697.1, U601.3 (P1.4/A4): now also H602.1
- new net Vena3: R643.1
- new net Vena4: R644.1
Other:
- moved on the sheet: C601, R603, R604, R623, R624, R633, R634, R643, R691, R692, R696, R697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
