File: kicad01_power_board_for_nuclear_team/007_output_socket.kicad_sch (KiCad schematic)
At the start: 0 parts

Commit message: x
Parts:
- added R705, R718, R724: R0603_1M, Resistor_SMD:R_0603_1608Metric, symbol 01dyn_lib:R0603_1M
Connections:
- new net V18out: R718.2
- new net V24out: R724.2
- new net V5out: R705.2
Changed lines of the file:
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@@
 (kicad_sch (version 20211123) (generator eeschema)
   (paper "A4")
+  (wire (pts (xy 217.17 52.07) (xy 217.17 50.8))
+    (stroke (width 0) (type default) (color 0 0 0 0))
+  )
+  (wire (pts (xy 109.22 49.53) (xy 119.38 49.53))
+    (stroke (width 0) (type default) (color 0 0 0 0))
+  )
+  (wire (pts (xy 167.64 62.23) (xy 167.64 59.69))
+    (stroke (width 0) (type default) (color 0 0 0 0))
+  )
+  (wire (pts (xy 157.48 50.8) (xy 167.64 50.8))
+    (stroke (width 0) (type default) (color 0 0 0 0))
+  )
+  (wire (pts (xy 119.38 50.8) (xy 119.38 49.53))
+    (stroke (width 0) (type default) (color 0 0 0 0))
+  )
+  (wire (pts (xy 217.17 62.23) (xy 217.17 59.69))
+    (stroke (width 0) (type default) (color 0 0 0 0))
+  )
+  (wire (pts (xy 107.95 60.96) (xy 119.38 60.96))
+    (stroke (width 0) (type default) (color 0 0 0 0))
+  )
+  (wire (pts (xy 205.74 62.23) (xy 217.17 62.23))
+    (stroke (width 0) (type default) (color 0 0 0 0))
+  )
+  (wire (pts (xy 156.21 62.23) (xy 167.64 62.23))
+    (stroke (width 0) (type default) (color 0 0 0 0))
+  )
+  (wire (pts (xy 167.64 52.07) (xy 167.64 50.8))
+    (stroke (width 0) (type default) (color 0 0 0 0))
+  )
+  (wire (pts (xy 119.38 60.96) (xy 119.38 58.42))
+    (stroke (width 0) (type default) (color 0 0 0 0))
+  )
+  (wire (pts (xy 207.01 50.8) (xy 217.17 50.8))
+    (stroke (width 0) (type default) (color 0 0 0 0))
+  )
+  (global_label "V24out" (shape input) (at 109.22 49.53 180) (fields_autoplaced)
+    (effects (font (size 1.27 1.27)) (justify right))
+    (property "Intersheet References" "${INTERSHEET_REFS}" (id 0) (at 100.2755 49.4506 0)
+      (effects (font (size 1.27 1.27)) (justify right) hide)
+    )
+  )
+  (global_label "V5out" (shape input) (at 207.01 50.8 180) (fields_autoplaced)
+    (effects (font (size 1.27 1.27)) (justify right))
+    (property "Intersheet References" "${INTERSHEET_REFS}" (id 0) (at 199.275 50.7206 0)
+      (effects (font (size 1.27 1.27)) (justify right) hide)
+    )
+  )
+  (global_label "V18out" (shape input) (at 157.48 50.8 180) (fields_autoplaced)
+    (effects (font (size 1.27 1.27)) (justify right))
+    (property "Intersheet References" "${INTERSHEET_REFS}" (id 0) (at 148.5355 50.8794 0)
+      (effects (font (size 1.27 1.27)) (justify right) hide)
+    )
+  )
+  (symbol (lib_id "01dyn_lib:GND_1") (at 156.21 62.23 0) (unit 1)
+    (in_bom yes) (on_board yes) (fields_autoplaced)
+    (property "Reference" "#PWR0115" (id 0) (at 156.21 68.58 0)
+      (effects (font (size 1.27 1.27)) hide)
+    )
+    (property "Value" "GND" (id 1) (at 156.21 66.04 0))
+    (property "Footprint" "" (id 2) (at 156.21 62.23 0)
+      (effects (font (size 1.27 1.27)) hide)
+    )
+    (property "Datasheet" "" (id 3) (at 156.21 62.23 0)
+      (effects (font (size 1.27 1.27)) hide)
+    )
+    (pin "1")
+  )
+  (symbol (lib_name "R0603_1M_2") (lib_id "01dyn_lib:R0603_1M") (at 167.64 55.88 90) (unit 1)
+    (in_bom yes) (on_board yes) (fields_autoplaced)
+    (property "Reference" "R718" (id 0) (at 170.18 55.245 90)
+      (effects (font (size 1.5 1.5)) (justify right))
+    )
+    (property "Value" "R0603_1M" (id 1) (at 169.037 57.658 0)
+      (effects (font (size 0.5 0.5)))
+    )
+    (property "Footprint" "Resistor_SMD:R_0603_1608Metric" (id 2) (at 157.48 54.61 0)
+      (effects (font (size 1.27 1.27)) hide)
+    )
+    (property "Datasheet" "~" (id 3) (at 167.64 55.88 90)
+      (effects (font (size 1.27 1.27)) hide)
+    )
+    (property "PartNum" "ERJ-U03F1004V" (id 4) (at 160.02 57.15 0)
+      (effects (font (size 1.27 1.27)) hide)
+    )
+    (property "PartDesc" "1 MOhms ±1% 0.1W, 1/10W Chip Resistor 0603 (1608 Metric) Anti-Sulfur, Automotive AEC-Q200 Thick Film" (id 5) (at 153.67 57.15 0)
+      (effects (font (size 1.27 1.27)) hide)
+    )
+    (pin "1")
+    (pin "2")
+  )
+  (symbol (lib_id "01dyn_lib:GND_1") (at 107.95 60.96 0) (unit 1)
+    (in_bom yes) (on_board yes) (fields_autoplaced)
+    (property "Reference" "#PWR0116" (id 0) (at 107.95 67.31 0)
+      (effects (font (size 1.27 1.27)) hide)
+    )
+    (property "Value" "GND" (id 1) (at 107.95 64.77 0))
+    (property "Footprint" "" (id 2) (at 107.95 60.96 0)
+      (effects (font (size 1.27 1.27)) hide)
+    )
+    (property "Datasheet" "" (id 3) (at 107.95 60.96 0)
+      (effects (font (size 1.27 1.27)) hide)
+    )
+    (pin "1")
+  )
+  (symbol (lib_id "01dyn_lib:GND_1") (at 205.74 62.23 0) (unit 1)
+    (in_bom yes) (on_board yes) (fields_autoplaced)
+    (property "Reference" "#PWR0114" (id 0) (at 205.74 68.58 0)
+      (effects (font (size 1.27 1.27)) hide)
+    )
+    (property "Value" "GND" (id 1) (at 205.74 66.04 0))
+    (property "Footprint" "" (id 2) (at 205.74 62.23 0)
+      (effects (font (size 1.27 1.27)) hide)
+    )
+    (property "Datasheet" "" (id 3) (at 205.74 62.23 0)
+      (effects (font (size 1.27 1.27)) hide)
+    )
+    (pin "1")
+  )
+  (symbol (lib_name "R0603_1M_1") (lib_id "01dyn_lib:R0603_1M") (at 217.17 55.88 90) (unit 1)
+    (in_bom yes) (on_board yes) (fields_autoplaced)
+    (property "Reference" "R705" (id 0) (at 219.71 55.245 90)
+      (effects (font (size 1.5 1.5)) (justify right))
+    )
+    (property "Value" "R0603_1M" (id 1) (at 218.567 57.658 0)
+      (effects (font (size 0.5 0.5)))
+    )
+    (property "Footprint" "Resistor_SMD:R_0603_1608Metric" (id 2) (at 207.01 54.61 0)
+      (effects (font (size 1.27 1.27)) hide)
+    )
+    (property "Datasheet" "~" (id 3) (at 217.17 55.88 90)
+      (effects (font (size 1.27 1.27)) hide)
+    )
+    (property "PartNum" "ERJ-U03F1004V" (id 4) (at 209.55 57.15 0)
+      (effects (font (size 1.27 1.27)) hide)
+    )
+    (property "PartDesc" "1 MOhms ±1% 0.1W, 1/10W Chip Resistor 0603 (1608 Metric) Anti-Sulfur, Automotive AEC-Q200 Thick Film" (id 5) (at 203.2 57.15 0)
+      (effects (font (size 1.27 1.27)) hide)
+    )
+    (pin "1")
+    (pin "2")
+  )
+  (symbol (lib_id "01dyn_lib:R0603_1M") (at 119.38 54.61 90) (unit 1)
+    (in_bom yes) (on_board yes) (fields_autoplaced)
+    (property "Reference" "R724" (id 0) (at 121.92 53.975 90)
+      (effects (font (size 1.5 1.5)) (justify right))
+    )
+    (property "Value" "R0603_1M" (id 1) (at 120.777 56.388 0)
+      (effects (font (size 0.5 0.5)))
+    )
+    (property "Footprint" "Resistor_SMD:R_0603_1608Metric" (id 2) (at 109.22 53.34 0)
+      (effects (font (size 1.27 1.27)) hide)
+    )
+    (property "Datasheet" "~" (id 3) (at 119.38 54.61 90)
+      (effects (font (size 1.27 1.27)) hide)
+    )
+    (property "PartNum" "ERJ-U03F1004V" (id 4) (at 111.76 55.88 0)
+      (effects (font (size 1.27 1.27)) hide)
+    )
+    (property "PartDesc" "1 MOhms ±1% 0.1W, 1/10W Chip Resistor 0603 (1608 Metric) Anti-Sulfur, Automotive AEC-Q200 Thick Film" (id 5) (at 105.41 55.88 0)
+      (effects (font (size 1.27 1.27)) hide)
+    )
+    (pin "1")
+    (pin "2")
+  )
 )

Commit message: ix
Parts:
- removed R705, R718, R724: R0603_1M, Resistor_SMD:R_0603_1608Metric, symbol 01dyn_lib:R0603_1M
- added C701, C711, C721: c0805_35v10u, 02_dyn_pcblib:C0805mix0603, symbol 1001_un:c0805_35v10u
- added H701, H711, H721: hdr_2x1_1-1123723-2, 02_dyn_pcblib:hdr_2x1_1-1123723-2, symbol 1001_un:hdr_2x1_1-1123723-2
Connections:
- net V18out: now also C711.2, H711.2
- net V24out: now also C701.2, H701.2
- net V5out: now also C721.2, H721.2
- new net GND: C701.1, C711.1, C721.1, H701.1, H711.1, H721.1

Commit message: x
Parts:
- C701, C711, C721: symbol 1001_un:c0805_35v10u -> 1003_cap:c0805_35v10u
Changed lines of the file:
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@@
     (pin "2")
   )
-  (symbol (lib_id "1001_un:c0805_35v10u") (at 132.08 63.5 0) (unit 1)
+  (symbol (lib_id "1003_cap:c0805_35v10u") (at 132.08 63.5 0) (unit 1)
     (in_bom yes) (on_board yes) (fields_autoplaced)
     (property "Reference" "C711" (id 0) (at 135.89 62.865 0)
@@
     (pin "1")
   )
-  (symbol (lib_id "1001_un:c0805_35v10u") (at 193.04 62.23 0) (unit 1)
+  (symbol (lib_id "1003_cap:c0805_35v10u") (at 193.04 62.23 0) (unit 1)
     (in_bom yes) (on_board yes) (fields_autoplaced)
     (property "Reference" "C721" (id 0) (at 196.85 61.595 0)
@@
     (pin "2")
   )
-  (symbol (lib_id "1001_un:c0805_35v10u") (at 71.12 60.96 0) (unit 1)
+  (symbol (lib_id "1003_cap:c0805_35v10u") (at 71.12 60.96 0) (unit 1)
     (in_bom yes) (on_board yes) (fields_autoplaced)
     (property "Reference" "C701" (id 0) (at 74.93 60.325 0)

Commit message: x
Parts:
- H701, H711, H721: symbol 1001_un:hdr_2x1_1-1123723-2 -> 1008_hdr:hdr_2x1_1-1123723-2
Changed lines of the file:
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@@
     (pin "1")
   )
-  (symbol (lib_id "1001_un:hdr_2x1_1-1123723-2") (at 125.73 63.5 90) (unit 1)
+  (symbol (lib_id "1008_hdr:hdr_2x1_1-1123723-2") (at 125.73 63.5 90) (unit 1)
     (in_bom yes) (on_board yes)
     (property "Reference" "H711" (id 0) (at 125.73 58.42 90)
@@
     (pin "2")
   )
-  (symbol (lib_id "1001_un:hdr_2x1_1-1123723-2") (at 64.77 60.96 90) (unit 1)
+  (symbol (lib_id "1008_hdr:hdr_2x1_1-1123723-2") (at 64.77 60.96 90) (unit 1)
     (in_bom yes) (on_board yes)
     (property "Reference" "H701" (id 0) (at 64.77 55.88 90)
@@
     (pin "2")
   )
-  (symbol (lib_id "1001_un:hdr_2x1_1-1123723-2") (at 186.69 63.5 90) (unit 1)
+  (symbol (lib_id "1008_hdr:hdr_2x1_1-1123723-2") (at 186.69 63.5 90) (unit 1)
     (in_bom yes) (on_board yes)
     (property "Reference" "H721" (id 0) (at 186.69 58.42 90)

Commit message: x
Parts:
- C701, C711, C721: footprint 02_dyn_pcblib:C0805mix0603 -> 2004_cap:C0805mix0603
- H701, H711, H721: footprint 02_dyn_pcblib:hdr_2x1_1-1123723-2 -> 2002_hdr:hdr_2x1_1-1123723-2
Changed lines of the file:
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@@
       (effects (font (size 0.4 0.4)))
     )
-    (property "Footprint" "02_dyn_pcblib:hdr_2x1_1-1123723-2" (id 2) (at 114.3 63.5 0)
+    (property "Footprint" "2002_hdr:hdr_2x1_1-1123723-2" (id 2) (at 114.3 63.5 0)
       (effects (font (size 1.27 1.27)) hide)
     )
@@
       (effects (font (size 0.4 0.4)))
     )
-    (property "Footprint" "02_dyn_pcblib:hdr_2x1_1-1123723-2" (id 2) (at 53.34 60.96 0)
+    (property "Footprint" "2002_hdr:hdr_2x1_1-1123723-2" (id 2) (at 53.34 60.96 0)
       (effects (font (size 1.27 1.27)) hide)
     )
@@
       (effects (font (size 0.5 0.5)))
     )
-    (property "Footprint" "02_dyn_pcblib:C0805mix0603" (id 2) (at 132.969 50.673 0)
+    (property "Footprint" "2004_cap:C0805mix0603" (id 2) (at 132.969 50.673 0)
       (effects (font (size 1.27 1.27)) hide)
     )
@@
       (effects (font (size 0.4 0.4)))
     )
-    (property "Footprint" "02_dyn_pcblib:hdr_2x1_1-1123723-2" (id 2) (at 175.26 63.5 0)
+    (property "Footprint" "2002_hdr:hdr_2x1_1-1123723-2" (id 2) (at 175.26 63.5 0)
       (effects (font (size 1.27 1.27)) hide)
     )
@@
       (effects (font (size 0.5 0.5)))
     )
-    (property "Footprint" "02_dyn_pcblib:C0805mix0603" (id 2) (at 193.929 49.403 0)
+    (property "Footprint" "2004_cap:C0805mix0603" (id 2) (at 193.929 49.403 0)
       (effects (font (size 1.27 1.27)) hide)
     )
@@
       (effects (font (size 0.5 0.5)))
     )
-    (property "Footprint" "02_dyn_pcblib:C0805mix0603" (id 2) (at 72.009 48.133 0)
+    (property "Footprint" "2004_cap:C0805mix0603" (id 2) (at 72.009 48.133 0)
       (effects (font (size 1.27 1.27)) hide)
     )
