File: kicad01_power_board_for_nuclear_team/008_board_and_testpoint.kicad_sch (KiCad schematic)
At the start: 1 part

Commit message: x
Parts:
- added H1, H2, H3, H4: hole2mm50_7mm40, 02_dyn_pcblib:hole2mm50_7mm40, symbol 1001_un:hole2mm50_7mm40
Connections:
- new net GND: H1.1, H2.1, H3.1, H4.1
Changed lines of the file:
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@@
 (kicad_sch (version 20211123) (generator eeschema)
   (paper "A4")
+  (junction (at 43.18 60.96) (diameter 0) (color 0 0 0 0)
+  )
+  (junction (at 43.18 69.85) (diameter 0) (color 0 0 0 0)
+  )
+  (junction (at 43.18 80.01) (diameter 0) (color 0 0 0 0)
+  )
+  (wire (pts (xy 43.18 69.85) (xy 46.99 69.85))
+    (stroke (width 0) (type default) (color 0 0 0 0))
+  )
+  (wire (pts (xy 43.18 50.8) (xy 46.99 50.8))
+    (stroke (width 0) (type default) (color 0 0 0 0))
+  )
+  (wire (pts (xy 43.18 87.63) (xy 43.18 80.01))
+    (stroke (width 0) (type default) (color 0 0 0 0))
+  )
+  (wire (pts (xy 43.18 69.85) (xy 43.18 60.96))
+    (stroke (width 0) (type default) (color 0 0 0 0))
+  )
+  (wire (pts (xy 43.18 60.96) (xy 43.18 50.8))
+    (stroke (width 0) (type default) (color 0 0 0 0))
+  )
+  (wire (pts (xy 43.18 80.01) (xy 46.99 80.01))
+    (stroke (width 0) (type default) (color 0 0 0 0))
+  )
+  (wire (pts (xy 43.18 60.96) (xy 46.99 60.96))
+    (stroke (width 0) (type default) (color 0 0 0 0))
+  )
+  (wire (pts (xy 43.18 80.01) (xy 43.18 69.85))
+    (stroke (width 0) (type default) (color 0 0 0 0))
+  )
+  (symbol (lib_id "power:GND") (at 43.18 87.63 0) (unit 1)
+    (in_bom yes) (on_board yes) (fields_autoplaced)
+    (property "Reference" "#PWR0117" (id 0) (at 43.18 93.98 0)
+      (effects (font (size 1.27 1.27)) hide)
+    )
+    (property "Value" "GND" (id 1) (at 43.18 91.44 0))
+    (property "Footprint" "" (id 2) (at 43.18 87.63 0)
+      (effects (font (size 1.27 1.27)) hide)
+    )
+    (property "Datasheet" "" (id 3) (at 43.18 87.63 0)
+      (effects (font (size 1.27 1.27)) hide)
+    )
+    (pin "1")
+  )
+  (symbol (lib_id "1001_un:hole2mm50_7mm40") (at 52.07 60.96 0) (unit 1)
+    (in_bom yes) (on_board yes) (fields_autoplaced)
+    (property "Reference" "H2" (id 0) (at 55.88 60.325 0)
+      (effects (font (size 1.5 1.5)) (justify left))
+    )
+    (property "Value" "hole2mm50_7mm40" (id 1) (at 52.197 62.865 0)
+      (effects (font (size 0.4 0.4)))
+    )
+    (property "Footprint" "02_dyn_pcblib:hole2mm50_7mm40" (id 2) (at 52.07 49.53 0)
+      (effects (font (size 1.27 1.27)) hide)
+    )
+    (property "Datasheet" "~" (id 3) (at 52.07 60.96 90)
+      (effects (font (size 1.27 1.27)) hide)
+    )
+    (property "PartNum" "hole2mm50_DNP" (id 4) (at 50.038 51.943 0)
+      (effects (font (size 1.27 1.27)) hide)
+    )
+    (property "PartDesc" "hole2mm50_DNP" (id 5) (at 49.53 46.99 0)
+      (effects (font (size 1.27 1.27)) hide)
+    )
+    (pin "1")
+  )
+  (symbol (lib_id "1001_un:hole2mm50_7mm40") (at 52.07 69.85 0) (unit 1)
+    (in_bom yes) (on_board yes) (fields_autoplaced)
+    (property "Reference" "H3" (id 0) (at 55.88 69.215 0)
+      (effects (font (size 1.5 1.5)) (justify left))
+    )
+    (property "Value" "hole2mm50_7mm40" (id 1) (at 52.197 71.755 0)
+      (effects (font (size 0.4 0.4)))
+    )
+    (property "Footprint" "02_dyn_pcblib:hole2mm50_7mm40" (id 2) (at 52.07 58.42 0)
+      (effects (font (size 1.27 1.27)) hide)
+    )
+    (property "Datasheet" "~" (id 3) (at 52.07 69.85 90)
+      (effects (font (size 1.27 1.27)) hide)
+    )
+    (property "PartNum" "hole2mm50_DNP" (id 4) (at 50.038 60.833 0)
+      (effects (font (size 1.27 1.27)) hide)
+    )
+    (property "PartDesc" "hole2mm50_DNP" (id 5) (at 49.53 55.88 0)
+      (effects (font (size 1.27 1.27)) hide)
+    )
+    (pin "1")
+  )
   (symbol (lib_id "1001_un:nucleco_power_board_v101") (at 49.53 36.83 0) (unit 1)
     (in_bom yes) (on_board yes)
@@
     )
   )
+  (symbol (lib_id "1001_un:hole2mm50_7mm40") (at 52.07 50.8 0) (unit 1)
+    (in_bom yes) (on_board yes) (fields_autoplaced)
+    (property "Reference" "H1" (id 0) (at 55.88 50.165 0)
+      (effects (font (size 1.5 1.5)) (justify left))
+    )
+    (property "Value" "hole2mm50_7mm40" (id 1) (at 52.197 52.705 0)
+      (effects (font (size 0.4 0.4)))
+    )
+    (property "Footprint" "02_dyn_pcblib:hole2mm50_7mm40" (id 2) (at 52.07 39.37 0)
+      (effects (font (size 1.27 1.27)) hide)
+    )
+    (property "Datasheet" "~" (id 3) (at 52.07 50.8 90)
+      (effects (font (size 1.27 1.27)) hide)
+    )
+    (property "PartNum" "hole2mm50_DNP" (id 4) (at 50.038 41.783 0)
+      (effects (font (size 1.27 1.27)) hide)
+    )
+    (property "PartDesc" "hole2mm50_DNP" (id 5) (at 49.53 36.83 0)
+      (effects (font (size 1.27 1.27)) hide)
+    )
+    (pin "1")
+  )
+  (symbol (lib_id "1001_un:hole2mm50_7mm40") (at 52.07 80.01 0) (unit 1)
+    (in_bom yes) (on_board yes) (fields_autoplaced)
+    (property "Reference" "H4" (id 0) (at 55.88 79.375 0)
+      (effects (font (size 1.5 1.5)) (justify left))
+    )
+    (property "Value" "hole2mm50_7mm40" (id 1) (at 52.197 81.915 0)
+      (effects (font (size 0.4 0.4)))
+    )
+    (property "Footprint" "02_dyn_pcblib:hole2mm50_7mm40" (id 2) (at 52.07 68.58 0)
+      (effects (font (size 1.27 1.27)) hide)
+    )
+    (property "Datasheet" "~" (id 3) (at 52.07 80.01 90)
+      (effects (font (size 1.27 1.27)) hide)
+    )
+    (property "PartNum" "hole2mm50_DNP" (id 4) (at 50.038 70.993 0)
+      (effects (font (size 1.27 1.27)) hide)
+    )
+    (property "PartDesc" "hole2mm50_DNP" (id 5) (at 49.53 66.04 0)
+      (effects (font (size 1.27 1.27)) hide)
+    )
+    (pin "1")
+  )
 )

Commit message: x
Parts:
- B801: symbol 1001_un:nucleco_power_board_v101 -> 1007_board:nucleco_power_board_v101
- H1, H2, H3, H4: symbol 1001_un:hole2mm50_7mm40 -> 1005_hole:hole2mm50_7mm40
Changed lines of the file:
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@@
     (pin "1")
   )
-  (symbol (lib_id "1001_un:hole2mm50_7mm40") (at 52.07 60.96 0) (unit 1)
+  (symbol (lib_id "1005_hole:hole2mm50_7mm40") (at 52.07 60.96 0) (unit 1)
     (in_bom yes) (on_board yes) (fields_autoplaced)
     (property "Reference" "H2" (id 0) (at 55.88 60.325 0)
@@
     (pin "1")
   )
-  (symbol (lib_id "1001_un:hole2mm50_7mm40") (at 52.07 69.85 0) (unit 1)
+  (symbol (lib_id "1005_hole:hole2mm50_7mm40") (at 52.07 69.85 0) (unit 1)
     (in_bom yes) (on_board yes) (fields_autoplaced)
     (property "Reference" "H3" (id 0) (at 55.88 69.215 0)
@@
     (pin "1")
   )
-  (symbol (lib_id "1001_un:nucleco_power_board_v101") (at 49.53 36.83 0) (unit 1)
+  (symbol (lib_id "1007_board:nucleco_power_board_v101") (at 49.53 36.83 0) (unit 1)
     (in_bom yes) (on_board yes)
     (property "Reference" "B801" (id 0) (at 45.72 35.56 0)
@@
     )
   )
-  (symbol (lib_id "1001_un:hole2mm50_7mm40") (at 52.07 50.8 0) (unit 1)
+  (symbol (lib_id "1005_hole:hole2mm50_7mm40") (at 52.07 50.8 0) (unit 1)
     (in_bom yes) (on_board yes) (fields_autoplaced)
     (property "Reference" "H1" (id 0) (at 55.88 50.165 0)
@@
     (pin "1")
   )
-  (symbol (lib_id "1001_un:hole2mm50_7mm40") (at 52.07 80.01 0) (unit 1)
+  (symbol (lib_id "1005_hole:hole2mm50_7mm40") (at 52.07 80.01 0) (unit 1)
     (in_bom yes) (on_board yes) (fields_autoplaced)
     (property "Reference" "H4" (id 0) (at 55.88 79.375 0)

Commit message: x
Parts:
- B801: footprint 02_dyn_pcblib:nucleco_power_board_v101 -> 2008_h3d:nucleco_power_board_v101
- H1, H2, H3, H4: footprint 02_dyn_pcblib:hole2mm50_7mm40 -> 2002_hdr:hole2mm50_7mm40
Changed lines of the file:
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@@
       (effects (font (size 0.4 0.4)))
     )
-    (property "Footprint" "02_dyn_pcblib:hole2mm50_7mm40" (id 2) (at 52.07 49.53 0)
+    (property "Footprint" "2002_hdr:hole2mm50_7mm40" (id 2) (at 52.07 49.53 0)
       (effects (font (size 1.27 1.27)) hide)
     )
@@
       (effects (font (size 0.4 0.4)))
     )
-    (property "Footprint" "02_dyn_pcblib:hole2mm50_7mm40" (id 2) (at 52.07 58.42 0)
+    (property "Footprint" "2002_hdr:hole2mm50_7mm40" (id 2) (at 52.07 58.42 0)
       (effects (font (size 1.27 1.27)) hide)
     )
@@
       (effects (font (size 0.5 0.5)))
     )
-    (property "Footprint" "02_dyn_pcblib:nucleco_power_board_v101" (id 2) (at 49.53 25.4 0)
+    (property "Footprint" "2008_h3d:nucleco_power_board_v101" (id 2) (at 49.53 25.4 0)
       (effects (font (size 1.27 1.27)) hide)
     )
@@
       (effects (font (size 0.4 0.4)))
     )
-    (property "Footprint" "02_dyn_pcblib:hole2mm50_7mm40" (id 2) (at 52.07 39.37 0)
+    (property "Footprint" "2002_hdr:hole2mm50_7mm40" (id 2) (at 52.07 39.37 0)
       (effects (font (size 1.27 1.27)) hide)
     )
@@
       (effects (font (size 0.4 0.4)))
     )
-    (property "Footprint" "02_dyn_pcblib:hole2mm50_7mm40" (id 2) (at 52.07 68.58 0)
+    (property "Footprint" "2002_hdr:hole2mm50_7mm40" (id 2) (at 52.07 68.58 0)
       (effects (font (size 1.27 1.27)) hide)
     )
